File: miains_timer_2/miains_timer_2.kicad_sch (KiCad schematic)
At the start: 40 parts, among them J1 PWR, J2 Conn_01x07, J3 AC_OUT, K1 ADW11, Q1 2N3904, SW1 SW_RST, U1 4027, U2 CD4060, U3 L7809, U4 4040

Commit message: a
Parts:
- removed K1: ADW11, Relay_THT:Relay_1P1T_NO_10x24x18.8mm_Panasonic_ADW11xxxxW_THT, symbol Relay:ADW11
- removed U3: L7809, Package_TO_SOT_THT:TO-220-3_Vertical, symbol Regulator_Linear:L7809
- added U?: L7812, symbol Regulator_Linear:L7812
- R4: value 1k -> 3k3
- R5: value 1k -> 3k
Connections:
- net +12V: now also C1.1, C5.1, C6.1, C7.1, C8.1, C9.1, R4.1, R5.1, R6.1, SW1.2 (B), U1.16 (VDD), U1.7 (S), U2.16 (Vcc), U4.16 (VDD), U?.3 (OUT); no longer C3.1, C4.1, D2.1 (K), D4.1 (K)
- net GND: now also U1.4 (R), U?.2 (GND); no longer U1.12 (R)
- net OSC_DIS: now also U1.14 (~{Q}); no longer U1.2 (~{Q})
- net OUT: now also U1.15 (Q); no longer U1.1 (Q)
- net RST: now also U1.12 (R); no longer U1.4 (R)
- net at J2.2 (Pin_2), R6.2: now also U1.9 (S); no longer U1.7 (S)
- removed net +5V: C1.1, C5.1, C6.1, C7.1, C8.1, C9.1, R4.1, R5.1, R6.1, SW1.2 (B), U1.16 (VDD), U1.9 (S), U2.16 (Vcc), U4.16 (VDD)
- new net: C3.1, C4.1, D2.1 (K), D4.1 (K), U?.1 (IN)
Other:
- note removed: "TODO NC contacts"
- moved on the sheet: D10, D12, D8, U1A, U1B
