File: weight_scale/weight_scale.kicad_pcb (KiCad board)
At the start: 2 copper layers, 20 parts, among them J1 Load cells, J2 ICSP_TagConnect, J3 UART, U1 MCP3421A0T-ECH, U2 ATmega169A-A, Y1 DNP

Commit message: a
Parts:
- added C10: 10n, Capacitor_SMD:C_0805_2012Metric_Pad1.18x1.45mm_HandSolder, F.Cu at (113.9, 43.9)
- added C11: 10n, Capacitor_SMD:C_0805_2012Metric_Pad1.18x1.45mm_HandSolder, F.Cu at (113.9, 39.8)
- added C12: 10u, Capacitor_SMD:C_1206_3216Metric_Pad1.33x1.80mm_HandSolder, F.Cu at (39.5, 62.5)
- added C13: 100n, Capacitor_SMD:C_0805_2012Metric_Pad1.18x1.45mm_HandSolder, F.Cu at (39.0, 60.0)
- added C14: 10u, Capacitor_SMD:C_1206_3216Metric_Pad1.33x1.80mm_HandSolder, F.Cu at (37.0, 53.5)
- added C15: 1u, Capacitor_SMD:C_0805_2012Metric_Pad1.18x1.45mm_HandSolder, F.Cu at (108.1, 54.4)
- added C16: 100n, Capacitor_SMD:C_0805_2012Metric_Pad1.18x1.45mm_HandSolder, F.Cu at (111.5, 61.0)
- added C17: 100n, Capacitor_SMD:C_0805_2012Metric_Pad1.18x1.45mm_HandSolder, F.Cu at (75.0, 67.0)
- added C18: 100n, Capacitor_SMD:C_0805_2012Metric_Pad1.18x1.45mm_HandSolder, F.Cu at (99.6, 47.6)
- added C9: 100n, Capacitor_SMD:C_0805_2012Metric_Pad1.18x1.45mm_HandSolder, F.Cu at (111.8, 41.9)
- added D2: CHG, LED_SMD:LED_0805_2012Metric_Pad1.15x1.40mm_HandSolder, F.Cu at (43.8, 55.2)
- added J4: BATT, Connector_PinHeader_2.54mm:PinHeader_1x02_P2.54mm_Horizontal, F.Cu at (33.6, 54.7)
- added J5: USB_B_Micro, Connector_USB:USB_Mini-B_Wuerth_65100516121_Horizontal, F.Cu at (34.6, 72.0)
- added L1: 10u, Inductor_SMD:L_0805_2012Metric_Pad1.15x1.40mm_HandSolder, F.Cu at (105.2, 47.5)
- added L2: 10u, Inductor_SMD:L_0805_2012Metric_Pad1.15x1.40mm_HandSolder, F.Cu at (115.0, 46.9)
- added R5: 5k1, Resistor_SMD:R_0805_2012Metric_Pad1.20x1.40mm_HandSolder, F.Cu at (43.0, 58.5)
- added R6: 1k, Resistor_SMD:R_0805_2012Metric_Pad1.20x1.40mm_HandSolder, F.Cu at (45.0, 58.5)
- added R7: 100, Resistor_SMD:R_0805_2012Metric_Pad1.20x1.40mm_HandSolder, F.Cu at (116.0, 39.9)
- added R8: 100, Resistor_SMD:R_0805_2012Metric_Pad1.20x1.40mm_HandSolder, F.Cu at (116.0, 43.9)
- added R9: 1k, Resistor_SMD:R_0805_2012Metric_Pad1.20x1.40mm_HandSolder, F.Cu at (86.0, 74.5)
- added U3: MCP73831-2-OT, Package_TO_SOT_SMD:SOT-23-5, F.Cu at (40.0, 56.4)
- added U4: GDC0570, footprints:GDC0570_LCD_6digits_2mmPitch, F.Cu at (103.3, 79.3)
- D1: value LED -> LED_Dual; footprint LED_SMD:LED_0805_2012Metric_Pad1.15x1.40mm_HandSolder -> LED_SMD:LED_Cree-PLCC4_3.2x2.8mm_CCW
- NT1: footprint Resistor_SMD:R_0805_2012Metric_Pad1.20x1.40mm_HandSolder -> NetTie:NetTie-2_SMD_Pad0.5mm; moved to B.Cu
- R1, R2: value 5k6 -> 5k1
- moved J1 67.4 mm to (120.9, 40.2), turned to 0 degrees
- moved C8 60.3 mm to (83.8, 68.1), turned to 180 degrees
- moved C7 59.4 mm to (83.8, 61.1), turned to 180 degrees
- moved Y1 52.8 mm to (88.6, 63.6), turned to -90 degrees
- moved C2 51.8 mm to (89.1, 61.0), turned to 180 degrees
- moved U1 46.8 mm to (108.8, 41.6), turned to -90 degrees
- moved NT1 44.8 mm to (115.2, 49.5), turned to -90 degrees
- moved J2 43.2 mm to (96.3, 52.4), turned to 180 degrees
- moved C6 43.0 mm to (77.5, 67.0), turned to 90 degrees
- moved C1 42.4 mm to (110.2, 45.3), turned to 0 degrees
- moved R1 41.5 mm to (105.0, 40.1), turned to 0 degrees
- moved R2 40.4 mm to (102.0, 41.0)
- moved J3 39.0 mm to (115.1, 51.2), turned to -90 degrees
- moved C3 38.3 mm to (109.7, 47.6), turned to 0 degrees
- moved U2 36.1 mm to (100.6, 64.6), turned to -90 degrees
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Connections:
- net +5V renamed +BATT
- C6 pad 1: /BTN -> /BTN0
- D1 pad 1: GND -> Net-(D1-A1)
- D1 pad 2: Net-(D1-A) -> Net-(D1-A2)
- J1 pad 1: GNDA -> /Vinp
- J1 pad 2: /Vinp -> /Vinn
- J1 pad 3: /Vinn -> Net-(J1-Pin_3)
- J1 pad 4: VDDA -> GNDA
- R1 pad 1: VDDA -> VDDF
- R2 pad 1: VDDA -> VDDF
- R3 pad 2: unconnected-(R3-Pad2) -> Net-(L1-Pad1)
- R4 pad 1: /LED -> /LED_1
- R4 pad 2: Net-(D1-A) -> Net-(D1-A1)
- U1 pad 1: /Vinp -> /Vinp_f
- U1 pad 6: /Vinn -> /Vinn_f
- U2 pad 1: unconnected-(U2-LCDCAP-Pad1) -> /Vlcdcap
- U2 pad 29: unconnected-(U2-PD4-Pad29) -> /BTN0
- U2 pad 30: unconnected-(U2-PD5-Pad30) -> /BTN1
- U2 pad 31: unconnected-(U2-PD6-Pad31) -> /LED_0
- U2 pad 32: unconnected-(U2-PD7-Pad32) -> /LED_1
- U2 pad 35: unconnected-(U2-PC0-Pad35) -> /SEG12
- U2 pad 36: unconnected-(U2-PC1-Pad36) -> /SEG11
- U2 pad 37: unconnected-(U2-PC2-Pad37) -> /SEG10
- U2 pad 38: unconnected-(U2-PC3-Pad38) -> /SEG9
- U2 pad 39: unconnected-(U2-PC4-Pad39) -> /SEG8
- U2 pad 4: /LED -> /PWR_loadCell
- U2 pad 40: unconnected-(U2-PC5-Pad40) -> /SEG7
- U2 pad 41: unconnected-(U2-PC6-Pad41) -> /SEG6
- U2 pad 42: unconnected-(U2-PC7-Pad42) -> /SEG5
- U2 pad 43: unconnected-(U2-PG2-Pad43) -> /SEG4
- U2 pad 44: unconnected-(U2-PA7-Pad44) -> /SEG3
- U2 pad 45: unconnected-(U2-PA6-Pad45) -> /SEG2
- U2 pad 46: unconnected-(U2-PA5-Pad46) -> /SEG1
- U2 pad 47: unconnected-(U2-PA4-Pad47) -> /SEG0
- U2 pad 5: /BTN -> /PWR_loadCell
- U2 pad 62: unconnected-(U2-AREF-Pad62) -> /Aref
- U2 pad 8: unconnected-(U2-PE6-Pad8) -> VDDF
Routing:
- net GND: track 0.00 -> 92.5 mm, vias 0 -> 24
- net +BATT: track 0.00 -> 70.2 mm
- net /SDA: track 0.00 -> 21.2 mm, vias 0 -> 2
- net /SCL: track 0.00 -> 20.1 mm
- net VDDF: track 0.00 -> 19.9 mm
- net +5V: track 0.00 -> 17.0 mm
- net RST: track 0.00 -> 16.5 mm
- net /COM0: track 0.00 -> 16.2 mm
- net VDDA: track 0.00 -> 15.2 mm
- net /BTN1: track 0.00 -> 14.3 mm
- net /BTN0: track 0.00 -> 14.2 mm
- net /COM1: track 0.00 -> 13.9 mm
- net /SEG12: track 0.00 -> 12.4 mm
- net GNDA: track 0.00 -> 12.3 mm, vias 0 -> 4
- net /PWR_loadCell: track 0.00 -> 12.1 mm
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- added copper zone on B.Cu, net GND
- added copper zone on B.Cu, net GNDA
- added copper zone on F.Cu, net GNDA
Other:
- board outline added: 93 x 60 mm

Commit message: PCINT and LCD low power
Connections:
- U2 pad 16: unconnected-(U2-PB6-Pad16) -> /BTN0
- U2 pad 17: unconnected-(U2-PB7-Pad17) -> /BTN1
- U2 pad 29: /BTN0 -> unconnected-(U2-PD4-Pad29)
- U2 pad 30: /BTN1 -> unconnected-(U2-PD5-Pad30)
Routing:
- net unconnected-(U2-PD5-Pad30): track 0.00 -> 14.3 mm
- net /BTN1: track 14.3 -> 0.00 mm
- net unconnected-(U2-PD4-Pad29): track 0.00 -> 14.2 mm
- net /BTN0: track 14.2 -> 0.00 mm
Changed lines of the file:
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@@
   (net 13 "unconnected-(U2-PB4-Pad14)")
   (net 14 "unconnected-(U2-PB5-Pad15)")
-  (net 15 "unconnected-(U2-PB6-Pad16)")
-  (net 16 "unconnected-(U2-PB7-Pad17)")
+  (net 15 "unconnected-(U2-PD4-Pad29)")
+  (net 16 "unconnected-(U2-PD5-Pad30)")
   (net 17 "unconnected-(U2-PG3-Pad18)")
   (net 18 "unconnected-(U2-PG4-Pad19)")
@@
       (net 14 "unconnected-(U2-PB5-Pad15)") (pinfunction "PB5") (pintype "bidirectional+no_connect"))
     (pad "16" smd rect (at -7.7 6 270) (size 1.5 0.55) (layers "F.Cu" "F.Paste" "F.Mask")
-      (net 15 "unconnected-(U2-PB6-Pad16)") (pinfunction "PB6") (pintype "bidirectional+no_connect"))
+      (net 69 "/BTN0") (pinfunction "PB6") (pintype "bidirectional"))
     (pad "17" smd rect (at -6 7.7) (size 1.5 0.55) (layers "F.Cu" "F.Paste" "F.Mask")
-      (net 16 "unconnected-(U2-PB7-Pad17)") (pinfunction "PB7") (pintype "bidirectional+no_connect"))
+      (net 70 "/BTN1") (pinfunction "PB7") (pintype "bidirectional"))
     (pad "18" smd rect (at -5.2 7.7) (size 1.5 0.55) (layers "F.Cu" "F.Paste" "F.Mask")
       (net 17 "unconnected-(U2-PG3-Pad18)") (pinfunction "PG3") (pintype "bidirectional+no_connect"))
@@
       (net 23 "unconnected-(U2-PD3-Pad28)") (pinfunction "PD3") (pintype "bidirectional+no_connect"))
     (pad "29" smd rect (at 3.6 7.7) (size 1.5 0.55) (layers "F.Cu" "F.Paste" "F.Mask")
-      (net 69 "/BTN0") (pinfunction "PD4") (pintype "bidirectional"))
+      (net 15 "unconnected-(U2-PD4-Pad29)") (pinfunction "PD4") (pintype "bidirectional"))
     (pad "30" smd rect (at 4.4 7.7) (size 1.5 0.55) (layers "F.Cu" "F.Paste" "F.Mask")
-      (net 70 "/BTN1") (pinfunction "PD5") (pintype "bidirectional"))
+      (net 16 "unconnected-(U2-PD5-Pad30)") (pinfunction "PD5") (pintype "bidirectional"))
     (pad "31" smd rect (at 5.2 7.7) (size 1.5 0.55) (layers "F.Cu" "F.Paste" "F.Mask")
       (net 74 "/LED_0") (pinfunction "PD6") (pintype "bidirectional"))
@@
   (segment (start 107.88125 40.28125) (end 106.14375 40.28125) (width 0.5) (layer "F.Cu") (net 12))
   (segment (start 102.56 56.9) (end 102.56 44.59) (width 0.5) (layer "F.Cu") (net 12))
+  (segment (start 92.86 68.2) (end 89.8 68.2) (width 0.5) (layer "F.Cu") (net 15))
+  (segment (start 89.8 68.2) (end 86.5 71.5) (width 0.5) (layer "F.Cu") (net 15))
+  (segment (start 86.5 71.5) (end 80 71.5) (width 0.5) (layer "F.Cu") (net 15))
+  (segment (start 92.86 69) (end 90.5 69) (width 0.5) (layer "F.Cu") (net 16))
+  (segment (start 87 72.5) (end 80 72.5) (width 0.5) (layer "F.Cu") (net 16))
+  (segment (start 90.5 69) (end 87 72.5) (width 0.5) (layer "F.Cu") (net 16))
   (segment (start 106.56875 42.98125) (end 106.55 43) (width 0.5) (layer "F.Cu") (net 19))
   (segment (start 103.8 42.05) (end 102.05 42.05) (width 0.5) (layer "F.Cu") (net 19))
@@
   (segment (start 105.76 72.3) (end 105.76 73.425) (width 0.5) (layer "F.Cu") (net 68))
   (segment (start 111.31 78.975) (end 111.31 79.3) (width 0.5) (layer "F.Cu") (net 68))
-  (segment (start 92.86 68.2) (end 89.8 68.2) (width 0.5) (layer "F.Cu") (net 69))
-  (segment (start 89.8 68.2) (end 86.5 71.5) (width 0.5) (layer "F.Cu") (net 69))
-  (segment (start 86.5 71.5) (end 80 71.5) (width 0.5) (layer "F.Cu") (net 69))
-  (segment (start 92.86 69) (end 90.5 69) (width 0.5) (layer "F.Cu") (net 70))
-  (segment (start 87 72.5) (end 80 72.5) (width 0.5) (layer "F.Cu") (net 70))
-  (segment (start 90.5 69) (end 87 72.5) (width 0.5) (layer "F.Cu") (net 70))
   (segment (start 83 76.2) (end 84.7 76.2) (width 0.5) (layer "F.Cu") (net 71))
   (segment (start 84.7 76.2) (end 85 76.5) (width 0.5) (layer "F.Cu") (net 71))
