File: weight_scale/Hardware/_autosave-weight_scale.kicad_pcb (KiCad board)
At the start: 2 copper layers, 51 x 51.7 mm, 53 parts, among them J1 Load cells, J2 ICSP_TagConnect, J3 UART, J4 BATT, J5 USB_B_Micro, Q1 Q_PMOS_GDS, U1 MCP6V67EMS, U2 ATmega169A-A, U3 MCP73831-2-OT, U4 GDC0570, U5 MCP3462, U6 MCP1711, Y1 DNP

Commit message: add
Routing:
- net /TX: track 5.94 -> 5.20 mm
- net /BTN0: track 15.4 -> 14.7 mm
Changed lines of the file:
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@@
     (fp_line (start 21 0) (end 17 0)
       (stroke (width 0.12) (type default)) (layer "F.SilkS"))
-    (fp_line (start -19 -14) (end -19 1.5)
-      (stroke (width 0.12) (type default)) (layer "F.CrtYd"))
-    (fp_line (start -19 0) (end -19 -14)
-      (stroke (width 0.12) (type default)) (layer "F.CrtYd"))
-    (fp_line (start -19 1.5) (end 21 1.5)
-      (stroke (width 0.12) (type default)) (layer "F.CrtYd"))
     (fp_line (start -16.85 -1.25) (end 16.85 -1.25)
       (stroke (width 0.05) (type default)) (layer "F.CrtYd"))
@@
     (fp_line (start 16.85 1.25) (end -16.85 1.25)
       (stroke (width 0.05) (type default)) (layer "F.CrtYd"))
-    (fp_line (start 21 -14) (end -19 -14)
-      (stroke (width 0.12) (type default)) (layer "F.CrtYd"))
-    (fp_line (start 21 -14) (end -19 -14)
-      (stroke (width 0.12) (type default)) (layer "F.CrtYd"))
-    (fp_line (start 21 1.5) (end 21 -14)
-      (stroke (width 0.12) (type default)) (layer "F.CrtYd"))
+    (fp_line (start -19 -14) (end -19 1.5)
+      (stroke (width 0.12) (type default)) (layer "F.Fab"))
+    (fp_line (start -19 1.5) (end 21 1.5)
+      (stroke (width 0.12) (type default)) (layer "F.Fab"))
     (fp_line (start -18.5 -14) (end 20.5 -14)
       (stroke (width 0.1) (type default)) (layer "F.Fab"))
@@
       (stroke (width 0.12) (type default)) (layer "F.Fab"))
     (fp_line (start 20.5 -2) (end 20.5 -14)
+      (stroke (width 0.12) (type default)) (layer "F.Fab"))
+    (fp_line (start 21 -14) (end -19 -14)
+      (stroke (width 0.12) (type default)) (layer "F.Fab"))
+    (fp_line (start 21 1.5) (end 21 -14)
       (stroke (width 0.12) (type default)) (layer "F.Fab"))
     (pad "1" thru_hole oval (at -16 0) (size 1.2 2) (drill 0.8) (layers "*.Cu" "*.Mask")
@@
   (segment (start 114.775 44.25) (end 115.875 45.35) (width 0.8) (layer "F.Cu") (net 1))
   (segment (start 119.45 36.6375) (end 120.6 36.6) (width 0.4) (layer "F.Cu") (net 1))
-  (segment (start 120.6 36.6) (end 120.5625 36.6375) (width 0.4) (layer "F.Cu") (net 1))
   (via (at 113.5 35.7) (size 0.8) (drill 0.4) (layers "F.Cu" "B.Cu") (net 1))
   (via (at 120.6 36.6) (size 0.8) (drill 0.4) (layers "F.Cu" "B.Cu") (net 1))
@@
   (segment (start 87.4 33.96) (end 87.4 35.26) (width 0.6) (layer "F.Cu") (net 8))
   (segment (start 86.8625 45.9975) (end 86.9 45.96) (width 0.6) (layer "F.Cu") (net 8))
-  (segment (start 87.4 35.26) (end 87.4 35.36) (width 0.6) (layer "F.Cu") (net 8))
   (segment (start 86.9 45.26) (end 86.9 45.96) (width 0.6) (layer "F.Cu") (net 8))
   (via (at 86.8 46.86) (size 0.8) (drill 0.4) (layers "F.Cu" "B.Cu") (net 8))
@@
   (segment (start 105.185 54.11) (end 105.185 49.645) (width 0.5) (layer "F.Cu") (net 34))
   (segment (start 104.385 54.11) (end 104.385 48.915) (width 0.5) (layer "F.Cu") (net 35))
-  (segment (start 104.385 48.915) (end 103.88 48.41) (width 0.5) (layer "F.Cu") (net 35))
-  (segment (start 104.385 48.43) (end 104.405 48.41) (width 0.5) (layer "F.Cu") (net 35))
   (segment (start 112.735 76.26) (end 105.985 69.51) (width 0.5) (layer "F.Cu") (net 36))
   (segment (start 112.735 76.51) (end 112.735 76.26) (width 0.5) (layer "F.Cu") (net 36))
@@
   (segment (start 86.5175 68.1175) (end 85.925 68.71) (width 0.5) (layer "F.Cu") (net 65))
   (segment (start 85.8 67.4) (end 86.5175 68.1175) (width 0.5) (layer "F.Cu") (net 65))
-  (segment (start 80.1 68.71) (end 79.425 68.71) (width 0.5) (layer "F.Cu") (net 65))
   (segment (start 92.285 65.41) (end 89.225 65.41) (width 0.5) (layer "F.Cu") (net 65))
   (segment (start 85.6375 67.4) (end 85.8 67.4) (width 0.5) (layer "F.Cu") (net 65))
@@
   (segment (start 109.025 27.625) (end 109 27.6) (width 0.6) (layer "F.Cu") (net 80))
   (segment (start 106.7 33.9) (end 106.7 37.9875) (width 0.5) (layer "F.Cu") (net 80))
-  (segment (start 106.7125 33.8875) (end 106.7125 33.7875) (width 0.5) (layer "F.Cu") (net 80))
   (segment (start 107 45.5) (end 107 43.4) (width 0.5) (layer "F.Cu") (net 80))
   (segment (start 106.675 40) (end 106.675 43.075) (width 0.5) (layer "F.Cu") (net 80))
@@
   (segment (start 109.025 28.85) (end 109.025 27.625) (width 0.6) (layer "F.Cu") (net 80))
   (segment (start 107 43.4) (end 106.675 43.075) (width 0.5) (layer "F.Cu") (net 80))
-  (segment (start 106.7 33.9) (end 106.7125 33.8875) (width 0.5) (layer "F.Cu") (net 80))
-  (segment (start 106.7125 33.9125) (end 106.7 33.9) (width 0.5) (layer "F.Cu") (net 80))
   (via (at 106.7 33.9) (size 0.8) (drill 0.4) (layers "F.Cu" "B.Cu") (net 80))
   (via (at 109 27.6) (size 0.8) (drill 0.4) (layers "F.Cu" "B.Cu") (net 80))
@@
     (polygon
       (pts
-        (xy 74 78)
-        (xy 125 78)
+        (xy 74 78.2)
+        (xy 125 78.2)
         (xy 125 26.5)
         (xy 74 26.5)
