File: weight_scale/Hardware/_autosave-weight_scale.kicad_sch (KiCad schematic)
At the start: 56 parts, among them J1 Load cells, J2 ICSP_TagConnect, J3 UART, J4 BATT, J5 USB_B_Micro, Q1 Q_PMOS_GDS, SW0 USER, SW1 USER, SW2 PWR, U1 MCP6V67EMS, U2 ATmega169A-A, U3 MCP73831-2-OT, U4 GDC0570, U5 MCP3462, U6 MCP1711, Y1 DNP

Commit message: add
Parts:
- added SW3: SW_Push, symbol Switch:SW_Push
- J4: footprint Connector_PinHeader_2.54mm:PinHeader_1x02_P2.54mm_Horizontal -> Connector_PinHeader_2.54mm:PinHeader_1x02_P2.54mm_Vertical
Changed lines of the file:
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@@
       (effects (font (size 1.27 1.27)) (justify left))
     )
-    (property "Footprint" "Connector_PinHeader_2.54mm:PinHeader_1x02_P2.54mm_Horizontal" (at 277.495 151.13 0)
+    (property "Footprint" "Connector_PinHeader_2.54mm:PinHeader_1x02_P2.54mm_Vertical" (at 277.495 151.13 0)
       (effects (font (size 1.27 1.27)) hide)
     )
@@
         )
       )
+    )
+  )
+  (symbol (lib_id "Switch:SW_Push") (at 46.355 187.96 0) (unit 1)
+    (in_bom yes) (on_board yes) (dnp no) (fields_autoplaced)
+    (property "Reference" "SW3" (at 46.355 182.0291 0)
+      (effects (font (size 1.27 1.27)))
+    )
+    (property "Value" "SW_Push" (at 46.355 183.9501 0)
+      (effects (font (size 1.27 1.27)))
+    )
+    (property "Footprint" "" (at 46.355 182.88 0)
+      (effects (font (size 1.27 1.27)) hide)
+    )
+    (property "Datasheet" "~" (at 46.355 182.88 0)
+      (effects (font (size 1.27 1.27)) hide)
+    )
+    (pin "1")
+    (pin "2")
+    (instances
+      (project "weight_scale"
+        (path "/c22e0349-8909-491e-993f-d6877deccd92"
+          (reference "SW3") (unit 1)
+        )
+      )
