File: weight_scale/Hardware/weight_scale.kicad_pcb (KiCad board)
At the start: 2 copper layers, 51 x 51.7 mm, 53 parts, among them J1 Load cells, J2 ICSP_TagConnect, J3 UART, J4 BATT, J5 USB_B_Micro, Q1 Q_PMOS_GDS, U1 MCP6V67EMS, U2 ATmega169A-A, U3 MCP73831-2-OT, U4 GDC0570, U5 MCP3462, U6 MCP1711, Y1 DNP

Commit message: add
Parts:
- added SW1: PWR, footprints:SW_PUSH_6mm_2pins, F.Cu at (113.2, 52.0)
- added SW2: BTN0, footprints:SW_PUSH_6mm_2pins, F.Cu at (80.2, 50.1)
- added SW3: BTN1, footprints:SW_PUSH_6mm_2pins, F.Cu at (80.2, 64.4)
- J1: value Load cells -> Load cell; footprint Connector_Samtec_HPM_THT:Samtec_HPM-04-01-x-S_Straight_1x04_Pitch5.08mm -> footprints:282834-4
- moved J1 15.6 mm to (84.5, 30.1)
- moved C11 11.5 mm to (76.4, 34.9), turned to 0 degrees
- moved C6 10.5 mm to (79.3, 58.3), turned to 0 degrees
- moved C17 8.20 mm to (78.0, 75.4), turned to -90 degrees
- moved R7 8.17 mm to (78.4, 37.4), turned to 180 degrees
- moved C9 6.26 mm to (80.4, 34.9), turned to 0 degrees
- moved C10 3.29 mm to (84.4, 34.9), turned to 0 degrees
- moved R8 2.53 mm to (82.4, 37.4), turned to 0 degrees
Connections:
- J1 pad 1: /Vinp -> Net-(J1-Pin_1)
- J1 pad 3: GNDA -> /Vinp
- J1 pad 4: Net-(J1-Pin_4) -> GNDA
- L2 pad 1: Net-(J1-Pin_4) -> Net-(J1-Pin_1)
Routing:
- net +BATT: track 9.02 -> 34.4 mm
- net Net-(U6-~{SHDN}): track 20.4 -> 36.6 mm, vias 2 -> 3
- net /BTN0: track 15.4 -> 29.4 mm
- net Net-(J1-Pin_4): track 10.9 -> 0.00 mm
- net /Vinp_f: track 2.31 -> 13.1 mm
- net /Vinp: track 21.1 -> 28.6 mm
- net /BTN1: track 12.4 -> 20.0 mm
- net GNDA: track 16.4 -> 22.4 mm, vias 7 -> 6
- net /Vinn: track 20.4 -> 26.1 mm
- net /Vfbp: track 18.1 -> 14.6 mm
- net Net-(J1-Pin_1): track 0.00 -> 2.79 mm
- net GND: track 100.2 -> 97.6 mm, vias 25 -> 29
- net /TX: track 5.94 -> 5.20 mm
Other:
- board text added: "E+ S- S+ E-"
- board text removed: "E+ E- S- S+"

Commit message: uart under test
Connections:
- U5 pad 5: /Voutn -> /Vinn
- U5 pad 6: /Vinn -> /Vinp
- U5 pad 7: /Vinp -> /Voutn
Routing:
- net /Voutn: track 10.9 -> 12.5 mm, vias 0 -> 2
Changed lines of the file:
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@@
       (net 6 "VDDA") (pinfunction "REFIN+") (pintype "input"))
     (pad "5" smd roundrect (at -2.8625 -0.325) (size 1.475 0.4) (layers "F.Cu" "F.Paste" "F.Mask") (roundrect_rratio 0.25)
-      (net 12 "/Voutn") (pinfunction "CH0") (pintype "input"))
+      (net 9 "/Vinn") (pinfunction "CH0") (pintype "input"))
     (pad "6" smd roundrect (at -2.8625 0.325) (size 1.475 0.4) (layers "F.Cu" "F.Paste" "F.Mask") (roundrect_rratio 0.25)
-      (net 9 "/Vinn") (pinfunction "CH1") (pintype "input"))
+      (net 10 "/Vinp") (pinfunction "CH1") (pintype "input"))
     (pad "7" smd roundrect (at -2.8625 0.975) (size 1.475 0.4) (layers "F.Cu" "F.Paste" "F.Mask") (roundrect_rratio 0.25)
-      (net 10 "/Vinp") (pinfunction "CH2") (pintype "input"))
+      (net 12 "/Voutn") (pinfunction "CH2") (pintype "input"))
     (pad "8" smd roundrect (at -2.8625 1.625) (size 1.475 0.4) (layers "F.Cu" "F.Paste" "F.Mask") (roundrect_rratio 0.25)
       (net 5 "/Voutp") (pinfunction "CH3") (pintype "input"))
@@
   (segment (start 103.2475 35.853997) (end 101.8 34.406497) (width 1) (layer "F.Cu") (net 4))
   (segment (start 89.035 43.435) (end 89.035 45.825) (width 0.6) (layer "F.Cu") (net 5))
-  (segment (start 90.851678 41.9595) (end 91.202178 42.31) (width 0.4) (layer "F.Cu") (net 5))
+  (segment (start 93.000707 42.7) (end 91.592178 42.7) (width 0.4) (layer "F.Cu") (net 5))
   (segment (start 88.9 45.96) (end 88.9 47.9225) (width 0.6) (layer "F.Cu") (net 5))
   (segment (start 88.9 47.9225) (end 88.9375 47.96) (width 0.6) (layer "F.Cu") (net 5))
   (segment (start 89.5005 41.9595) (end 90.851678 41.9595) (width 0.4) (layer "F.Cu") (net 5))
+  (segment (start 91.592178 42.7) (end 90.851678 41.9595) (width 0.4) (layer "F.Cu") (net 5))
   (segment (start 89.035 45.825) (end 88.9 45.96) (width 0.6) (layer "F.Cu") (net 5))
+  (segment (start 95.5 42.31) (end 93.390707 42.31) (width 0.4) (layer "F.Cu") (net 5))
   (segment (start 89.035 42.425) (end 89.5005 41.9595) (width 0.4) (layer "F.Cu") (net 5))
   (segment (start 89.035 43.435) (end 89.035 42.425) (width 0.4) (layer "F.Cu") (net 5))
-  (segment (start 91.202178 42.31) (end 95.5 42.31) (width 0.4) (layer "F.Cu") (net 5))
+  (segment (start 93.390707 42.31) (end 93.000707 42.7) (width 0.4) (layer "F.Cu") (net 5))
   (segment (start 89.6375 30.06) (end 89.325 30.06) (width 1) (layer "F.Cu") (net 6))
   (segment (start 95.5 39.71) (end 96.9 39.71) (width 0.4) (layer "F.Cu") (net 6))
@@
   (segment (start 87.8 35.9) (end 87.5 35.6) (width 0.4) (layer "B.Cu") (net 8))
   (segment (start 87.8 42.1) (end 87.8 35.9) (width 0.4) (layer "B.Cu") (net 8))
+  (segment (start 82.859501 40.659501) (end 81.4375 39.2375) (width 0.4) (layer "F.Cu") (net 9))
+  (segment (start 95.5 40.36) (end 93.307822 40.36) (width 0.4) (layer "F.Cu") (net 9))
+  (segment (start 93.307822 40.36) (end 93.248322 40.3005) (width 0.4) (layer "F.Cu") (net 9))
+  (segment (start 81.475 34.86875) (end 81.475 30.585) (width 0.8) (layer "F.Cu") (net 9))
   (segment (start 81.4375 39.2375) (end 81.4375 37.36875) (width 0.4) (layer "F.Cu") (net 9))
-  (segment (start 91.340499 40.659501) (end 82.859501 40.659501) (width 0.4) (layer "F.Cu") (net 9))
-  (segment (start 81.475 34.86875) (end 81.475 30.585) (width 0.8) (layer "F.Cu") (net 9))
   (segment (start 81.475 30.585) (end 81.96 30.1) (width 0.8) (layer "F.Cu") (net 9))
-  (segment (start 91.81 41.01) (end 91.4 40.6) (width 0.4) (layer "F.Cu") (net 9))
-  (segment (start 91.4 40.6) (end 91.340499 40.659501) (width 0.4) (layer "F.Cu") (net 9))
-  (segment (start 82.859501 40.659501) (end 81.4375 39.2375) (width 0.4) (layer "F.Cu") (net 9))
+  (segment (start 93.248322 40.3005) (end 91.351678 40.3005) (width 0.4) (layer "F.Cu") (net 9))
   (segment (start 83.4 34.86875) (end 81.475 34.86875) (width 0.8) (layer "F.Cu") (net 9))
   (segment (start 81.4375 34.90625) (end 81.475 34.86875) (width 0.8) (layer "F.Cu") (net 9))
+  (segment (start 90.992677 40.659501) (end 82.859501 40.659501) (width 0.4) (layer "F.Cu") (net 9))
+  (segment (start 91.351678 40.3005) (end 90.992677 40.659501) (width 0.4) (layer "F.Cu") (net 9))
   (segment (start 81.4375 37.36875) (end 81.4375 34.90625) (width 0.8) (layer "F.Cu") (net 9))
-  (segment (start 95.5 41.01) (end 91.81 41.01) (width 0.4) (layer "F.Cu") (net 9))
-  (segment (start 91.56 41.66) (end 91.2 41.3) (width 0.4) (layer "F.Cu") (net 10))
+  (segment (start 91.508089 40.991911) (end 91.2 41.3) (width 0.4) (layer "F.Cu") (net 10))
   (segment (start 81.1 41.3) (end 79.4375 39.6375) (width 0.4) (layer "F.Cu") (net 10))
+  (segment (start 79.4375 39.6375) (end 79.4375 37.36875) (width 0.4) (layer "F.Cu") (net 10))
   (segment (start 77.475 34.86875) (end 79.4 34.86875) (width 0.8) (layer "F.Cu") (net 10))
   (segment (start 79.4 37.33125) (end 79.4375 37.36875) (width 0.8) (layer "F.Cu") (net 10))
-  (segment (start 79.4375 39.6375) (end 79.4375 37.36875) (width 0.4) (layer "F.Cu") (net 10))
-  (segment (start 95.5 41.66) (end 91.56 41.66) (width 0.4) (layer "F.Cu") (net 10))
+  (segment (start 91.2 41.3) (end 81.1 41.3) (width 0.4) (layer "F.Cu") (net 10))
   (segment (start 79.4 30.12) (end 79.42 30.1) (width 0.8) (layer "F.Cu") (net 10))
   (segment (start 79.4 34.86875) (end 79.4 30.12) (width 0.8) (layer "F.Cu") (net 10))
   (segment (start 77.6575 34.68625) (end 77.475 34.86875) (width 1) (layer "F.Cu") (net 10))
-  (segment (start 91.2 41.3) (end 81.1 41.3) (width 0.4) (layer "F.Cu") (net 10))
+  (segment (start 95.481911 40.991911) (end 91.508089 40.991911) (width 0.4) (layer "F.Cu") (net 10))
+  (segment (start 95.5 41.01) (end 95.481911 40.991911) (width 0.4) (layer "F.Cu") (net 10))
   (segment (start 79.4 34.86875) (end 79.4 37.33125) (width 0.8) (layer "F.Cu") (net 10))
   (segment (start 89.035 36.225) (end 89.3 35.96) (width 0.6) (layer "F.Cu") (net 11))
@@
   (segment (start 89.035 38.485) (end 89.035 36.225) (width 0.6) (layer "F.Cu") (net 11))
   (segment (start 89.2625 35.9225) (end 89.3 35.96) (width 0.6) (layer "F.Cu") (net 11))
+  (segment (start 93.09 41.66) (end 92.75 42) (width 0.4) (layer "F.Cu") (net 12))
+  (segment (start 91.3 35.96) (end 91.3 38.4) (width 0.6) (layer "F.Cu") (net 12))
   (segment (start 91.3375 33.96) (end 91.3375 35.9225) (width 0.6) (layer "F.Cu") (net 12))
   (segment (start 91.3375 35.9225) (end 91.3 35.96) (width 0.6) (layer "F.Cu") (net 12))
-  (segment (start 92.18 40.36) (end 90.305 38.485) (width 0.4) (layer "F.Cu") (net 12))
-  (segment (start 91.3 35.96) (end 91.3 37.49) (width 0.6) (layer "F.Cu") (net 12))
-  (segment (start 95.5 40.36) (end 92.18 40.36) (width 0.4) (layer "F.Cu") (net 12))
-  (segment (start 91.3 37.49) (end 90.305 38.485) (width 0.6) (layer "F.Cu") (net 12))
+  (segment (start 91.3 38.5) (end 90.32 38.5) (width 0.6) (layer "F.Cu") (net 12))
+  (segment (start 90.32 38.5) (end 90.305 38.485) (width 0.6) (layer "F.Cu") (net 12))
+  (segment (start 91.3 38.4) (end 91.3 38.5) (width 0.6) (layer "F.Cu") (net 12))
+  (segment (start 95.5 41.66) (end 93.09 41.66) (width 0.4) (layer "F.Cu") (net 12))
+  (via (at 92.778631 41.791411) (size 0.8) (drill 0.4) (layers "F.Cu" "B.Cu") (free) (net 12))
+  (via (at 91.3 38.4) (size 0.8) (drill 0.4) (layers "F.Cu" "B.Cu") (net 12))
+  (segment (start 91.3 40.31278) (end 92.778631 41.791411) (width 0.6) (layer "B.Cu") (net 12))
+  (segment (start 91.3 38.4) (end 91.3 40.31278) (width 0.6) (layer "B.Cu") (net 12))
   (segment (start 111.35 42.85) (end 115.75 47.25) (width 0.4) (layer "F.Cu") (net 30))
   (segment (start 113.55 30.1725) (end 114.71 29.0125) (width 0.6) (layer "F.Cu") (net 30))

Commit message: uart under test
Other:
- board text added: "USB Recharge"
- board text removed: "USB Charge"
Changed lines of the file:
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@@
     (property "ki_keywords" "dual opamp zero drift")
     (attr smd)
-    (fp_text reference "U1" (at 1.29 -3.85 -180) (layer "F.SilkS")
+    (fp_text reference "U1" (at 1.94 -3.8 -180) (layer "F.SilkS")
         (effects (font (size 1 1) (thickness 0.15)))
     )
@@
     (property "ki_keywords" "150mA low-noise LDO linear voltage regulator fixed positive")
     (attr smd)
-    (fp_text reference "U6" (at 0.3875 2.55) (layer "F.SilkS")
+    (fp_text reference "U6" (at 3.0875 1.1) (layer "F.SilkS")
         (effects (font (size 1 1) (thickness 0.15)))
     )
@@
     (effects (font (size 1 1) (thickness 0.15)) (justify left bottom))
   )
-  (gr_text "USB\nCharge" (at 124.4 57.5 90) (layer "F.SilkS")
+  (gr_text "USB\nRecharge" (at 124.6 60 90) (layer "F.SilkS")
     (effects (font (size 1.5 1.5) (thickness 0.3) bold) (justify left bottom))
   )

Commit message: ADC basics
Parts:
- added H1: MountingHole_Pad, MountingHole:MountingHole_3.2mm_M3_Pad_Via, F.Cu at (77.6, 46.1)
- added H2: MountingHole_Pad, MountingHole:MountingHole_3.2mm_M3_Pad_Via, F.Cu at (120.1, 66.1)
- added R13: 1Meg, Resistor_SMD:R_0805_2012Metric_Pad1.20x1.40mm_HandSolder, F.Cu at (108.6, 43.0)
- R1: value 220 -> 330
- U1: value MCP6V67EMS -> MCP6V07
- moved R12 2.57 mm to (106.6, 43.0), turned to -90 degrees
Routing:
- net /RX: track 6.21 -> 11.5 mm
- net /PWR_en: track 10.7 -> 12.9 mm
- net GND: track 97.6 -> 99.7 mm
- net Net-(U6-~{SHDN}): track 36.6 -> 35.9 mm
