File: weight_scale/Hardware/weight_scale.kicad_sch (KiCad schematic)
At the start: 56 parts, among them J1 Load cells, J2 ICSP_TagConnect, J3 UART, J4 BATT, J5 USB_B_Micro, Q1 Q_PMOS_GDS, SW0 USER, SW1 USER, SW2 PWR, U1 MCP6V67EMS, U2 ATmega169A-A, U3 MCP73831-2-OT, U4 GDC0570, U5 MCP3462, U6 MCP1711, Y1 DNP

Commit message: add
Parts:
- removed SW0, SW1: USER, symbol Switch:SW_MEC_5E
- removed SW2: PWR, symbol Switch:SW_MEC_5E
- added SW1: PWR, footprints:SW_PUSH_6mm_2pins, symbol Switch:SW_Push
- added SW2: BTN0, footprints:SW_PUSH_6mm_2pins, symbol Switch:SW_Push
- added SW3: BTN1, footprints:SW_PUSH_6mm_2pins, symbol Switch:SW_Push
- J1: value Load cells -> Load cell; footprint Connector_Samtec_HPM_THT:Samtec_HPM-04-01-x-S_Straight_1x04_Pitch5.08mm -> footprints:282834-4
- J4: footprint Connector_PinHeader_2.54mm:PinHeader_1x02_P2.54mm_Horizontal -> Connector_PinHeader_2.54mm:PinHeader_1x02_P2.54mm_Vertical
Connections:
- net +BATT: now also SW1.2
- net BTN0: now also SW2.2
- net BTN1: now also SW3.2
- net GND: now also SW2.1, SW3.1
- net GNDA: now also J1.4 (Pin_4); no longer J1.3 (Pin_3)
- net Vinp: now also J1.3 (Pin_3); no longer J1.1 (Pin_1)
- net at C18.1, R11.1, R12.1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: now also SW1.1
- net at L2.1: now also J1.1 (Pin_1); no longer J1.4 (Pin_4)
Other:
- moved on the sheet: C6, J1

Commit message: uart under test
Parts:
- R1: value 220 -> 330
- U1: value MCP6V67EMS -> MCP6V07
Connections:
- net Vinn: now also U5.5 (CH0); no longer U5.6 (CH1)
- net Vinp: now also U5.6 (CH1); no longer U5.7 (CH2)
- net Voutn: now also U5.7 (CH2); no longer U5.5 (CH0)
Changed lines of the file:
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@@
     (effects (font (size 1.27 1.27)) (justify left bottom))
   )
-  (label "Voutn" (at 172.72 31.75 0) (fields_autoplaced)
+  (label "Voutn" (at 172.72 36.83 0) (fields_autoplaced)
     (effects (font (size 1.27 1.27)) (justify left bottom))
   )
@@
     (effects (font (size 1.27 1.27)) (justify left bottom))
   )
-  (label "Vinn" (at 172.72 34.29 0) (fields_autoplaced)
+  (label "Vinn" (at 172.72 31.75 0) (fields_autoplaced)
     (effects (font (size 1.27 1.27)) (justify left bottom))
   )
@@
     (effects (font (size 1.27 1.27)) (justify left bottom))
   )
-  (label "Vinp" (at 172.72 36.83 0) (fields_autoplaced)
+  (label "Vinp" (at 172.72 34.29 0) (fields_autoplaced)
     (effects (font (size 1.27 1.27)) (justify left bottom))
   )
@@
       (effects (font (size 1.27 1.27)) (justify right))
     )
-    (property "Value" "220" (at 137.033 37.4723 0)
+    (property "Value" "330" (at 137.033 37.4723 0)
       (effects (font (size 1.27 1.27)) (justify right))
     )
@@
       (effects (font (size 1.27 1.27)))
     )
-    (property "Value" "MCP6V67EMS" (at 142.875 56.3485 0)
+    (property "Value" "MCP6V07" (at 142.875 56.3485 0)
       (effects (font (size 1.27 1.27)))
     )
@@
       (effects (font (size 1.27 1.27)) (justify left))
     )
-    (property "Value" "MCP6V67EMS" (at 154.305 74.3023 0)
+    (property "Value" "MCP6V07" (at 154.305 74.3023 0)
       (effects (font (size 1.27 1.27)) (justify left))
     )
@@
       (effects (font (size 1.27 1.27)))
     )
-    (property "Value" "MCP6V67EMS" (at 142.875 18.5961 0)
-      (effects (font (size 1.27 1.27)))
-    )
+    (property "Value" "MCP6V07" (at 142.875 18.5961 0)
+      (effects (font (size 1.27 1.27)))
+    )

Commit message: ADC basics
Parts:
- added R13: 1Meg, Resistor_SMD:R_0805_2012Metric_Pad1.20x1.40mm_HandSolder, symbol Device:R
Connections:
- net GND: now also R13.2
- net RX: now also R13.1
Changed lines of the file:
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@@
     (stroke (width 0) (type default))
   )
+  (wire (pts (xy 38.735 111.76) (xy 38.735 109.22))
+    (stroke (width 0) (type default))
+  )
   (wire (pts (xy 198.755 145.415) (xy 198.755 147.955))
     (stroke (width 0) (type default))
@@
     (stroke (width 0) (type default))
   )
-  (wire (pts (xy 24.13 109.22) (xy 26.67 109.22))
+  (wire (pts (xy 24.13 109.22) (xy 38.735 109.22))
     (stroke (width 0) (type default))
   )
@@
     )
   )
+  (symbol (lib_id "Device:R") (at 38.735 115.57 0) (unit 1)
+    (in_bom yes) (on_board yes) (dnp no) (fields_autoplaced)
+    (property "Reference" "R13" (at 40.513 114.9263 0)
+      (effects (font (size 1.27 1.27)) (justify left))
+    )
+    (property "Value" "1Meg" (at 40.513 116.8473 0)
+      (effects (font (size 1.27 1.27)) (justify left))
+    )
+    (property "Footprint" "Resistor_SMD:R_0805_2012Metric_Pad1.20x1.40mm_HandSolder" (at 36.957 115.57 90)
+      (effects (font (size 1.27 1.27)) hide)
+    )
+    (property "Datasheet" "~" (at 38.735 115.57 0)
+      (effects (font (size 1.27 1.27)) hide)
+    )
+    (pin "1")
+    (pin "2")
+    (instances
+      (project "weight_scale"
+        (path "/c22e0349-8909-491e-993f-d6877deccd92"
+          (reference "R13") (unit 1)
+        )
+      )
+    )
+  )
   (symbol (lib_id "Device:C") (at 274.32 122.555 0) (unit 1)
     (in_bom yes) (on_board yes) (dnp no) (fields_autoplaced)
@@
         )
       )
+    )
+  )
+  (symbol (lib_id "power:GND") (at 38.735 119.38 0) (unit 1)
+    (in_bom yes) (on_board yes) (dnp no) (fields_autoplaced)
+    (property "Reference" "#PWR041" (at 38.735 125.73 0)
+      (effects (font (size 1.27 1.27)) hide)
+    )
+    (property "Value" "GND" (at 38.735 123.5155 0)
+      (effects (font (size 1.27 1.27)))
+    )
+    (property "Footprint" "" (at 38.735 119.38 0)
+      (effects (font (size 1.27 1.27)) hide)
+    )
+    (property "Datasheet" "" (at 38.735 119.38 0)
+      (effects (font (size 1.27 1.27)) hide)
+    )
+    (pin "1")
+    (instances
+      (project "weight_scale"
+        (path "/c22e0349-8909-491e-993f-d6877deccd92"
+          (reference "#PWR041") (unit 1)
+        )
+      )

Commit message: ADC basics
Parts:
- added H1, H2: MountingHole_Pad, MountingHole:MountingHole_3.2mm_M3_Pad_Via, symbol Mechanical:MountingHole_Pad
Connections:
- net GND: now also H1.1, H2.1
Other:
- note added: "TODO: Check USB connector Battery polarity Button footprint"
- note removed: "TODO: Check USB connector Check I2C pullup Check input filter Battery polarity Button footprint"
Changed lines of the file:
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@@
     (effects (font (size 1.27 1.27)) (justify left bottom))
   )
-  (text "TODO:\nCheck USB connector\nCheck I2C pullup\nCheck input filter\nBattery polarity\nButton footprint"
+  (text "TODO:\nCheck USB connector\nBattery polarity\nButton footprint"
     (at 135.255 167.64 0)
     (effects (font (size 1.27 1.27) (color 255 0 48 1)) (justify left bottom))
@@
     )
   )
+  (symbol (lib_id "power:GND") (at 33.655 191.135 0) (unit 1)
+    (in_bom yes) (on_board yes) (dnp no) (fields_autoplaced)
+    (property "Reference" "#PWR044" (at 33.655 197.485 0)
+      (effects (font (size 1.27 1.27)) hide)
+    )
+    (property "Value" "GND" (at 33.655 195.2705 0)
+      (effects (font (size 1.27 1.27)))
+    )
+    (property "Footprint" "" (at 33.655 191.135 0)
+      (effects (font (size 1.27 1.27)) hide)
+    )
+    (property "Datasheet" "" (at 33.655 191.135 0)
+      (effects (font (size 1.27 1.27)) hide)
+    )
+    (pin "1")
+    (instances
+      (project "weight_scale"
+        (path "/c22e0349-8909-491e-993f-d6877deccd92"
+          (reference "#PWR044") (unit 1)
+        )
+      )
+    )
+  )
   (symbol (lib_id "Device:C") (at 158.115 28.575 0) (unit 1)
     (in_bom yes) (on_board yes) (dnp no) (fields_autoplaced)
@@
     )
   )
+  (symbol (lib_id "power:GND") (at 40.005 191.135 0) (unit 1)
+    (in_bom yes) (on_board yes) (dnp no) (fields_autoplaced)
+    (property "Reference" "#PWR045" (at 40.005 197.485 0)
+      (effects (font (size 1.27 1.27)) hide)
+    )
+    (property "Value" "GND" (at 40.005 195.2705 0)
+      (effects (font (size 1.27 1.27)))
+    )
+    (property "Footprint" "" (at 40.005 191.135 0)
+      (effects (font (size 1.27 1.27)) hide)
+    )
+    (property "Datasheet" "" (at 40.005 191.135 0)
+      (effects (font (size 1.27 1.27)) hide)
+    )
+    (pin "1")
+    (instances
+      (project "weight_scale"
+        (path "/c22e0349-8909-491e-993f-d6877deccd92"
+          (reference "#PWR045") (unit 1)
+        )
+      )
+    )
+  )
   (symbol (lib_id "power:GNDA") (at 209.55 78.74 0) (unit 1)
     (in_bom yes) (on_board yes) (dnp no) (fields_autoplaced)
@@
         (path "/c22e0349-8909-491e-993f-d6877deccd92"
           (reference "#PWR05") (unit 1)
+        )
+      )
+    )
+  )
+  (symbol (lib_id "Mechanical:MountingHole_Pad") (at 33.655 188.595 0) (unit 1)
+    (in_bom yes) (on_board yes) (dnp no) (fields_autoplaced)
+    (property "Reference" "H1" (at 33.655 182.5371 0)
+      (effects (font (size 1.27 1.27)))
+    )
+    (property "Value" "MountingHole_Pad" (at 33.655 184.4581 0)
+      (effects (font (size 1.27 1.27)))
+    )
+    (property "Footprint" "MountingHole:MountingHole_3.2mm_M3_Pad_Via" (at 33.655 188.595 0)
+      (effects (font (size 1.27 1.27)) hide)
+    )
+    (property "Datasheet" "~" (at 33.655 188.595 0)
+      (effects (font (size 1.27 1.27)) hide)
+    )
+    (pin "1")
+    (instances
+      (project "weight_scale"
+        (path "/c22e0349-8909-491e-993f-d6877deccd92"
+          (reference "H1") (unit 1)
         )
       )
@@
         )
       )
+    )
+  )
+  (symbol (lib_id "Mechanical:MountingHole_Pad") (at 40.005 188.595 0) (unit 1)
+    (in_bom yes) (on_board yes) (dnp no) (fields_autoplaced)
+    (property "Reference" "H2" (at 42.545 186.6813 0)
+      (effects (font (size 1.27 1.27)) (justify left))
+    )
+    (property "Value" "MountingHole_Pad" (at 42.545 188.6023 0)
+      (effects (font (size 1.27 1.27)) (justify left))
+    )
+    (property "Footprint" "MountingHole:MountingHole_3.2mm_M3_Pad_Via" (at 40.005 188.595 0)
+      (effects (font (size 1.27 1.27)) hide)
+    )
+    (property "Datasheet" "~" (at 40.005 188.595 0)
+      (effects (font (size 1.27 1.27)) hide)
+    )
+    (pin "1")
+    (instances
+      (project "weight_scale"
+        (path "/c22e0349-8909-491e-993f-d6877deccd92"
+          (reference "H2") (unit 1)
+        )
+      )

Commit message: a
Parts:
- removed L2: 10u, Inductor_SMD:L_0805_2012Metric_Pad1.15x1.40mm_HandSolder, symbol Device:L_Ferrite
Connections:
- net VDDA: now also J1.1 (Pin_1)
Changed lines of the file:
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@@
     (stroke (width 0) (type default))
   )
-  (wire (pts (xy 94.615 31.75) (xy 87.63 31.75))
+  (wire (pts (xy 90.805 31.75) (xy 87.63 31.75))
     (stroke (width 0) (type default))
   )
@@
     (stroke (width 0) (type default))
   )
-  (wire (pts (xy 94.615 24.13) (xy 94.615 25.4))
-    (stroke (width 0) (type default))
-  )
   (bus (pts (xy 115.57 161.925) (xy 115.57 164.465))
     (stroke (width 0) (type default))
@@
     )
   )
-  (symbol (lib_id "power:VDDA") (at 94.615 25.4 0) (unit 1)
+  (symbol (lib_id "power:VDDA") (at 90.805 31.75 0) (unit 1)
     (in_bom yes) (on_board yes) (dnp no) (fields_autoplaced)
-    (property "Reference" "#PWR012" (at 94.615 29.21 0)
+    (property "Reference" "#PWR012" (at 90.805 35.56 0)
       (effects (font (size 1.27 1.27)) hide)
     )
-    (property "Value" "VDDA" (at 94.615 21.8981 0)
+    (property "Value" "VDDA" (at 90.805 28.2481 0)
       (effects (font (size 1.27 1.27)))
     )
-    (property "Footprint" "" (at 94.615 25.4 0)
+    (property "Footprint" "" (at 90.805 31.75 0)
       (effects (font (size 1.27 1.27)) hide)
     )
-    (property "Datasheet" "" (at 94.615 25.4 0)
+    (property "Datasheet" "" (at 90.805 31.75 0)
       (effects (font (size 1.27 1.27)) hide)
     )
@@
         )
       )
-    )
-  )
-  (symbol (lib_id "Device:L_Ferrite") (at 94.615 27.94 180) (unit 1)
-    (in_bom yes) (on_board yes) (dnp no) (fields_autoplaced)
-    (property "Reference" "L2" (at 95.25 27.2963 0)
-      (effects (font (size 1.27 1.27)) (justify right))
-    )
-    (property "Value" "10u" (at 95.25 29.2173 0)
-      (effects (font (size 1.27 1.27)) (justify right))
-    )
-    (property "Footprint" "Inductor_SMD:L_0805_2012Metric_Pad1.15x1.40mm_HandSolder" (at 94.615 27.94 0)
-      (effects (font (size 1.27 1.27)) hide)
-    )
-    (property "Datasheet" "~" (at 94.615 27.94 0)
-      (effects (font (size 1.27 1.27)) hide)
-    )
-    (pin "1")
-    (pin "2")
-    (instances
-      (project "weight_scale"
-        (path "/c22e0349-8909-491e-993f-d6877deccd92"
-          (reference "L2") (unit 1)
-        )
-      )
