File: RGB_strip_driver/RGB_strip_driver.kicad_pcb (KiCad board)
At the start: 2 copper layers, 46.7 x 19 mm, 33 parts, among them J1 PWR, J2 Prog, J3 LED, Q1 2N7002, Q2 2N7002, Q3 2N7002, Q4 VN3205, Q5 VN3205, Q6 VN3205, SW1 TL3330AF130QG, U1 ADP3336ARMZ, U2 PIC12F510-ISN

Commit message: added board gerbers
Other:
- net class Default removed
- board text added: "- +"
- board text added: "B R G V+"
