File: transistor_clock/DivByTwo.kicad_sch (KiCad schematic)
At the start: 20 parts, among them Q105 MMBT3906, Q21 MMBT3904, Q9 MMBT3906

Commit message: seconds_minor_wrapup
Parts:
- C76, D255, RV1: Assembly (none) -> False
- D22: value D -> 1N4148W; Assembly (none) -> True; LCSC_PN (none) -> C81598; Price (none) -> 0.0061
- Q105, Q9: value MMBT3906 -> MMBT5401; Assembly (none) -> True; LCSC_PN (none) -> C8326; Price (none) -> 0.0137
- Q121: renamed from Q21; Assembly (none) -> True; LCSC_PN (none) -> C20526; Price (none) -> 0.0094
- R20: LCSC_PN (none) -> C21190; Price (none) -> 0.0005
- R20: Assembly (none) -> True; LCSC_PN (none) -> C25804; Price (none) -> 0.0008
- R244: renamed from R41; LCSC_PN (none) -> C21190; Price (none) -> 0.0005
- R247: renamed from R41; Assembly (none) -> True; LCSC_PN (none) -> C25803; Price (none) -> 0.0009
- renumbered C6 to C33, C4 to C77, R41 to R246, R45 to R248, R41 to R249

Commit message: seconds_major_wrapup
Parts:
- removed D22: 1N4148W, Diode_SMD:D_SOD-123, symbol Device:D
- removed D255: LED, LED_SMD:LED_0603_1608Metric, symbol Device:LED
- removed R20: 1k, Resistor_SMD:R_0603_1608Metric, symbol Device:R
- removed R246: 2k2, Resistor_SMD:R_0603_1608Metric, symbol Device:R
- added R237: 10k, Resistor_SMD:R_0603_1608Metric, symbol Device:R
- C33: value 1.5u -> 1u
- R20: value 1k -> 2k2; Assembly (none) -> True
- R20: value 10k -> 100k; LCSC_PN C25804 -> C25803; Price 0.0008 -> 0.0009
- R244: Assembly (none) -> True
- R248: value 330 -> 2k2; Assembly (none) -> True; LCSC_PN (none) -> C21190; Price (none) -> 0.0005
- R249: value 2k2 -> 10k; Assembly (none) -> True; LCSC_PN (none) -> C25804; Price (none) -> 0.0008
Connections:
- net at Q105.1 (B), Q121.3 (C), R20.1: now also R237.2; no longer R249.2
- new net: R237.1, R249.2
Other:
- moved on the sheet: R249
