File: transistor_clock/2counter.kicad_sch (KiCad schematic)
At the start: 8 parts, among them Q11 MMBT3904

Commit message: seconds_minor_wrapup
Parts:
- C2, C76: Assembly (none) -> False
- D23: value D -> 1N4148W; Assembly (none) -> True; LCSC_PN (none) -> C81598; Price (none) -> 0.0061
- Q11: Assembly (none) -> True; LCSC_PN (none) -> C20526; Price (none) -> 0.0094
- R20: LCSC_PN (none) -> C21190; Price (none) -> 0.0005
- renumbered R82 to R17
Changed lines of the file:
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@@
+      (effects (font (size 1.27 1.27)) hide)
+    )
+    (property "Assembly" "" (at 39.37 97.79 0)
+      (effects (font (size 1.27 1.27)) hide)
+    )
+    (property "LCSC_PN" "" (at 39.37 97.79 0)
+      (effects (font (size 1.27 1.27)) hide)
+    )
+    (property "Price" "" (at 39.37 97.79 0)
       (effects (font (size 1.27 1.27)) hide)
     )
@@
       (effects (font (size 1.27 1.27)) hide)
     )
+    (property "Assembly" "" (at 46.99 97.79 0)
+      (effects (font (size 1.27 1.27)) hide)
+    )
+    (property "LCSC_PN" "C21190" (at 46.99 97.79 0)
+      (effects (font (size 1.27 1.27)) hide)
+    )
+    (property "Price" "0.0005" (at 46.99 97.79 0)
+      (effects (font (size 1.27 1.27)) hide)
+    )
     (pin "1")
     (pin "2")
@@
       (effects (font (size 1.27 1.27)) hide)
     )
+    (property "Assembly" "False" (at 73.66 81.28 0)
+      (effects (font (size 1.27 1.27)) hide)
+    )
+    (property "LCSC_PN" "" (at 73.66 81.28 0)
+      (effects (font (size 1.27 1.27)) hide)
+    )
+    (property "Price" "" (at 73.66 81.28 0)
+      (effects (font (size 1.27 1.27)) hide)
+    )
     (pin "1")
     (pin "2")
@@
       (effects (font (size 1.27 1.27)) hide)
     )
+    (property "Assembly" "False" (at 26.67 72.39 0)
+      (effects (font (size 1.27 1.27)) hide)
+    )
+    (property "LCSC_PN" "" (at 26.67 72.39 0)
+      (effects (font (size 1.27 1.27)) hide)
+    )
+    (property "Price" "" (at 26.67 72.39 0)
+      (effects (font (size 1.27 1.27)) hide)
+    )
     (pin "1")
     (pin "2")
@@
   (symbol (lib_id "Device:R") (at 66.04 72.39 0) (unit 1)
     (in_bom yes) (on_board yes) (dnp no) (fields_autoplaced)
-    (property "Reference" "R82" (at 67.818 71.7463 0)
+    (property "Reference" "R17" (at 67.818 71.7463 0)
       (effects (font (size 1.27 1.27)) (justify left))
     )
@@
     )
     (property "Datasheet" "~" (at 66.04 72.39 0)
+      (effects (font (size 1.27 1.27)) hide)
+    )
+    (property "Assembly" "" (at 66.04 72.39 0)
+      (effects (font (size 1.27 1.27)) hide)
+    )
+    (property "LCSC_PN" "" (at 66.04 72.39 0)
+      (effects (font (size 1.27 1.27)) hide)
+    )
+    (property "Price" "" (at 66.04 72.39 0)
       (effects (font (size 1.27 1.27)) hide)
     )
@@
       (effects (font (size 1.27 1.27)) hide)
     )
+    (property "Assembly" "" (at 36.83 72.39 0)
+      (effects (font (size 1.27 1.27)) hide)
+    )
+    (property "LCSC_PN" "" (at 36.83 72.39 0)
+      (effects (font (size 1.27 1.27)) hide)
+    )
+    (property "Price" "" (at 36.83 72.39 0)
+      (effects (font (size 1.27 1.27)) hide)
+    )
     (pin "1")
     (pin "2")
@@
   (symbol (lib_id "power:GND") (at 54.61 105.41 0) (unit 1)
     (in_bom yes) (on_board yes) (dnp no) (fields_autoplaced)
-    (property "Reference" "#PWR051" (at 54.61 111.76 0)
+    (property "Reference" "#PWR034" (at 54.61 111.76 0)
       (effects (font (size 1.27 1.27)) hide)
     )
@@
   (symbol (lib_id "power:GND") (at 66.04 105.41 0) (unit 1)
     (in_bom yes) (on_board yes) (dnp no) (fields_autoplaced)
-    (property "Reference" "#PWR053" (at 66.04 111.76 0)
+    (property "Reference" "#PWR033" (at 66.04 111.76 0)
       (effects (font (size 1.27 1.27)) hide)
     )
@@
       (effects (font (size 1.27 1.27)) (justify left) hide)
     )
+    (property "Assembly" "True" (at 63.5 97.79 0)
+      (effects (font (size 1.27 1.27)) hide)
+    )
+    (property "LCSC_PN" "C20526" (at 63.5 97.79 0)
+      (effects (font (size 1.27 1.27)) hide)
+    )
+    (property "Price" "0.0094" (at 63.5 97.79 0)
+      (effects (font (size 1.27 1.27)) hide)
+    )
     (pin "1")
     (pin "2")
@@
   (symbol (lib_id "power:GND") (at 26.67 76.2 0) (unit 1)
     (in_bom yes) (on_board yes) (dnp no) (fields_autoplaced)
-    (property "Reference" "#PWR050" (at 26.67 82.55 0)
+    (property "Reference" "#PWR09" (at 26.67 82.55 0)
       (effects (font (size 1.27 1.27)) hide)
     )
@@
   (symbol (lib_id "power:GND") (at 36.83 76.2 0) (unit 1)
     (in_bom yes) (on_board yes) (dnp no) (fields_autoplaced)
-    (property "Reference" "#PWR050" (at 36.83 82.55 0)
+    (property "Reference" "#PWR09" (at 36.83 82.55 0)
       (effects (font (size 1.27 1.27)) hide)
     )
@@
   (symbol (lib_id "power:VCC") (at 31.75 68.58 0) (unit 1)
     (in_bom yes) (on_board yes) (dnp no) (fields_autoplaced)
-    (property "Reference" "#PWR052" (at 31.75 72.39 0)
+    (property "Reference" "#PWR022" (at 31.75 72.39 0)
       (effects (font (size 1.27 1.27)) hide)
     )
@@
       (effects (font (size 1.27 1.27)) (justify left))
     )
-    (property "Value" "D" (at 56.642 102.8773 90)
+    (property "Value" "1N4148W" (at 56.642 102.8773 90)
       (effects (font (size 1.27 1.27)) (justify left))
     )
@@
     )
     (property "Sim.Pins" "1=K 2=A" (at 54.61 101.6 0)
+      (effects (font (size 1.27 1.27)) hide)
+    )
+    (property "Assembly" "True" (at 54.61 101.6 0)
+      (effects (font (size 1.27 1.27)) hide)
+    )
+    (property "LCSC_PN" "C81598" (at 54.61 101.6 0)
+      (effects (font (size 1.27 1.27)) hide)
+    )
+    (property "Price" "0.0061" (at 54.61 101.6 0)
       (effects (font (size 1.27 1.27)) hide)
     )
@@
   (symbol (lib_id "power:GND") (at 73.66 85.09 0) (unit 1)
     (in_bom yes) (on_board yes) (dnp no) (fields_autoplaced)
-    (property "Reference" "#PWR054" (at 73.66 91.44 0)
+    (property "Reference" "#PWR07" (at 73.66 91.44 0)
       (effects (font (size 1.27 1.27)) hide)
     )
@@
   (symbol (lib_id "power:VCC") (at 66.04 68.58 0) (unit 1)
     (in_bom yes) (on_board yes) (dnp no) (fields_autoplaced)
-    (property "Reference" "#PWR052" (at 66.04 72.39 0)
-      (effects (font (size 1.27 1.27)) hide)
-    )
+    (property "Reference" "#PWR022" (at 66.04 72.39 0)
+      (effects (font (size 1.27 1.27)) hide)
+    )

Commit message: seconds_major_wrapup
Parts:
- R17: Assembly (none) -> True; LCSC_PN (none) -> C25803; Price (none) -> 0.0009
- R20: Assembly (none) -> True
Changed lines of the file:
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@@
       (effects (font (size 1.27 1.27)) hide)
     )
-    (property "Assembly" "" (at 46.99 97.79 0)
+    (property "Assembly" "True" (at 46.99 97.79 0)
       (effects (font (size 1.27 1.27)) hide)
     )
@@
       (effects (font (size 1.27 1.27)) hide)
     )
-    (property "Assembly" "" (at 66.04 72.39 0)
+    (property "Assembly" "True" (at 66.04 72.39 0)
       (effects (font (size 1.27 1.27)) hide)
     )
-    (property "LCSC_PN" "" (at 66.04 72.39 0)
+    (property "LCSC_PN" "C25803" (at 66.04 72.39 0)
       (effects (font (size 1.27 1.27)) hide)
     )
-    (property "Price" "" (at 66.04 72.39 0)
+    (property "Price" "0.0009" (at 66.04 72.39 0)
       (effects (font (size 1.27 1.27)) hide)
     )

Commit message: seconds_major_wrapup
Parts:
- C46: LCSC_PN (none) -> C14663; Price (none) -> 0.0021
Changed lines of the file:
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@@
       (effects (font (size 1.27 1.27)) hide)
     )
-    (property "LCSC_PN" "" (at 36.83 72.39 0)
+    (property "LCSC_PN" "C14663" (at 36.83 72.39 0)
       (effects (font (size 1.27 1.27)) hide)
     )
-    (property "Price" "" (at 36.83 72.39 0)
+    (property "Price" "0.0021" (at 36.83 72.39 0)
       (effects (font (size 1.27 1.27)) hide)
     )
