File: transistor_clock/adjust.kicad_sch (KiCad schematic)
At the start: 17 parts, among them Q131 MMBT3906, Q136 MMBT3904, SW1 Fast, SW2 Slow

Commit message: seconds_minor_wrapup
Parts:
- C76, SW1, SW2: Assembly (none) -> False
- D148: renamed from D285; value D -> 1N4148W; Assembly (none) -> True; LCSC_PN (none) -> C81598; Price (none) -> 0.0061
- D58: renamed from D298; value D -> 1N4148W; Assembly (none) -> True; LCSC_PN (none) -> C81598; Price (none) -> 0.0061
- Q47: renamed from Q131; value MMBT3906 -> MMBT5401; Assembly (none) -> True; LCSC_PN (none) -> C8326; Price (none) -> 0.0137
- Q48: renamed from Q136; Assembly (none) -> True; LCSC_PN (none) -> C20526; Price (none) -> 0.0094
- R15: renamed from R110; Assembly (none) -> True; LCSC_PN (none) -> C25804; Price (none) -> 0.0008
- renumbered C4 to C21, C34 to C46, C4 to C77, R110 to R15, R275 to R157, R170 to R195, R55 to R97

Commit message: seconds_major_wrapup
Other:
- note added: "TODO fix cap/osc"
Changed lines of the file:
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@@
     (stroke (width 0) (type default))
+  )
+  (text "TODO fix cap/osc" (at 82.55 148.59 0)
+    (effects (font (size 1.27 1.27)) (justify left bottom))
   )
   (hierarchical_label "clk" (shape output) (at 166.37 129.54 0) (fields_autoplaced)

Commit message: seconds_major_wrapup
Parts:
- C46, C77: LCSC_PN (none) -> C14663; Price (none) -> 0.0021
Changed lines of the file:
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@@
       (effects (font (size 1.27 1.27)) hide)
     )
-    (property "LCSC_PN" "" (at 153.67 81.28 0)
-      (effects (font (size 1.27 1.27)) hide)
-    )
-    (property "Price" "" (at 153.67 81.28 0)
+    (property "LCSC_PN" "C14663" (at 153.67 81.28 0)
+      (effects (font (size 1.27 1.27)) hide)
+    )
+    (property "Price" "0.0021" (at 153.67 81.28 0)
       (effects (font (size 1.27 1.27)) hide)
     )
@@
       (effects (font (size 1.27 1.27)) hide)
     )
-    (property "LCSC_PN" "" (at 83.82 134.62 0)
-      (effects (font (size 1.27 1.27)) hide)
-    )
-    (property "Price" "" (at 83.82 134.62 0)
-      (effects (font (size 1.27 1.27)) hide)
-    )
+    (property "LCSC_PN" "C14663" (at 83.82 134.62 0)
+      (effects (font (size 1.27 1.27)) hide)
+    )
+    (property "Price" "0.0021" (at 83.82 134.62 0)
+      (effects (font (size 1.27 1.27)) hide)
+    )

Commit message: a
Parts:
- renumbered C46 to C13, C21 to C61, D148 to D258, D58 to D301, Q48 to Q130, Q47 to Q90, R195 to R169, R97 to R283, R157 to R283, R15 to R63

Commit message: added content
Parts:
- C21: renamed from C61; footprint Capacitor_SMD:C_0603_1608Metric -> Capacitor_SMD:C_0805_2012Metric
- C76: value 100u -> 10u; footprint (none) -> Capacitor_SMD:C_0805_2012Metric; Assembly False -> True; LCSC_PN (none) -> C15850; Price (none) -> 0.0105
- renumbered C13 to C46, D258 to D148, D301 to D58, Q90 to Q47, Q130 to Q48, R63 to R15, R283 to R157, R169 to R195, R283 to R97
