File: transistor_clock/segment.kicad_sch (KiCad schematic)
At the start: 4 parts, among them Q63 MMBT3904

Commit message: seconds_minor_wrapup
Parts:
- D135: renamed from D126; footprint LED_SMD:LED_0603_1608Metric -> footprints:LED_filament_38mm; Assembly (none) -> False; Price (none) -> 0.41
- Q42: renamed from Q63; Assembly (none) -> True; LCSC_PN (none) -> C20526; Price (none) -> 0.0094
- R212: renamed from R58; Assembly (none) -> True; LCSC_PN (none) -> C25803; Price (none) -> 0.0009
- R85: renamed from R59; Assembly (none) -> True; LCSC_PN (none) -> C22962; Price (none) -> 0.0009

Commit message: a
Parts:
- Q63: renamed from Q42; value MMBT3904 -> MMBT5551; LCSC_PN C20526 -> C2145; Price 0.0094 -> 0.0136
- R127: renamed from R85; value 220 -> 10k; LCSC_PN C22962 -> C25804; Price 0.0009 -> 0.0008
- renumbered D135 to D199, R212 to R58
Other:
- note added: "1800K 68V 30mA"
- note removed: "12V"
- note removed: "4.4V-8.4V 20mA-38mA 320mW"
- note removed: "5V-9V"
- note removed: "60mW-114mW"
- note removed: "92mW-22mW"
- note removed: "9V"

Commit message: added content
Parts:
- Q63: value MMBT5551 -> MMBT3904; LCSC_PN C2145 -> C20526; Price 0.0136 -> 0.0094

Commit message: added content
Parts:
- renumbered D199 to D135, Q63 to Q42, R58 to R212, R127 to R85
