File: transistor_clock/sync.kicad_sch (KiCad schematic)
At the start: 18 parts, among them Q109 MMBT3906, Q139 MMBT3906, Q89 MMBT3904

Commit message: seconds_minor_wrapup
Parts:
- C76: Assembly (none) -> False
- D142: renamed from D286; value D -> 1N4148W; Assembly (none) -> True; LCSC_PN (none) -> C81598; Price (none) -> 0.0061
- Q102: renamed from Q139; value MMBT3906 -> MMBT5401; Assembly (none) -> True; LCSC_PN (none) -> C8326; Price (none) -> 0.0137
- Q52: renamed from Q109; value MMBT3906 -> MMBT5401; Assembly (none) -> True; LCSC_PN (none) -> C8326; Price (none) -> 0.0137
- Q53: renamed from Q89; Assembly (none) -> True; LCSC_PN (none) -> C20526; Price (none) -> 0.0094
- R137: renamed from R229; Assembly (none) -> True; LCSC_PN (none) -> C25804; Price (none) -> 0.0008
- R195: renamed from R295; Assembly (none) -> True; LCSC_PN (none) -> C25803; Price (none) -> 0.0009
- renumbered C40 to C23, C64 to C48, R229 to R137, R295 to R195, R287 to R97

Commit message: seconds_major_wrapup
Parts:
- C33: renamed from C48; value 100n -> 10n
- R141: renamed from R97; value 22k -> 100k; Assembly (none) -> True; LCSC_PN (none) -> C25803; Price (none) -> 0.0009
- R23: renamed from R195; value 470 -> 1k; Assembly (none) -> True; LCSC_PN (none) -> C21190; Price (none) -> 0.0005
- R23: renamed from R195; value 2k2 -> 10k; Assembly (none) -> True; LCSC_PN (none) -> C25804; Price (none) -> 0.0008
- R83: renamed from R137; value 3k8 -> 10k; Assembly (none) -> True; LCSC_PN (none) -> C25804; Price (none) -> 0.0008
- R83: renamed from R137; value 47k -> 100k; Assembly (none) -> True; LCSC_PN (none) -> C25803; Price (none) -> 0.0009
- renumbered C23 to C56, D142 to D297, Q53 to Q124, Q52 to Q125, Q102 to Q69, R195 to R23, R137 to R83
Other:
- note added: "100n"
- note added: "22k"
- note added: "2k2"
- note added: "3k8"
- note added: "470"
- note added: "47k"
- note added: "New: Vh 12V, Vl 0V, vhyst 12.2V I=1.2mA Old: Vh 16.5V, Vl -7.9V, vhyst 24.5V I=3.9mA"

Commit message: seconds_major_wrapup
Parts:
- C46: LCSC_PN (none) -> C14663; Price (none) -> 0.0021
- C52: renamed from C33; LCSC_PN (none) -> C57112; Price (none) -> 0.0022
- renumbered C56 to C65, D297 to D306, Q69 to Q113, Q124 to Q142, Q125 to Q143, R23 to R113, R141 to R229, R83 to R299

Commit message: a
Parts:
- renumbered C52 to C22, C65 to C36, D306 to D265, Q113 to Q50, Q142 to Q78, Q143 to Q88, R229 to R103, R113 to R137, R299 to R169

Commit message: added content
Parts:
- C60: renamed from C22; footprint Capacitor_SMD:C_0603_1608Metric -> Capacitor_SMD:C_0805_2012Metric
- C76: value 100u -> 10u; footprint (none) -> Capacitor_SMD:C_0805_2012Metric; Assembly False -> True; LCSC_PN (none) -> C15850; Price (none) -> 0.0105
- C78: renamed from C36; footprint Capacitor_SMD:C_0603_1608Metric -> Capacitor_SMD:C_0805_2012Metric
- renumbered D265 to D253, D265 to D300, Q78 to Q127, Q50 to Q131, Q88 to Q69, R169 to R113, R103 to R271, R137 to R279

Commit message: added content
Parts:
- renumbered C60 to C67, C78 to C9, D300 to D266, D253 to D62, Q131 to Q145, Q69 to Q18, Q127 to Q19, R279 to R259, R271 to R299, R113 to R35

Commit message: added content
Parts:
- renumbered C46 to C33, D266 to D265, R35 to R299
Changed lines of the file:
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@@
   (symbol (lib_id "Device:R") (at 152.4 63.5 180) (unit 1)
     (in_bom yes) (on_board yes) (dnp no) (fields_autoplaced)
-    (property "Reference" "R35" (at 154.178 62.8563 0)
+    (property "Reference" "R299" (at 154.178 62.8563 0)
       (effects (font (size 1.27 1.27)) (justify right))
     )
@@
   (symbol (lib_id "Device:C") (at 153.67 87.63 180) (unit 1)
     (in_bom yes) (on_board yes) (dnp no) (fields_autoplaced)
-    (property "Reference" "C46" (at 156.591 86.9863 0)
+    (property "Reference" "C33" (at 156.591 86.9863 0)
       (effects (font (size 1.27 1.27)) (justify right))
     )
@@
   (symbol (lib_id "Device:R") (at 144.78 41.91 0) (mirror x) (unit 1)
     (in_bom yes) (on_board yes) (dnp no) (fields_autoplaced)
-    (property "Reference" "R35" (at 143.0021 41.2663 0)
+    (property "Reference" "R299" (at 143.0021 41.2663 0)
       (effects (font (size 1.27 1.27)) (justify right))
     )
@@
   (symbol (lib_id "power:GND") (at 152.4 67.31 0) (unit 1)
     (in_bom yes) (on_board yes) (dnp no) (fields_autoplaced)
-    (property "Reference" "#PWR039" (at 152.4 73.66 0)
+    (property "Reference" "#PWR0234" (at 152.4 73.66 0)
       (effects (font (size 1.27 1.27)) hide)
     )
@@
   (symbol (lib_id "Device:R") (at 134.62 48.26 90) (unit 1)
     (in_bom yes) (on_board yes) (dnp no) (fields_autoplaced)
-    (property "Reference" "R35" (at 134.62 44.2341 90)
+    (property "Reference" "R299" (at 134.62 44.2341 90)
       (effects (font (size 1.27 1.27)))
     )
@@
   (symbol (lib_id "Device:D") (at 118.11 64.77 90) (unit 1)
     (in_bom yes) (on_board yes) (dnp no) (fields_autoplaced)
-    (property "Reference" "D266" (at 120.142 64.1263 90)
+    (property "Reference" "D265" (at 120.142 64.1263 90)
       (effects (font (size 1.27 1.27)) (justify right))
     )

Commit message: added content
Parts:
- renumbered C9 to C22, C67 to C37, D265 to D132, D62 to D299, Q18 to Q129, Q19 to Q51, Q145 to Q81, R299 to R107, R299 to R165, R259 to R77
