File: transistor_clock/transistor_clock.kicad_sch (KiCad schematic)
At the start: 20 parts, among them J1 Conn_01x02, Q21 MMBT3904

Commit message: seconds_minor_wrapup
Parts:
- added D282 (x2): LED, footprints:LED_filament_38mm, symbol Device:LED
- added R20, R209 (x2): TBD, Resistor_SMD:R_0603_1608Metric, symbol Device:R
- C49: renamed from C7; Assembly (none) -> False
- J1, TP5: Assembly (none) -> False
- Q107: renamed from Q21; Assembly (none) -> True; LCSC_PN (none) -> C20526; Price (none) -> 0.0094
- R20: Assembly (none) -> True; LCSC_PN (none) -> C25804; Price (none) -> 0.0008
- TP1, TP10, TP11, TP12, TP13, TP14, TP2, TP3, TP4, TP6, TP7, TP8, TP9: footprint (none) -> footprints:RCSRCW_0C_testpoint_1206; Assembly (none) -> False
- renumbered R53 to R1
Connections:
- net GND: now also R209.2, R209.2
- net VCC: now also R20.1; no longer TP6.1
- new net Dot_H-M: D282.1 (K), R209.1
- new net Dot_M-S: D282.1 (K), R209.1
- new net VD: D282.2 (A), D282.2 (A), R20.2, TP6.1

Commit message: seconds_major_wrapup
Parts:
- R20: LCSC_PN C25804 -> (none); Price 0.0008 -> (none)
- R49: renamed from R209; LCSC_PN C22962 -> (none); Price 0.0009 -> (none)
- renumbered D282 to D121
Other:
- note added: "1.2mA"
- note added: "8.5ms ON"
- note added: "Dividers: Removed LEDs. New: 900µA Old: 10.5mA"
- note added: "TODO"
- moved on the sheet: D121, R49, TP1, TP10, TP11, TP12, TP13, TP14, TP2, TP3, TP4, TP5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

Commit message: seconds_major_wrapup
Parts:
- renumbered D121 to D282, R49 to R209
Other:
- sheet Div_By_2 renamed Div_By_5
- sheet Div_By_5: file DivByTwo.kicad_sch -> DivBy5.kicad_sch

Commit message: a
Parts:
- renumbered D282 to D121, R209 to R49

Commit message: added content
Parts:
- removed R20: TBD, Resistor_SMD:R_0603_1608Metric, symbol Device:R
- added D144 (x4): 1N4148W, Diode_SMD:D_SOD-123, symbol Device:D
- added SW2: Heures, footprints:SW_PUSH_6mm_2pins, symbol Switch:SW_Push
- added SW2: Minutes, footprints:SW_PUSH_6mm_2pins, symbol Switch:SW_Push
- C49: footprint (none) -> Capacitor_SMD:C_0805_2012Metric; Assembly False -> True; LCSC_PN (none) -> C15850; Price (none) -> 0.0105
- R209: renamed from R49; value TBD -> 10k; LCSC_PN (none) -> C25804; Price (none) -> 0.0008
- renumbered D121 to D282
Connections:
- net clk_1hr: now also D144.1 (K), D144.1 (K), D144.2 (A)
- net clk_1min: now also D144.2 (A)
- net clk_1s: now also SW2.1, SW2.1
- new net: D144.2 (A), SW2.2 (x2)
- new net Minutes/Clk_in: D144.1 (K), D144.1 (K)
Other:
- removed sheet Time adjust
- sheet PSU ports: added Vleds; removed none
- note added: "Value TBD"
- note removed: "1.2mA"
- note removed: "Dividers: Removed LEDs. New: 900µA Old: 10.5mA"
- note removed: "TODO: Vleds"
- moved on the sheet: C49, Q107, R1, R20

Commit message: added content
Parts:
- added H2, H3, H4: M4, MountingHole:MountingHole_4.3mm_M4, symbol Mechanical:MountingHole
- added JP1, JP2: VCC, Jumper:SolderJumper-2_P1.3mm_Open_RoundedPad1.0x1.5mm, symbol Jumper:Jumper_2_Open
- renumbered D282 to D121, D144 to D302, R209 to R49
Connections:
- net VCC: now also JP1.2 (B); no longer TP5.1
- net VD: now also JP2.1 (A); no longer TP6.1
- net clk_1hr: no longer D302.1 (K), D302.1 (K)
- new net Hours/Clk_in: D302.1 (K), D302.1 (K)
- new net PSU/12V_out: JP1.1 (A), TP5.1
- new net PSU/Vleds: JP2.2 (B), TP6.1
Other:
- moved on the sheet: C49, D144, D302, J1, Q107, R1, R20, SW2, TP1, TP10, TP11, TP12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

Commit message: added content
Parts:
- removed SW2: Heures, footprints:SW_PUSH_6mm_2pins, symbol Switch:SW_Push
- removed SW2: Minutes, footprints:SW_PUSH_6mm_2pins, symbol Switch:SW_Push
- added SW1: Heures, footprints:TL3330, symbol Switch:SW_DPST
- added SW2: Minutes, footprints:TL3330, symbol Switch:SW_DPST
- renumbered C49 to C2, D302 to D132, D144 to D141, D121 to D282, Q107 to Q11, R49 to R209
Connections:
- net GND: now also SW1.3, SW1.4, SW2.3, SW2.4
- net clk_1s: now also SW1.2, SW2.2
- net at D132.2 (A): now also SW2.1
- net at D132.2 (A): now also SW1.1

Commit message: added content
Parts:
- renumbered D282 to D121, D141 to D132, D132 to D298, R209 to R49
