File: transistor_clock/scr_stage.kicad_sch (KiCad schematic)
At the start: 8 parts, among them Q115 MMBT3904, Q55 MMBT3906

Commit message: seconds_minor_wrapup
Parts:
- D305: renamed from D144; value D -> 1N4148W; Assembly (none) -> True; LCSC_PN (none) -> C81598; Price (none) -> 0.0061
- Q133: renamed from Q55; value MMBT3906 -> MMBT5401; Assembly (none) -> True; LCSC_PN (none) -> C8326; Price (none) -> 0.0137
- Q68: renamed from Q115; Assembly (none) -> True; LCSC_PN (none) -> C20526; Price (none) -> 0.0094
- R276: renamed from R110; Assembly (none) -> True; LCSC_PN (none) -> C22787; Price (none) -> 0.001
- R277: renamed from R111; Assembly (none) -> True; LCSC_PN (none) -> C25804; Price (none) -> 0.0008
- R278: renamed from R112; Assembly (none) -> True; LCSC_PN (none) -> C22787; Price (none) -> 0.001
- R279: renamed from R113; Assembly (none) -> True; LCSC_PN (none) -> C25804; Price (none) -> 0.0008
- renumbered C35 to C86

Commit message: seconds_major_wrapup
Parts:
- C86: LCSC_PN (none) -> C57112; Price (none) -> 0.0022
Changed lines of the file:
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@@
       (effects (font (size 1.27 1.27)) hide)
     )
-    (property "LCSC_PN" "" (at 138.43 76.2 0)
+    (property "LCSC_PN" "C57112" (at 138.43 76.2 0)
       (effects (font (size 1.27 1.27)) hide)
     )
-    (property "Price" "" (at 138.43 76.2 0)
+    (property "Price" "0.0022" (at 138.43 76.2 0)
       (effects (font (size 1.27 1.27)) hide)
     )

Commit message: a
Parts:
- renumbered C86 to C52, D305 to D264, Q68 to Q134, Q133 to Q86, R276 to R172, R277 to R173, R278 to R174, R279 to R175

Commit message: added content
Parts:
- C93: renamed from C52; value 10n -> 1n; LCSC_PN C57112 -> C1588; Price 0.0022 -> 0.0027
- R304: renamed from R172; value 120 -> 2k2; LCSC_PN C22787 -> C4190; Price 0.001 -> 0.0009
- R306: renamed from R174; value 120 -> 2k2; LCSC_PN C22787 -> C4190; Price 0.001 -> 0.0009
- renumbered D264 to D312, Q86 to Q163, Q134 to Q84, R173 to R305, R175 to R307

Commit message: added content
Parts:
- renumbered C93 to C32, D312 to D139, Q163 to Q109, Q84 to Q112, R304 to R134, R305 to R135, R306 to R136, R307 to R137

Commit message: added content
Parts:
- renumbered Q112 to Q142, R134 to R148, R135 to R149, R136 to R150, R137 to R151
Changed lines of the file:
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@@
   (symbol (lib_id "Device:R") (at 137.16 91.44 90) (unit 1)
     (in_bom yes) (on_board yes) (dnp no) (fields_autoplaced)
-    (property "Reference" "R137" (at 137.16 87.4141 90)
+    (property "Reference" "R151" (at 137.16 87.4141 90)
       (effects (font (size 1.27 1.27)))
     )
@@
   (symbol (lib_id "Device:R") (at 120.65 71.12 0) (unit 1)
     (in_bom yes) (on_board yes) (dnp no) (fields_autoplaced)
-    (property "Reference" "R134" (at 122.428 70.4763 0)
+    (property "Reference" "R148" (at 122.428 70.4763 0)
       (effects (font (size 1.27 1.27)) (justify left))
     )
@@
   (symbol (lib_id "power:GND") (at 120.65 111.76 0) (unit 1)
     (in_bom yes) (on_board yes) (dnp no) (fields_autoplaced)
-    (property "Reference" "#PWR0163" (at 120.65 118.11 0)
+    (property "Reference" "#PWR0169" (at 120.65 118.11 0)
       (effects (font (size 1.27 1.27)) hide)
     )
@@
   (symbol (lib_id "Device:R") (at 120.65 100.33 0) (unit 1)
     (in_bom yes) (on_board yes) (dnp no) (fields_autoplaced)
-    (property "Reference" "R135" (at 122.428 99.6863 0)
+    (property "Reference" "R149" (at 122.428 99.6863 0)
       (effects (font (size 1.27 1.27)) (justify left))
     )
@@
   (symbol (lib_id "Transistor_BJT:MMBT3904") (at 125.73 96.52 0) (unit 1)
     (in_bom yes) (on_board yes) (dnp no) (fields_autoplaced)
-    (property "Reference" "Q112" (at 130.81 94.615 0)
+    (property "Reference" "Q142" (at 130.81 94.615 0)
       (effects (font (size 1.27 1.27)) (justify left))
     )
@@
   (symbol (lib_id "Device:R") (at 120.65 107.95 0) (unit 1)
     (in_bom yes) (on_board yes) (dnp no) (fields_autoplaced)
-    (property "Reference" "R136" (at 122.428 107.3063 0)
+    (property "Reference" "R150" (at 122.428 107.3063 0)
       (effects (font (size 1.27 1.27)) (justify left))
     )

Commit message: added content
Parts:
- renumbered C32 to C44, D139 to D264, Q109 to Q102, Q142 to Q11, R148 to R94, R149 to R95, R150 to R96, R151 to R97

Commit message: a
Parts:
- C44: Assembly (none) -> True
- Q11: value MMBT3904 -> MMBT5551; LCSC_PN C20526 -> C2145; Price 0.0094 -> 0.0136
Changed lines of the file:
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@@
       (effects (font (size 1.27 1.27)) (justify left))
     )
-    (property "Value" "MMBT3904" (at 130.81 96.52 0)
+    (property "Value" "MMBT5551" (at 130.81 96.52 0)
       (effects (font (size 1.27 1.27)) (justify left))
     )
@@
       (effects (font (size 1.27 1.27)) hide)
     )
-    (property "LCSC_PN" "C20526" (at 125.73 96.52 0)
+    (property "LCSC_PN" "C2145" (at 125.73 96.52 0)
       (effects (font (size 1.27 1.27)) hide)
     )
-    (property "Price" "0.0094" (at 125.73 96.52 0)
+    (property "Price" "0.0136" (at 125.73 96.52 0)
       (effects (font (size 1.27 1.27)) hide)
     )
@@
       (effects (font (size 1.27 1.27)) hide)
     )
-    (property "Assembly" "" (at 138.43 76.2 0)
+    (property "Assembly" "True" (at 138.43 76.2 0)
       (effects (font (size 1.27 1.27)) hide)
     )
