File: transistor_clock/6counter.kicad_sch (KiCad schematic)
At the start: 8 parts, among them Q11 MMBT3904

Commit message: seconds_minor_wrapup
Parts:
- C2, C76: Assembly (none) -> False
- D23: value D -> 1N4148W; Assembly (none) -> True; LCSC_PN (none) -> C81598; Price (none) -> 0.0061
- Q11: Assembly (none) -> True; LCSC_PN (none) -> C20526; Price (none) -> 0.0094
- R20: LCSC_PN (none) -> C21190; Price (none) -> 0.0005
Changed lines of the file:
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@@
   (symbol (lib_id "power:VCC") (at 33.02 67.31 0) (unit 1)
     (in_bom yes) (on_board yes) (dnp no) (fields_autoplaced)
-    (property "Reference" "#PWR052" (at 33.02 71.12 0)
+    (property "Reference" "#PWR022" (at 33.02 71.12 0)
       (effects (font (size 1.27 1.27)) hide)
     )
@@
       (effects (font (size 1.27 1.27)) hide)
     )
+    (property "Assembly" "" (at 66.04 72.39 0)
+      (effects (font (size 1.27 1.27)) hide)
+    )
+    (property "LCSC_PN" "" (at 66.04 72.39 0)
+      (effects (font (size 1.27 1.27)) hide)
+    )
+    (property "Price" "" (at 66.04 72.39 0)
+      (effects (font (size 1.27 1.27)) hide)
+    )
     (pin "1")
     (pin "2")
@@
       (effects (font (size 1.27 1.27)) hide)
     )
+    (property "Assembly" "False" (at 73.66 81.28 0)
+      (effects (font (size 1.27 1.27)) hide)
+    )
+    (property "LCSC_PN" "" (at 73.66 81.28 0)
+      (effects (font (size 1.27 1.27)) hide)
+    )
+    (property "Price" "" (at 73.66 81.28 0)
+      (effects (font (size 1.27 1.27)) hide)
+    )
     (pin "1")
     (pin "2")
@@
       (effects (font (size 1.27 1.27)) hide)
     )
+    (property "Assembly" "False" (at 27.94 71.12 0)
+      (effects (font (size 1.27 1.27)) hide)
+    )
+    (property "LCSC_PN" "" (at 27.94 71.12 0)
+      (effects (font (size 1.27 1.27)) hide)
+    )
+    (property "Price" "" (at 27.94 71.12 0)
+      (effects (font (size 1.27 1.27)) hide)
+    )
     (pin "1")
     (pin "2")
@@
       (effects (font (size 1.27 1.27)) hide)
     )
+    (property "Assembly" "" (at 39.37 97.79 0)
+      (effects (font (size 1.27 1.27)) hide)
+    )
+    (property "LCSC_PN" "" (at 39.37 97.79 0)
+      (effects (font (size 1.27 1.27)) hide)
+    )
+    (property "Price" "" (at 39.37 97.79 0)
+      (effects (font (size 1.27 1.27)) hide)
+    )
     (pin "1")
     (pin "2")
@@
       (effects (font (size 1.27 1.27)) hide)
     )
+    (property "Assembly" "" (at 46.99 97.79 0)
+      (effects (font (size 1.27 1.27)) hide)
+    )
+    (property "LCSC_PN" "C21190" (at 46.99 97.79 0)
+      (effects (font (size 1.27 1.27)) hide)
+    )
+    (property "Price" "0.0005" (at 46.99 97.79 0)
+      (effects (font (size 1.27 1.27)) hide)
+    )
     (pin "1")
     (pin "2")
@@
   (symbol (lib_id "power:GND") (at 38.1 74.93 0) (unit 1)
     (in_bom yes) (on_board yes) (dnp no) (fields_autoplaced)
-    (property "Reference" "#PWR050" (at 38.1 81.28 0)
+    (property "Reference" "#PWR09" (at 38.1 81.28 0)
       (effects (font (size 1.27 1.27)) hide)
     )
@@
   (symbol (lib_id "power:GND") (at 27.94 74.93 0) (unit 1)
     (in_bom yes) (on_board yes) (dnp no) (fields_autoplaced)
-    (property "Reference" "#PWR050" (at 27.94 81.28 0)
+    (property "Reference" "#PWR09" (at 27.94 81.28 0)
       (effects (font (size 1.27 1.27)) hide)
     )
@@
       (effects (font (size 1.27 1.27)) hide)
     )
+    (property "Assembly" "" (at 38.1 71.12 0)
+      (effects (font (size 1.27 1.27)) hide)
+    )
+    (property "LCSC_PN" "" (at 38.1 71.12 0)
+      (effects (font (size 1.27 1.27)) hide)
+    )
+    (property "Price" "" (at 38.1 71.12 0)
+      (effects (font (size 1.27 1.27)) hide)
+    )
     (pin "1")
     (pin "2")
@@
           (reference "C51") (unit 1)
         )
+        (path "/b32464e6-c3c7-41da-ac79-643e545075e2/e603d182-4df8-47af-be90-10669ba852bc"
+          (reference "C77") (unit 1)
+        )
         (path "/b32464e6-c3c7-41da-ac79-643e545075e2/f60bc725-791e-421e-aa65-9d00c6f8a7a8/e4b3f9d6-b335-4f04-8cec-00b858f4333b/22eae6c2-6c36-46b7-8a11-c7d457080034"
           (reference "C54") (unit 1)
         )
-        (path "/b32464e6-c3c7-41da-ac79-643e545075e2/e603d182-4df8-47af-be90-10669ba852bc"
-          (reference "C77") (unit 1)
-        )
-        (path "/b32464e6-c3c7-41da-ac79-643e545075e2/fc84256b-6a0b-4a66-8a9d-3464331d8c4b/cadfc701-a229-43d0-bd3d-a4fb656a51ec"
-          (reference "C1") (unit 1)
+        (path "/b32464e6-c3c7-41da-ac79-643e545075e2/369b0561-6154-45b1-b267-ff673911a7b5/f7326efb-cfc5-42e3-bc99-3d82c7965823"
+          (reference "C20") (unit 1)
+        )
+        (path "/b32464e6-c3c7-41da-ac79-643e545075e2/fc837116-7951-4754-b134-6b29a9ce0d20/f7326efb-cfc5-42e3-bc99-3d82c7965823"
+          (reference "C29") (unit 1)
+        )
+        (path "/b32464e6-c3c7-41da-ac79-643e545075e2/fc84256b-6a0b-4a66-8a9d-3464331d8c4b/cadfc701-a229-43d0-bd3d-a4fb656a51ec/28fcebf3-a860-4674-8b07-a85c9eaa7b85"
+          (reference "C2") (unit 1)
         )
         (path "/b32464e6-c3c7-41da-ac79-643e545075e2/7ea6f02c-98d6-4cc3-9d12-1d5708d2f4a9/cadfc701-a229-43d0-bd3d-a4fb656a51ec/28fcebf3-a860-4674-8b07-a85c9eaa7b85"
           (reference "C33") (unit 1)
         )
-        (path "/b32464e6-c3c7-41da-ac79-643e545075e2/fc84256b-6a0b-4a66-8a9d-3464331d8c4b/cadfc701-a229-43d0-bd3d-a4fb656a51ec/28fcebf3-a860-4674-8b07-a85c9eaa7b85"
-          (reference "C2") (unit 1)
-        )
         (path "/b32464e6-c3c7-41da-ac79-643e545075e2/f60bc725-791e-421e-aa65-9d00c6f8a7a8/b51d637d-960d-44ae-9d65-17e24c553fce/28fcebf3-a860-4674-8b07-a85c9eaa7b85"
           (reference "C46") (unit 1)
         )
-        (path "/b32464e6-c3c7-41da-ac79-643e545075e2/369b0561-6154-45b1-b267-ff673911a7b5/f7326efb-cfc5-42e3-bc99-3d82c7965823"
-          (reference "C20") (unit 1)
-        )
-        (path "/b32464e6-c3c7-41da-ac79-643e545075e2/fc837116-7951-4754-b134-6b29a9ce0d20/f7326efb-cfc5-42e3-bc99-3d82c7965823"
-          (reference "C29") (unit 1)
+        (path "/b32464e6-c3c7-41da-ac79-643e545075e2/fc84256b-6a0b-4a66-8a9d-3464331d8c4b/cadfc701-a229-43d0-bd3d-a4fb656a51ec"
+          (reference "C1") (unit 1)
         )
       )
@@
       (effects (font (size 1.27 1.27)) (justify left) hide)
     )
+    (property "Assembly" "True" (at 63.5 97.79 0)
+      (effects (font (size 1.27 1.27)) hide)
+    )
+    (property "LCSC_PN" "C20526" (at 63.5 97.79 0)
+      (effects (font (size 1.27 1.27)) hide)
+    )
+    (property "Price" "0.0094" (at 63.5 97.79 0)
+      (effects (font (size 1.27 1.27)) hide)
+    )
     (pin "1")
     (pin "2")
@@
       (effects (font (size 1.27 1.27)) (justify left))
     )
-    (property "Value" "D" (at 56.642 102.8773 90)
+    (property "Value" "1N4148W" (at 56.642 102.8773 90)
       (effects (font (size 1.27 1.27)) (justify left))
     )
@@
       (effects (font (size 1.27 1.27)) hide)
     )
+    (property "Assembly" "True" (at 54.61 101.6 0)
+      (effects (font (size 1.27 1.27)) hide)
+    )
+    (property "LCSC_PN" "C81598" (at 54.61 101.6 0)
+      (effects (font (size 1.27 1.27)) hide)
+    )
+    (property "Price" "0.0061" (at 54.61 101.6 0)
+      (effects (font (size 1.27 1.27)) hide)
+    )

Commit message: seconds_major_wrapup
Parts:
- R17: Assembly (none) -> True; LCSC_PN (none) -> C25803; Price (none) -> 0.0009
- R20: Assembly (none) -> True
Changed lines of the file:
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@@
       (effects (font (size 1.27 1.27)) hide)
     )
-    (property "Assembly" "" (at 66.04 72.39 0)
+    (property "Assembly" "True" (at 66.04 72.39 0)
       (effects (font (size 1.27 1.27)) hide)
     )
-    (property "LCSC_PN" "" (at 66.04 72.39 0)
+    (property "LCSC_PN" "C25803" (at 66.04 72.39 0)
       (effects (font (size 1.27 1.27)) hide)
     )
-    (property "Price" "" (at 66.04 72.39 0)
+    (property "Price" "0.0009" (at 66.04 72.39 0)
       (effects (font (size 1.27 1.27)) hide)
     )
@@
       (effects (font (size 1.27 1.27)) hide)
     )
-    (property "Assembly" "" (at 46.99 97.79 0)
+    (property "Assembly" "True" (at 46.99 97.79 0)
       (effects (font (size 1.27 1.27)) hide)
     )

Commit message: seconds_major_wrapup
Parts:
- C51: LCSC_PN (none) -> C14663; Price (none) -> 0.0021
Changed lines of the file:
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@@
       (effects (font (size 1.27 1.27)) hide)
     )
-    (property "LCSC_PN" "" (at 38.1 71.12 0)
+    (property "LCSC_PN" "C14663" (at 38.1 71.12 0)
       (effects (font (size 1.27 1.27)) hide)
     )
-    (property "Price" "" (at 38.1 71.12 0)
+    (property "Price" "0.0021" (at 38.1 71.12 0)
       (effects (font (size 1.27 1.27)) hide)
     )

Commit message: added content
Parts:
- C2: footprint (none) -> Capacitor_SMD:C_0805_2012Metric; Assembly False -> True; LCSC_PN (none) -> C15850; Price (none) -> 0.0105
- C2: value 220n -> 100n; LCSC_PN (none) -> C14663; Price (none) -> 0.0021
- C76: value 100u -> 10u; footprint (none) -> Capacitor_SMD:C_0805_2012Metric; Assembly False -> True; LCSC_PN (none) -> C15850; Price (none) -> 0.0105
- R17: value 270 -> 2k2; LCSC_PN C25803 -> C4190
- R20: value 1k -> 10k; LCSC_PN C21190 -> C25804; Price 0.0005 -> 0.0008
Other:
- moved on the sheet: C2, R20
Changed lines of the file:
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@@
     (stroke (width 0) (type default))
   )
-  (wire (pts (xy 54.61 97.79) (xy 50.8 97.79))
+  (wire (pts (xy 54.61 97.79) (xy 43.18 97.79))
     (stroke (width 0) (type default))
   )
@@
     (effects (font (size 1.27 1.27)) (justify right))
   )
-  (hierarchical_label "Clk_in" (shape input) (at 35.56 97.79 180) (fields_autoplaced)
+  (hierarchical_label "Clk_in" (shape input) (at 27.94 97.79 180) (fields_autoplaced)
     (effects (font (size 1.27 1.27)) (justify right))
   )
@@
           (reference "#PWR0114") (unit 1)
         )
-        (path "/b32464e6-c3c7-41da-ac79-643e545075e2/f60bc725-791e-421e-aa65-9d00c6f8a7a8/b51d637d-960d-44ae-9d65-17e24c553fce"
-          (reference "#PWR0133") (unit 1)
-        )
-        (path "/b32464e6-c3c7-41da-ac79-643e545075e2/f60bc725-791e-421e-aa65-9d00c6f8a7a8/e4b3f9d6-b335-4f04-8cec-00b858f4333b"
-          (reference "#PWR0164") (unit 1)
-        )
         (path "/b32464e6-c3c7-41da-ac79-643e545075e2"
           (reference "#PWR0191") (unit 1)
@@
       (effects (font (size 1.27 1.27)) (justify left))
     )
-    (property "Value" "270" (at 67.818 73.6673 0)
+    (property "Value" "2k2" (at 67.818 73.6673 0)
       (effects (font (size 1.27 1.27)) (justify left))
     )
@@
       (effects (font (size 1.27 1.27)) hide)
     )
-    (property "LCSC_PN" "C25803" (at 66.04 72.39 0)
+    (property "LCSC_PN" "C4190" (at 66.04 72.39 0)
       (effects (font (size 1.27 1.27)) hide)
     )
@@
       (effects (font (size 1.27 1.27)) (justify right))
     )
-    (property "Footprint" "" (at 72.6948 77.47 0)
+    (property "Footprint" "Capacitor_SMD:C_0805_2012Metric" (at 72.6948 77.47 0)
       (effects (font (size 1.27 1.27)) hide)
     )
@@
       (effects (font (size 1.27 1.27)) hide)
     )
-    (property "Assembly" "False" (at 73.66 81.28 0)
-      (effects (font (size 1.27 1.27)) hide)
-    )
-    (property "LCSC_PN" "" (at 73.66 81.28 0)
-      (effects (font (size 1.27 1.27)) hide)
-    )
-    (property "Price" "" (at 73.66 81.28 0)
+    (property "Assembly" "True" (at 73.66 81.28 0)
+      (effects (font (size 1.27 1.27)) hide)
+    )
+    (property "LCSC_PN" "C15850" (at 73.66 81.28 0)
+      (effects (font (size 1.27 1.27)) hide)
+    )
+    (property "Price" "0.0105" (at 73.66 81.28 0)
       (effects (font (size 1.27 1.27)) hide)
     )
@@
       (effects (font (size 1.27 1.27)) (justify left))
     )
-    (property "Value" "100u" (at 30.861 71.5083 0)
+    (property "Value" "10u" (at 30.861 71.5083 0)
       (effects (font (size 1.27 1.27)) (justify left))
     )
-    (property "Footprint" "" (at 28.9052 74.93 0)
+    (property "Footprint" "Capacitor_SMD:C_0805_2012Metric" (at 28.9052 74.93 0)
       (effects (font (size 1.27 1.27)) hide)
     )
@@
       (effects (font (size 1.27 1.27)) hide)
     )
-    (property "Assembly" "False" (at 27.94 71.12 0)
-      (effects (font (size 1.27 1.27)) hide)
-    )
-    (property "LCSC_PN" "" (at 27.94 71.12 0)
-      (effects (font (size 1.27 1.27)) hide)
-    )
-    (property "Price" "" (at 27.94 71.12 0)
+    (property "Assembly" "True" (at 27.94 71.12 0)
+      (effects (font (size 1.27 1.27)) hide)
+    )
+    (property "LCSC_PN" "C15850" (at 27.94 71.12 0)
+      (effects (font (size 1.27 1.27)) hide)
+    )
+    (property "Price" "0.0105" (at 27.94 71.12 0)
       (effects (font (size 1.27 1.27)) hide)
     )
@@
     )
   )
-  (symbol (lib_id "Device:C") (at 39.37 97.79 90) (unit 1)
-    (in_bom yes) (on_board yes) (dnp no) (fields_autoplaced)
-    (property "Reference" "C2" (at 39.37 92.6211 90)
-      (effects (font (size 1.27 1.27)))
-    )
-    (property "Value" "220n" (at 39.37 94.5421 90)
-      (effects (font (size 1.27 1.27)))
-    )
-    (property "Footprint" "Capacitor_SMD:C_0603_1608Metric" (at 43.18 96.8248 0)
-      (effects (font (size 1.27 1.27)) hide)
-    )
-    (property "Datasheet" "~" (at 39.37 97.79 0)
-      (effects (font (size 1.27 1.27)) hide)
-    )
-    (property "Assembly" "" (at 39.37 97.79 0)
-      (effects (font (size 1.27 1.27)) hide)
-    )
-    (property "LCSC_PN" "" (at 39.37 97.79 0)
-      (effects (font (size 1.27 1.27)) hide)
-    )
-    (property "Price" "" (at 39.37 97.79 0)
+  (symbol (lib_id "Device:C") (at 31.75 97.79 90) (unit 1)
+    (in_bom yes) (on_board yes) (dnp no) (fields_autoplaced)
+    (property "Reference" "C2" (at 31.75 92.6211 90)
+      (effects (font (size 1.27 1.27)))
+    )
+    (property "Value" "100n" (at 31.75 94.5421 90)
+      (effects (font (size 1.27 1.27)))
+    )
+    (property "Footprint" "Capacitor_SMD:C_0603_1608Metric" (at 35.56 96.8248 0)
+      (effects (font (size 1.27 1.27)) hide)
+    )
+    (property "Datasheet" "~" (at 31.75 97.79 0)
+      (effects (font (size 1.27 1.27)) hide)
+    )
+    (property "Assembly" "" (at 31.75 97.79 0)
+      (effects (font (size 1.27 1.27)) hide)
+    )
+    (property "LCSC_PN" "C14663" (at 31.75 97.79 0)
+      (effects (font (size 1.27 1.27)) hide)
+    )
+    (property "Price" "0.0021" (at 31.75 97.79 0)
       (effects (font (size 1.27 1.27)) hide)
     )
@@
     )
   )
-  (symbol (lib_id "Device:R") (at 46.99 97.79 90) (unit 1)
-    (in_bom yes) (on_board yes) (dnp no) (fields_autoplaced)
-    (property "Reference" "R20" (at 46.99 93.7641 90)
-      (effects (font (size 1.27 1.27)))
-    )
-    (property "Value" "1k" (at 46.99 95.6851 90)
-      (effects (font (size 1.27 1.27)))
-    )
-    (property "Footprint" "Resistor_SMD:R_0603_1608Metric" (at 46.99 99.568 90)
-      (effects (font (size 1.27 1.27)) hide)
-    )
-    (property "Datasheet" "~" (at 46.99 97.79 0)
-      (effects (font (size 1.27 1.27)) hide)
-    )
-    (property "Assembly" "True" (at 46.99 97.79 0)
-      (effects (font (size 1.27 1.27)) hide)
-    )
-    (property "LCSC_PN" "C21190" (at 46.99 97.79 0)
-      (effects (font (size 1.27 1.27)) hide)
-    )
-    (property "Price" "0.0005" (at 46.99 97.79 0)
+  (symbol (lib_id "Device:R") (at 39.37 97.79 90) (unit 1)
+    (in_bom yes) (on_board yes) (dnp no) (fields_autoplaced)
+    (property "Reference" "R20" (at 39.37 93.7641 90)
+      (effects (font (size 1.27 1.27)))
+    )
+    (property "Value" "10k" (at 39.37 95.6851 90)
+      (effects (font (size 1.27 1.27)))
+    )
+    (property "Footprint" "Resistor_SMD:R_0603_1608Metric" (at 39.37 99.568 90)
+      (effects (font (size 1.27 1.27)) hide)
+    )
+    (property "Datasheet" "~" (at 39.37 97.79 0)
+      (effects (font (size 1.27 1.27)) hide)
+    )
+    (property "Assembly" "True" (at 39.37 97.79 0)
+      (effects (font (size 1.27 1.27)) hide)
+    )
+    (property "LCSC_PN" "C25804" (at 39.37 97.79 0)
+      (effects (font (size 1.27 1.27)) hide)
+    )
+    (property "Price" "0.0008" (at 39.37 97.79 0)
       (effects (font (size 1.27 1.27)) hide)
     )
@@
           (reference "#PWR0112") (unit 1)
         )
-        (path "/b32464e6-c3c7-41da-ac79-643e545075e2/f60bc725-791e-421e-aa65-9d00c6f8a7a8/b51d637d-960d-44ae-9d65-17e24c553fce"
-          (reference "#PWR0131") (unit 1)
-        )
-        (path "/b32464e6-c3c7-41da-ac79-643e545075e2/f60bc725-791e-421e-aa65-9d00c6f8a7a8/e4b3f9d6-b335-4f04-8cec-00b858f4333b"
-          (reference "#PWR0162") (unit 1)
-        )
         (path "/b32464e6-c3c7-41da-ac79-643e545075e2"
           (reference "#PWR0181") (unit 1)
@@
           (reference "#PWR0112") (unit 1)
         )
-        (path "/b32464e6-c3c7-41da-ac79-643e545075e2/f60bc725-791e-421e-aa65-9d00c6f8a7a8/b51d637d-960d-44ae-9d65-17e24c553fce"
-          (reference "#PWR0131") (unit 1)
-        )
-        (path "/b32464e6-c3c7-41da-ac79-643e545075e2/f60bc725-791e-421e-aa65-9d00c6f8a7a8/e4b3f9d6-b335-4f04-8cec-00b858f4333b"
-          (reference "#PWR0162") (unit 1)
-        )
         (path "/b32464e6-c3c7-41da-ac79-643e545075e2"
           (reference "#PWR0181") (unit 1)
@@
     (instances
       (project "transistor_clock"
-        (path "/b32464e6-c3c7-41da-ac79-643e545075e2/f60bc725-791e-421e-aa65-9d00c6f8a7a8/e4b3f9d6-b335-4f04-8cec-00b858f4333b/96e6f7be-f6c4-492d-846f-fd0cf1759d6a"
-          (reference "C51") (unit 1)
-        )
         (path "/b32464e6-c3c7-41da-ac79-643e545075e2/e603d182-4df8-47af-be90-10669ba852bc"
           (reference "C77") (unit 1)
         )
-        (path "/b32464e6-c3c7-41da-ac79-643e545075e2/f60bc725-791e-421e-aa65-9d00c6f8a7a8/e4b3f9d6-b335-4f04-8cec-00b858f4333b/22eae6c2-6c36-46b7-8a11-c7d457080034"
-          (reference "C54") (unit 1)
-        )
         (path "/b32464e6-c3c7-41da-ac79-643e545075e2/369b0561-6154-45b1-b267-ff673911a7b5/f7326efb-cfc5-42e3-bc99-3d82c7965823"
           (reference "C20") (unit 1)
@@
           (reference "C33") (unit 1)
         )
-        (path "/b32464e6-c3c7-41da-ac79-643e545075e2/f60bc725-791e-421e-aa65-9d00c6f8a7a8/b51d637d-960d-44ae-9d65-17e24c553fce/28fcebf3-a860-4674-8b07-a85c9eaa7b85"
-          (reference "C46") (unit 1)
-        )
-        (path "/b32464e6-c3c7-41da-ac79-643e545075e2/fc84256b-6a0b-4a66-8a9d-3464331d8c4b/cadfc701-a229-43d0-bd3d-a4fb656a51ec"
+        (path "/b32464e6-c3c7-41da-ac79-643e545075e2/fc84256b-6a0b-4a66-8a9d-3464331d8c4b/cadfc701-a229-43d0-bd3d-a4fb656a51ec"

Commit message: added content
Parts:
- renumbered C51 to C77
Changed lines of the file:
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@@
   (symbol (lib_id "Device:C") (at 38.1 71.12 180) (unit 1)
     (in_bom yes) (on_board yes) (dnp no) (fields_autoplaced)
-    (property "Reference" "C51" (at 41.021 70.4763 0)
+    (property "Reference" "C77" (at 41.021 70.4763 0)
       (effects (font (size 1.27 1.27)) (justify right))
     )

Commit message: a
Parts:
- C2, C77: Assembly (none) -> True
- Q11: value MMBT3904 -> MMBT5551; LCSC_PN C20526 -> C2145; Price 0.0094 -> 0.0136
Changed lines of the file:
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@@
       (effects (font (size 1.27 1.27)) hide)
     )
-    (property "Assembly" "" (at 31.75 97.79 0)
+    (property "Assembly" "True" (at 31.75 97.79 0)
       (effects (font (size 1.27 1.27)) hide)
     )
@@
       (effects (font (size 1.27 1.27)) hide)
     )
-    (property "Assembly" "" (at 38.1 71.12 0)
+    (property "Assembly" "True" (at 38.1 71.12 0)
       (effects (font (size 1.27 1.27)) hide)
     )
@@
       (effects (font (size 1.27 1.27)) (justify left))
     )
-    (property "Value" "MMBT3904" (at 68.58 97.79 0)
+    (property "Value" "MMBT5551" (at 68.58 97.79 0)
       (effects (font (size 1.27 1.27)) (justify left))
     )
@@
       (effects (font (size 1.27 1.27)) hide)
     )
-    (property "LCSC_PN" "C20526" (at 63.5 97.79 0)
-      (effects (font (size 1.27 1.27)) hide)
-    )
-    (property "Price" "0.0094" (at 63.5 97.79 0)
-      (effects (font (size 1.27 1.27)) hide)
-    )
+    (property "LCSC_PN" "C2145" (at 63.5 97.79 0)
+      (effects (font (size 1.27 1.27)) hide)
+    )
+    (property "Price" "0.0136" (at 63.5 97.79 0)
+      (effects (font (size 1.27 1.27)) hide)
+    )

Commit message: a
Parts:
- renumbered C76 to C19, C77 to C20, C2 to C21, C2 to C22, D23 to D123, Q11 to Q26, R20 to R52, R17 to R53
