File: transistor_clock/DivBy5.kicad_sch (KiCad schematic)
At the start: 17 parts, among them Q105 MMBT5401, Q121 MMBT3904, Q9 MMBT5401

Commit message: seconds_major_wrapup
Parts:
- C77: LCSC_PN (none) -> C14663; Price (none) -> 0.0021
- renumbered Q121 to Q107, R244 to R213, R237 to R213, R247 to R213, R249 to R213, R248 to R252

Commit message: added content
Parts:
- C33: footprint (none) -> Capacitor_SMD:C_0805_2012Metric
- C76: value 100u -> 10u; footprint (none) -> Capacitor_SMD:C_0805_2012Metric; Assembly False -> True; LCSC_PN (none) -> C15850; Price (none) -> 0.0105
- R20, R252: LCSC_PN C21190 -> C4190; Price 0.0005 -> 0.0009

Commit message: added content
Parts:
- RV1: footprint (none) -> Potentiometer_THT:Potentiometer_Vishay_T73YP_Vertical
Changed lines of the file:
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@@
       (effects (font (size 1.27 1.27)) (justify right))
     )
-    (property "Footprint" "" (at 97.79 72.39 0)
+    (property "Footprint" "Potentiometer_THT:Potentiometer_Vishay_T73YP_Vertical" (at 97.79 72.39 0)
       (effects (font (size 1.27 1.27)) hide)
     )

Commit message: added content
Parts:
- renumbered Q107 to Q11, Q105 to Q75, R213 to R20
Changed lines of the file:
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@@
   (symbol (lib_id "Transistor_BJT:MMBT3906") (at 121.92 100.33 180) (unit 1)
     (in_bom yes) (on_board yes) (dnp no)
-    (property "Reference" "Q105" (at 116.84 102.235 0)
+    (property "Reference" "Q75" (at 116.84 102.235 0)
       (effects (font (size 1.27 1.27)) (justify left))
     )
@@
   (symbol (lib_id "Transistor_BJT:MMBT3906") (at 95.25 88.9 0) (mirror x) (unit 1)
     (in_bom yes) (on_board yes) (dnp no)
-    (property "Reference" "Q105" (at 100.33 90.805 0)
+    (property "Reference" "Q75" (at 100.33 90.805 0)
       (effects (font (size 1.27 1.27)) (justify left))
     )
@@
   (symbol (lib_id "Device:R") (at 107.95 95.25 90) (unit 1)
     (in_bom yes) (on_board yes) (dnp no) (fields_autoplaced)
-    (property "Reference" "R213" (at 107.95 91.2241 90)
+    (property "Reference" "R20" (at 107.95 91.2241 90)
       (effects (font (size 1.27 1.27)))
     )
@@
   (symbol (lib_id "Device:R") (at 142.24 93.98 0) (unit 1)
     (in_bom yes) (on_board yes) (dnp no) (fields_autoplaced)
-    (property "Reference" "R213" (at 144.018 93.3363 0)
+    (property "Reference" "R20" (at 144.018 93.3363 0)
       (effects (font (size 1.27 1.27)) (justify left))
     )
@@
   (symbol (lib_id "Device:R") (at 119.38 111.76 0) (unit 1)
     (in_bom yes) (on_board yes) (dnp no)
-    (property "Reference" "R213" (at 121.158 111.1163 0)
+    (property "Reference" "R20" (at 121.158 111.1163 0)
       (effects (font (size 1.27 1.27)) (justify left))
     )
@@
   (symbol (lib_id "Transistor_BJT:MMBT3904") (at 124.46 105.41 0) (unit 1)
     (in_bom yes) (on_board yes) (dnp no) (fields_autoplaced)
-    (property "Reference" "Q107" (at 129.54 103.505 0)
+    (property "Reference" "Q11" (at 129.54 103.505 0)
       (effects (font (size 1.27 1.27)) (justify left))
     )
@@
   (symbol (lib_id "Device:R") (at 142.24 86.36 0) (unit 1)
     (in_bom yes) (on_board yes) (dnp no) (fields_autoplaced)
-    (property "Reference" "R213" (at 144.018 85.7163 0)
-      (effects (font (size 1.27 1.27)) (justify left))
-    )
+    (property "Reference" "R20" (at 144.018 85.7163 0)
+      (effects (font (size 1.27 1.27)) (justify left))
+    )

Commit message: a
Parts:
- removed R20: 2k2, Resistor_SMD:R_0603_1608Metric, symbol Device:R
- added R20: DNP, Resistor_SMD:R_0603_1608Metric, symbol Device:R
- added R20: 2k2, Resistor_SMD:R_0603_1608Metric, symbol Device:R
- C33: Assembly (none) -> False
- C77: Assembly (none) -> True
- Q11: value MMBT3904 -> MMBT5551; LCSC_PN C20526 -> C2145; Price 0.0094 -> 0.0136
- RV1: Assembly False -> OK
Connections:
- net VCC: now also R20.2
- net at Q75.2 (E): now also R20.1
- net at RV1.3: now also R20.1, R20.2
Other:
- note added: "2k"
- note added: "3k9"

Commit message: a
Parts:
- renumbered C33 to C71, C76 to C72, C77 to C73, D22 to D293, Q75 to Q119, Q75 to Q120, Q11 to Q121, Q9 to Q122, R20 to R237, R20 to R243, R20 to R244, R20 to R247, R252 to R248, R20 to R249, R20 to R250, R20 to R251, R20 to R269, RV1 to RV2
