File: transistor_clock/DivByTen.kicad_sch (KiCad schematic)
At the start: 26 parts, among them Q21 MMBT3904, Q23 MMBT3904, Q65 MMBT3906

Commit message: seconds_minor_wrapup
Parts:
- C67, D291, RV1: Assembly (none) -> False
- D23: renamed from D39; value D -> 1N4148W; Assembly (none) -> True; LCSC_PN (none) -> C81598; Price (none) -> 0.0061
- D23: renamed from D22; value D -> 1N4148W; Assembly (none) -> True; LCSC_PN (none) -> C81598; Price (none) -> 0.0061
- Q107: renamed from Q23; Assembly (none) -> True; LCSC_PN (none) -> C20526; Price (none) -> 0.0094
- Q110: renamed from Q65; value MMBT3906 -> MMBT5401; Assembly (none) -> True; LCSC_PN (none) -> C8326; Price (none) -> 0.0137
- Q115: renamed from Q21; Assembly (none) -> True; LCSC_PN (none) -> C20526; Price (none) -> 0.0094
- R20: renamed from R45; Assembly (none) -> True; LCSC_PN (none) -> C25803; Price (none) -> 0.0009
- R20: renamed from R45; Assembly (none) -> True; LCSC_PN (none) -> C25804; Price (none) -> 0.0008
- R20: renamed from R45; LCSC_PN (none) -> C21190; Price (none) -> 0.0005
- R213: renamed from R20; Assembly (none) -> True; LCSC_PN (none) -> C25804; Price (none) -> 0.0008
- R213: renamed from R41; LCSC_PN (none) -> C21190; Price (none) -> 0.0005
- R230: renamed from R53; Assembly (none) -> True; LCSC_PN (none) -> C25803; Price (none) -> 0.0009
- R232: renamed from R41; Assembly (none) -> True; LCSC_PN (none) -> C25804; Price (none) -> 0.0008
- renumbered C29 to C33, C27 to C51, C53 to C54, R45 to R20, R20 to R213

Commit message: seconds_major_wrapup
Parts:
- removed D23: 1N4148W, Diode_SMD:D_SOD-123, symbol Device:D
- removed D291: LED, LED_SMD:LED_0603_1608Metric, symbol Device:LED
- removed R213: 1k, Resistor_SMD:R_0603_1608Metric, symbol Device:R
- C51: value 220n -> 100n
- C54: value 1.5u -> 1u
- R20: value 2k2 -> 10k; Assembly (none) -> True; LCSC_PN (none) -> C25804; Price (none) -> 0.0008
- R20: value 100 -> 2k2; Assembly (none) -> True; LCSC_PN (none) -> C21190; Price (none) -> 0.0005
- R20: value 10k -> 100k; LCSC_PN C25804 -> C25803; Price 0.0008 -> 0.0009
- R20: Assembly (none) -> True
- R213: value 330 -> 2k2; Assembly (none) -> True; LCSC_PN (none) -> C21190; Price (none) -> 0.0005
- RV1: value 100 -> 1k
Connections:
- net GND: no longer R20.2
- net at R20.1: now also R20.2
- net at Q107.3 (C), Q110.1 (B), R20.1: now also R20.2; no longer R20.2
Other:
- note added: "1.5u"
- note added: "2k 3k9"
- moved on the sheet: R20

Commit message: seconds_major_wrapup
Parts:
- C33, C51: LCSC_PN (none) -> C14663; Price (none) -> 0.0021
Changed lines of the file:
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@@
       (effects (font (size 1.27 1.27)) hide)
     )
-    (property "LCSC_PN" "" (at 114.3 101.6 0)
-      (effects (font (size 1.27 1.27)) hide)
-    )
-    (property "Price" "" (at 114.3 101.6 0)
+    (property "LCSC_PN" "C14663" (at 114.3 101.6 0)
+      (effects (font (size 1.27 1.27)) hide)
+    )
+    (property "Price" "0.0021" (at 114.3 101.6 0)
       (effects (font (size 1.27 1.27)) hide)
     )
@@
       (effects (font (size 1.27 1.27)) hide)
     )
-    (property "LCSC_PN" "" (at 105.41 71.12 0)
-      (effects (font (size 1.27 1.27)) hide)
-    )
-    (property "Price" "" (at 105.41 71.12 0)
-      (effects (font (size 1.27 1.27)) hide)
-    )
+    (property "LCSC_PN" "C14663" (at 105.41 71.12 0)
+      (effects (font (size 1.27 1.27)) hide)
+    )
+    (property "Price" "0.0021" (at 105.41 71.12 0)
+      (effects (font (size 1.27 1.27)) hide)
+    )

Commit message: added content
Parts:
- C54: footprint (none) -> Capacitor_SMD:C_0805_2012Metric
- C67: value 100u -> 10u; footprint (none) -> Capacitor_SMD:C_0805_2012Metric; Assembly False -> True; LCSC_PN (none) -> C15850; Price (none) -> 0.0105
- R20, R213: LCSC_PN C21190 -> C4190; Price 0.0005 -> 0.0009

Commit message: added content
Parts:
- RV1: footprint (none) -> Potentiometer_THT:Potentiometer_Vishay_T73YP_Vertical
Changed lines of the file:
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@@
       (effects (font (size 1.27 1.27)) (justify right))
     )
-    (property "Footprint" "" (at 139.7 54.61 0)
+    (property "Footprint" "Potentiometer_THT:Potentiometer_Vishay_T73YP_Vertical" (at 139.7 54.61 0)
       (effects (font (size 1.27 1.27)) hide)
     )

Commit message: added content
Parts:
- renumbered C54 to C33, C51 to C33, Q107 to Q11, Q110 to Q75, R213 to R20
Connections:
- net at Q75.2 (E): now also R20.2; no longer D23.1 (K)
- net at C33.2, Q75.3 (C): now also D23.2 (A); no longer R20.1
- new net: D23.1 (K), R20.1
Other:
- moved on the sheet: D23, R20
Changed lines of the file:
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@@
   (symbol (lib_id "Transistor_BJT:MMBT3906") (at 163.83 82.55 180) (unit 1)
     (in_bom yes) (on_board yes) (dnp no)
-    (property "Reference" "Q110" (at 158.75 84.455 0)
+    (property "Reference" "Q75" (at 158.75 84.455 0)
       (effects (font (size 1.27 1.27)) (justify left))
     )
@@
   (symbol (lib_id "Device:R") (at 97.79 71.12 90) (unit 1)
     (in_bom yes) (on_board yes) (dnp no) (fields_autoplaced)
-    (property "Reference" "R213" (at 97.79 67.0941 90)
+    (property "Reference" "R20" (at 97.79 67.0941 90)
       (effects (font (size 1.27 1.27)))
     )
@@
   (symbol (lib_id "Transistor_BJT:MMBT3906") (at 137.16 71.12 0) (mirror x) (unit 1)
     (in_bom yes) (on_board yes) (dnp no)
-    (property "Reference" "Q110" (at 142.24 73.025 0)
+    (property "Reference" "Q75" (at 142.24 73.025 0)
       (effects (font (size 1.27 1.27)) (justify left))
     )
@@
   (symbol (lib_id "Device:C") (at 139.7 82.55 180) (unit 1)
     (in_bom yes) (on_board yes) (dnp no) (fields_autoplaced)
-    (property "Reference" "C54" (at 142.621 81.9063 0)
+    (property "Reference" "C33" (at 142.621 81.9063 0)
       (effects (font (size 1.27 1.27)) (justify right))
     )
@@
   (symbol (lib_id "Transistor_BJT:MMBT3904") (at 166.37 87.63 0) (unit 1)
     (in_bom yes) (on_board yes) (dnp no) (fields_autoplaced)
-    (property "Reference" "Q107" (at 171.45 85.725 0)
+    (property "Reference" "Q11" (at 171.45 85.725 0)
       (effects (font (size 1.27 1.27)) (justify left))
     )
@@
   (symbol (lib_id "Device:R") (at 184.15 57.15 0) (unit 1)
     (in_bom yes) (on_board yes) (dnp no) (fields_autoplaced)
-    (property "Reference" "R213" (at 185.928 56.5063 0)
+    (property "Reference" "R20" (at 185.928 56.5063 0)
       (effects (font (size 1.27 1.27)) (justify left))
     )
@@
   (symbol (lib_id "Device:C") (at 105.41 71.12 90) (unit 1)
     (in_bom yes) (on_board yes) (dnp no) (fields_autoplaced)
-    (property "Reference" "C51" (at 105.41 65.9511 90)
+    (property "Reference" "C33" (at 105.41 65.9511 90)
       (effects (font (size 1.27 1.27)))
     )
@@
     )
   )
-  (symbol (lib_id "Device:D") (at 157.48 77.47 180) (unit 1)
-    (in_bom yes) (on_board yes) (dnp no) (fields_autoplaced)
-    (property "Reference" "D23" (at 157.48 73.1901 0)
-      (effects (font (size 1.27 1.27)))
-    )
-    (property "Value" "1N4148W" (at 157.48 75.1111 0)
-      (effects (font (size 1.27 1.27)))
-    )
-    (property "Footprint" "Diode_SMD:D_SOD-123" (at 157.48 77.47 0)
-      (effects (font (size 1.27 1.27)) hide)
-    )
-    (property "Datasheet" "~" (at 157.48 77.47 0)
-      (effects (font (size 1.27 1.27)) hide)
-    )
-    (property "Sim.Device" "D" (at 157.48 77.47 0)
-      (effects (font (size 1.27 1.27)) hide)
-    )
-    (property "Sim.Pins" "1=K 2=A" (at 157.48 77.47 0)
-      (effects (font (size 1.27 1.27)) hide)
-    )
-    (property "Assembly" "True" (at 157.48 77.47 0)
-      (effects (font (size 1.27 1.27)) hide)
-    )
-    (property "LCSC_PN" "C81598" (at 157.48 77.47 0)
-      (effects (font (size 1.27 1.27)) hide)
-    )
-    (property "Price" "0.0061" (at 157.48 77.47 0)
+  (symbol (lib_id "Device:D") (at 149.86 77.47 180) (unit 1)
+    (in_bom yes) (on_board yes) (dnp no) (fields_autoplaced)
+    (property "Reference" "D23" (at 149.86 73.1901 0)
+      (effects (font (size 1.27 1.27)))
+    )
+    (property "Value" "1N4148W" (at 149.86 75.1111 0)
+      (effects (font (size 1.27 1.27)))
+    )
+    (property "Footprint" "Diode_SMD:D_SOD-123" (at 149.86 77.47 0)
+      (effects (font (size 1.27 1.27)) hide)
+    )
+    (property "Datasheet" "~" (at 149.86 77.47 0)
+      (effects (font (size 1.27 1.27)) hide)
+    )
+    (property "Sim.Device" "D" (at 149.86 77.47 0)
+      (effects (font (size 1.27 1.27)) hide)
+    )
+    (property "Sim.Pins" "1=K 2=A" (at 149.86 77.47 0)
+      (effects (font (size 1.27 1.27)) hide)
+    )
+    (property "Assembly" "True" (at 149.86 77.47 0)
+      (effects (font (size 1.27 1.27)) hide)
+    )
+    (property "LCSC_PN" "C81598" (at 149.86 77.47 0)
+      (effects (font (size 1.27 1.27)) hide)
+    )
+    (property "Price" "0.0061" (at 149.86 77.47 0)
       (effects (font (size 1.27 1.27)) hide)
     )
@@
     )
   )
-  (symbol (lib_id "Device:R") (at 149.86 77.47 90) (unit 1)
-    (in_bom yes) (on_board yes) (dnp no) (fields_autoplaced)
-    (property "Reference" "R20" (at 149.86 73.4441 90)
-      (effects (font (size 1.27 1.27)))
-    )
-    (property "Value" "1k" (at 149.86 75.3651 90)
-      (effects (font (size 1.27 1.27)))
-    )
-    (property "Footprint" "Resistor_SMD:R_0603_1608Metric" (at 149.86 79.248 90)
-      (effects (font (size 1.27 1.27)) hide)
-    )
-    (property "Datasheet" "~" (at 149.86 77.47 0)
-      (effects (font (size 1.27 1.27)) hide)
-    )
-    (property "Assembly" "True" (at 149.86 77.47 0)
-      (effects (font (size 1.27 1.27)) hide)
-    )
-    (property "LCSC_PN" "C21190" (at 149.86 77.47 0)
-      (effects (font (size 1.27 1.27)) hide)
-    )
-    (property "Price" "0.0005" (at 149.86 77.47 0)
-      (effects (font (size 1.27 1.27)) hide)
-    )
+  (symbol (lib_id "Device:R") (at 157.48 77.47 90) (unit 1)
+    (in_bom yes) (on_board yes) (dnp no) (fields_autoplaced)
+    (property "Reference" "R20" (at 157.48 73.4441 90)
+      (effects (font (size 1.27 1.27)))
+    )
+    (property "Value" "1k" (at 157.48 75.3651 90)
+      (effects (font (size 1.27 1.27)))
+    )
+    (property "Footprint" "Resistor_SMD:R_0603_1608Metric" (at 157.48 79.248 90)
+      (effects (font (size 1.27 1.27)) hide)
+    )
+    (property "Datasheet" "~" (at 157.48 77.47 0)
+      (effects (font (size 1.27 1.27)) hide)
+    )
+    (property "Assembly" "True" (at 157.48 77.47 0)
+      (effects (font (size 1.27 1.27)) hide)
+    )
+    (property "LCSC_PN" "C21190" (at 157.48 77.47 0)
+      (effects (font (size 1.27 1.27)) hide)
+    )
+    (property "Price" "0.0005" (at 157.48 77.47 0)
+      (effects (font (size 1.27 1.27)) hide)
+    )

Commit message: a
Parts:
- added R20: DNP, Resistor_SMD:R_0603_1608Metric, symbol Device:R
- C33: Assembly (none) -> True
- C33: Assembly (none) -> False
- Q11, Q115: value MMBT3904 -> MMBT5551; LCSC_PN C20526 -> C2145; Price 0.0094 -> 0.0136
- R20: Assembly (none) -> OK
- RV1: Assembly False -> OK
Connections:
- net VCC: now also R20.2
- net at R20.2, RV1.3: now also R20.1
Other:
- note added: "2k"
- note added: "3k9"
- note removed: "2k 3k9"
- moved on the sheet: R20, RV1

Commit message: a
Parts:
- renumbered C33 to C68, C33 to C69, C33 to C70, D23 to D289, D23 to D290, Q75 to Q116, Q75 to Q117, Q11 to Q118, R20 to R231, R20 to R233, R20 to R234, R20 to R235, R20 to R236, R20 to R238, R20 to R239, R20 to R240, R20 to R241, R20 to R242, R20 to R267
