File: transistor_clock/hours.kicad_sch (KiCad schematic)
At the start: 0 parts

Commit message: added content
Parts:
- added C2 (x2), C51 (x2): 100n, Capacitor_SMD:C_0603_1608Metric, symbol Device:C
- added C2 (x2): 10u, Capacitor_SMD:C_0805_2012Metric, symbol Device:C
- added C76 (x2): 10u, Capacitor_SMD:C_0805_2012Metric, symbol Device:C_Polarized
- added D23 (x11): 1N4148W, Diode_SMD:D_SOD-123, symbol Device:D
- added Q11 (x5): MMBT3904, Package_TO_SOT_SMD:SOT-23, symbol Transistor_BJT:MMBT3904
- added Q52: MMBT5401, Package_TO_SOT_SMD:SOT-23, symbol Transistor_BJT:MMBT3906
- added R17 (x3): 2k2, Resistor_SMD:R_0603_1608Metric, symbol Device:R
- added R20 (x5): 100k, Resistor_SMD:R_0603_1608Metric, symbol Device:R
- added R20 (x7): 10k, Resistor_SMD:R_0603_1608Metric, symbol Device:R
- added TP14: 24_rst, footprints:RCSRCW_0C_testpoint_1206, symbol Connector:TestPoint
Connections:
- net Clk_in: now also C2.1
- net Vref: now also C2.2, C2.2
- new net: Q11.1 (B), R20.1, R20.1 (x2)
- new net: C2.2, R20.1 (x2)
- new net: D23.1 (K), Q11.1 (B), R20.2, R20.2 (x2)
- new net: D23.1 (K), D23.1 (K), D23.1 (K), D23.1 (K), D23.1 (K), D23.1 (K), D23.1 (K), D23.1 (K), D23.1 (K), Q11.3 (C), R17.2
- new net: Q11.2 (E), Q11.3 (C)
- new net: Q11.3 (C), R20.1
- new net: Q52.1 (B), R20.1, R20.2
- new net: Q52.3 (C), R20.2
- new net 24_rst: Q11.1 (B), R20.1, R20.2, TP14.1
- new net CLK: Q11.3 (C), R17.2
- new net GND: C2.1, C2.1, C51.1, C51.1, C76.2, C76.2, D23.2 (A), D23.2 (A), Q11.2 (E), Q11.2 (E), Q11.2 (E), Q11.2 (E), R20.1, R20.1, R20.1, R20.2, R20.2
- new net I1: D23.2 (A)
- new net I2: D23.2 (A)
- new net I3: D23.2 (A)
- new net I4: D23.2 (A)
- new net I5: D23.2 (A)
- new net I6: D23.2 (A)
- new net I7: D23.2 (A)
- new net I8: D23.2 (A)
- new net I9: D23.2 (A)
- new net O0: C2.1
- new net O4: R20.2
- new net Oh2: R20.2
- new net SCR_stage10/RST: Q11.3 (C), R17.2
- new net VCC: C51.2, C51.2, C76.1, C76.1, Q52.2 (E), R17.1, R17.1, R17.1, R20.2
- no-connect marks 1 -> 0
Other:
- removed sheet 10Decoder
- removed sheet 10counter
- removed sheet 2counter
- added sheet 10Decoder1 (10decoder.kicad_sch)
- added sheet SCR_stage0 (scr_stage.kicad_sch)
- added sheet SCR_stage1 (scr_stage.kicad_sch)
- added sheet SCR_stage10 (scr_stage.kicad_sch)
- added sheet SCR_stage11 (scr_stage.kicad_sch)
- added sheet SCR_stage12 (scr_stage.kicad_sch)
- added sheet SCR_stage2 (scr_stage.kicad_sch)
- added sheet SCR_stage3 (scr_stage.kicad_sch)
- added sheet SCR_stage4 (scr_stage.kicad_sch)
- added sheet SCR_stage5 (scr_stage.kicad_sch)
- added sheet SCR_stage6 (scr_stage.kicad_sch)
- added sheet SCR_stage7 (scr_stage.kicad_sch)
- added sheet SCR_stage8 (scr_stage.kicad_sch)
- added sheet SCR_stage9 (scr_stage.kicad_sch)
- note removed: "TODO floating out?"
- note removed: "TODO rst input on 25?"

Commit message: added content
Parts:
- renumbered Q52 to Q131
Changed lines of the file:
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@@
   (symbol (lib_id "Transistor_BJT:MMBT3906") (at 55.88 142.24 0) (mirror x) (unit 1)
     (in_bom yes) (on_board yes) (dnp no)
-    (property "Reference" "Q52" (at 46.99 144.129 0)
+    (property "Reference" "Q131" (at 46.99 144.129 0)
       (effects (font (size 1.27 1.27)) (justify left))
     )
@@
     (instances
       (project "transistor_clock"
-        (path "/b32464e6-c3c7-41da-ac79-643e545075e2/7ea6f02c-98d6-4cc3-9d12-1d5708d2f4a9/cadfc701-a229-43d0-bd3d-a4fb656a51ec/0211eb0b-97a3-455a-a4b9-49336bda2571"
-          (reference "Q52") (unit 1)
+        (path "/b32464e6-c3c7-41da-ac79-643e545075e2/369b0561-6154-45b1-b267-ff673911a7b5/f7326efb-cfc5-42e3-bc99-3d82c7965823/09ad6700-0804-43e5-8393-34ed739096ca"
+          (reference "Q131") (unit 1)
         )
         (path "/b32464e6-c3c7-41da-ac79-643e545075e2/7ea6f02c-98d6-4cc3-9d12-1d5708d2f4a9/cadfc701-a229-43d0-bd3d-a4fb656a51ec/96e64c28-7545-40f7-aaf3-a4fd012e71a7"
@@
           (reference "Q109") (unit 1)
         )
-        (path "/b32464e6-c3c7-41da-ac79-643e545075e2/369b0561-6154-45b1-b267-ff673911a7b5/f7326efb-cfc5-42e3-bc99-3d82c7965823/09ad6700-0804-43e5-8393-34ed739096ca"
-          (reference "Q131") (unit 1)
+        (path "/b32464e6-c3c7-41da-ac79-643e545075e2/7ea6f02c-98d6-4cc3-9d12-1d5708d2f4a9/cadfc701-a229-43d0-bd3d-a4fb656a51ec/0211eb0b-97a3-455a-a4b9-49336bda2571"
+          (reference "Q52") (unit 1)
         )
         (path "/b32464e6-c3c7-41da-ac79-643e545075e2/f60bc725-791e-421e-aa65-9d00c6f8a7a8/9f238b1c-7481-4532-b9f9-510fd94ba217"
@@
           (reference "Q60") (unit 1)
         )
-        (path "/b32464e6-c3c7-41da-ac79-643e545075e2/fc84256b-6a0b-4a66-8a9d-3464331d8c4b/cadfc701-a229-43d0-bd3d-a4fb656a51ec/97296d8c-1e14-436e-9883-ea2ff2d821d3"
-          (reference "Q102") (unit 1)
+        (path "/b32464e6-c3c7-41da-ac79-643e545075e2/7ea6f02c-98d6-4cc3-9d12-1d5708d2f4a9/cadfc701-a229-43d0-bd3d-a4fb656a51ec/cdd346a2-af99-4cba-a870-25a15852fcab"
+          (reference "Q55") (unit 1)
         )
         (path "/b32464e6-c3c7-41da-ac79-643e545075e2/fc84256b-6a0b-4a66-8a9d-3464331d8c4b/cadfc701-a229-43d0-bd3d-a4fb656a51ec/cdd346a2-af99-4cba-a870-25a15852fcab"
@@
           (reference "Q12") (unit 1)
         )
-        (path "/b32464e6-c3c7-41da-ac79-643e545075e2/7ea6f02c-98d6-4cc3-9d12-1d5708d2f4a9/cadfc701-a229-43d0-bd3d-a4fb656a51ec/97296d8c-1e14-436e-9883-ea2ff2d821d3"
-          (reference "Q107") (unit 1)
+        (path "/b32464e6-c3c7-41da-ac79-643e545075e2/f60bc725-791e-421e-aa65-9d00c6f8a7a8/43b0c10f-7b98-421f-9761-1540af516aeb"
+          (reference "Q40") (unit 1)
         )
         (path "/b32464e6-c3c7-41da-ac79-643e545075e2/fc837116-7951-4754-b134-6b29a9ce0d20/f7326efb-cfc5-42e3-bc99-3d82c7965823/96f657b6-18d3-41c6-a281-d64d12e655e8"
@@
           (reference "Q72") (unit 1)
         )
-        (path "/b32464e6-c3c7-41da-ac79-643e545075e2/7ea6f02c-98d6-4cc3-9d12-1d5708d2f4a9/cadfc701-a229-43d0-bd3d-a4fb656a51ec/cdd346a2-af99-4cba-a870-25a15852fcab"
-          (reference "Q55") (unit 1)
+        (path "/b32464e6-c3c7-41da-ac79-643e545075e2/fc84256b-6a0b-4a66-8a9d-3464331d8c4b/cadfc701-a229-43d0-bd3d-a4fb656a51ec/97296d8c-1e14-436e-9883-ea2ff2d821d3"
+          (reference "Q102") (unit 1)
         )
         (path "/b32464e6-c3c7-41da-ac79-643e545075e2/fc84256b-6a0b-4a66-8a9d-3464331d8c4b/cadfc701-a229-43d0-bd3d-a4fb656a51ec/7f89f7e8-4eb0-459f-8749-acca2517c0c8"
@@
           (reference "Q10") (unit 1)
         )
-        (path "/b32464e6-c3c7-41da-ac79-643e545075e2/f60bc725-791e-421e-aa65-9d00c6f8a7a8/43b0c10f-7b98-421f-9761-1540af516aeb"
-          (reference "Q40") (unit 1)
+        (path "/b32464e6-c3c7-41da-ac79-643e545075e2/7ea6f02c-98d6-4cc3-9d12-1d5708d2f4a9/cadfc701-a229-43d0-bd3d-a4fb656a51ec/97296d8c-1e14-436e-9883-ea2ff2d821d3"
+          (reference "Q107") (unit 1)
         )
         (path "/b32464e6-c3c7-41da-ac79-643e545075e2/fc84256b-6a0b-4a66-8a9d-3464331d8c4b/cadfc701-a229-43d0-bd3d-a4fb656a51ec/63d41fd4-396e-4dd9-89ff-b770c4e35023"

Commit message: added content
Parts:
- renumbered C51 to C77
Changed lines of the file:
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@@
   (symbol (lib_id "Device:C") (at 44.45 30.48 180) (unit 1)
     (in_bom yes) (on_board yes) (dnp no) (fields_autoplaced)
-    (property "Reference" "C51" (at 47.371 29.8363 0)
+    (property "Reference" "C77" (at 47.371 29.8363 0)
       (effects (font (size 1.27 1.27)) (justify right))
     )
@@
   (symbol (lib_id "Device:C") (at 119.38 120.65 180) (unit 1)
     (in_bom yes) (on_board yes) (dnp no) (fields_autoplaced)
-    (property "Reference" "C51" (at 122.301 120.0063 0)
+    (property "Reference" "C77" (at 122.301 120.0063 0)
       (effects (font (size 1.27 1.27)) (justify right))
     )

Commit message: added content
Parts:
- renumbered Q131 to Q74

Commit message: a
Parts:
- C2, C77: Assembly (none) -> True
- Q11: value MMBT3904 -> MMBT5551; LCSC_PN C20526 -> C2145; Price 0.0094 -> 0.0136
- TP14: Assembly False -> OK
- renumbered Q74 to Q131

Commit message: a
Parts:
- renumbered C76 to C27, C2 to C41, C77 to C42, C2 to C43, C2 to C56, C2 to C57, C76 to C58, C77 to C59, D23 to D262, D23 to D271, D23 to D272, D23 to D273, D23 to D274, D23 to D275, D23 to D276, D23 to D277, D23 to D278, D23 to D287, D23 to D292, Q11 to Q111, Q11 to Q158, Q11 to Q84, Q11 to Q97, Q131 to Q98, Q11 to Q99, R20 to R168, R17 to R169, R20 to R194, R20 to R195, R20 to R196, R17 to R197, R20 to R198, R20 to R199, R20 to R222, R20 to R223, R20 to R327, R20 to R328, R17 to R329, R20 to R330, R20 to R331, TP14 to TP15
