File: transistor_clock/10counter.kicad_sch (KiCad schematic)
At the start: 8 parts, among them Q21 MMBT3904

Commit message: seconds_minor_wrapup
Parts:
- C44: renamed from C7; Assembly (none) -> False
- C76: Assembly (none) -> False
- D23: value D -> 1N4148W; Assembly (none) -> True; LCSC_PN (none) -> C81598; Price (none) -> 0.0061
- Q64: renamed from Q21; Assembly (none) -> True; LCSC_PN (none) -> C20526; Price (none) -> 0.0094
- R128: renamed from R41; LCSC_PN (none) -> C21190; Price (none) -> 0.0005
- renumbered R82 to R19
Other:
- sheet SCR_stage10 renamed SCR_stage4
- removed sheet SCR_stage11
- removed sheet SCR_stage12
- removed sheet SCR_stage13
- removed sheet SCR_stage14
- added sheet SCR_stage1 (scr_stage.kicad_sch)
- added sheet SCR_stage2 (scr_stage.kicad_sch)
- added sheet SCR_stage3 (scr_stage.kicad_sch)
- added sheet SCR_stage5 (scr_stage.kicad_sch)

Commit message: seconds_major_wrapup
Parts:
- R128: Assembly (none) -> True
- R19: Assembly (none) -> True; LCSC_PN (none) -> C25803; Price (none) -> 0.0009
Changed lines of the file:
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@@
       (effects (font (size 1.27 1.27)) hide)
     )
-    (property "Assembly" "" (at 66.04 72.39 0)
-      (effects (font (size 1.27 1.27)) hide)
-    )
-    (property "LCSC_PN" "" (at 66.04 72.39 0)
-      (effects (font (size 1.27 1.27)) hide)
-    )
-    (property "Price" "" (at 66.04 72.39 0)
+    (property "Assembly" "True" (at 66.04 72.39 0)
+      (effects (font (size 1.27 1.27)) hide)
+    )
+    (property "LCSC_PN" "C25803" (at 66.04 72.39 0)
+      (effects (font (size 1.27 1.27)) hide)
+    )
+    (property "Price" "0.0009" (at 66.04 72.39 0)
       (effects (font (size 1.27 1.27)) hide)
     )
@@
       (effects (font (size 1.27 1.27)) hide)
     )
-    (property "Assembly" "" (at 46.99 97.79 0)
-      (effects (font (size 1.27 1.27)) hide)
-    )
+    (property "Assembly" "True" (at 46.99 97.79 0)
+      (effects (font (size 1.27 1.27)) hide)
+    )

Commit message: seconds_major_wrapup
Parts:
- C46: LCSC_PN (none) -> C14663; Price (none) -> 0.0021
Changed lines of the file:
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@@
       (effects (font (size 1.27 1.27)) hide)
     )
-    (property "LCSC_PN" "" (at 38.1 71.12 0)
+    (property "LCSC_PN" "C14663" (at 38.1 71.12 0)
       (effects (font (size 1.27 1.27)) hide)
     )
-    (property "Price" "" (at 38.1 71.12 0)
+    (property "Price" "0.0021" (at 38.1 71.12 0)
       (effects (font (size 1.27 1.27)) hide)
     )

Commit message: added content
Parts:
- C2: value 220n -> 100n; LCSC_PN (none) -> C14663; Price (none) -> 0.0021
- C44: footprint (none) -> Capacitor_SMD:C_0805_2012Metric; Assembly False -> True; LCSC_PN (none) -> C15850; Price (none) -> 0.0105
- C76: value 100u -> 10u; footprint (none) -> Capacitor_SMD:C_0805_2012Metric; Assembly False -> True; LCSC_PN (none) -> C15850; Price (none) -> 0.0105
- R128: value 1k -> 10k; LCSC_PN C21190 -> C25804; Price 0.0005 -> 0.0008
- R19: value 270 -> 2k2; LCSC_PN C25803 -> C4190

Commit message: added content
Parts:
- renumbered C46 to C2, C44 to C39, Q64 to Q59, R128 to R118
Changed lines of the file:
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@@
   (symbol (lib_id "Device:C") (at 73.66 81.28 180) (unit 1)
     (in_bom yes) (on_board yes) (dnp no) (fields_autoplaced)
-    (property "Reference" "C44" (at 76.581 80.6363 0)
+    (property "Reference" "C39" (at 76.581 80.6363 0)
       (effects (font (size 1.27 1.27)) (justify right))
     )
@@
   (symbol (lib_id "Transistor_BJT:MMBT3904") (at 63.5 97.79 0) (unit 1)
     (in_bom yes) (on_board yes) (dnp no) (fields_autoplaced)
-    (property "Reference" "Q64" (at 68.58 95.885 0)
+    (property "Reference" "Q59" (at 68.58 95.885 0)
       (effects (font (size 1.27 1.27)) (justify left))
     )
@@
   (symbol (lib_id "Device:C") (at 38.1 71.12 180) (unit 1)
     (in_bom yes) (on_board yes) (dnp no) (fields_autoplaced)
-    (property "Reference" "C46" (at 41.021 70.4763 0)
+    (property "Reference" "C2" (at 41.021 70.4763 0)
       (effects (font (size 1.27 1.27)) (justify right))
     )
@@
   (symbol (lib_id "Device:R") (at 46.99 97.79 90) (unit 1)
     (in_bom yes) (on_board yes) (dnp no) (fields_autoplaced)
-    (property "Reference" "R128" (at 46.99 93.7641 90)
-      (effects (font (size 1.27 1.27)))
-    )
+    (property "Reference" "R118" (at 46.99 93.7641 90)
+      (effects (font (size 1.27 1.27)))
+    )

Commit message: a
Parts:
- C2: Assembly (none) -> True
- Q59: value MMBT3904 -> MMBT5551; LCSC_PN C20526 -> C2145; Price 0.0094 -> 0.0136
Changed lines of the file:
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@@
       (effects (font (size 1.27 1.27)) hide)
     )
-    (property "Assembly" "" (at 39.37 97.79 0)
+    (property "Assembly" "True" (at 39.37 97.79 0)
       (effects (font (size 1.27 1.27)) hide)
     )
@@
       (effects (font (size 1.27 1.27)) (justify left))
     )
-    (property "Value" "MMBT3904" (at 68.58 97.79 0)
+    (property "Value" "MMBT5551" (at 68.58 97.79 0)
       (effects (font (size 1.27 1.27)) (justify left))
     )
@@
       (effects (font (size 1.27 1.27)) hide)
     )
-    (property "LCSC_PN" "C20526" (at 63.5 97.79 0)
-      (effects (font (size 1.27 1.27)) hide)
-    )
-    (property "Price" "0.0094" (at 63.5 97.79 0)
+    (property "LCSC_PN" "C2145" (at 63.5 97.79 0)
+      (effects (font (size 1.27 1.27)) hide)
+    )
+    (property "Price" "0.0136" (at 63.5 97.79 0)
       (effects (font (size 1.27 1.27)) hide)
     )
@@
       (effects (font (size 1.27 1.27)) hide)
     )
-    (property "Assembly" "" (at 38.1 71.12 0)
-      (effects (font (size 1.27 1.27)) hide)
-    )
+    (property "Assembly" "True" (at 38.1 71.12 0)
+      (effects (font (size 1.27 1.27)) hide)
+    )

Commit message: a
Parts:
- renumbered C76 to C4, C2 to C5, C2 to C6, D23 to D57

Commit message: a
Parts:
- renumbered C4 to C36, C5 to C37, C6 to C38, D57 to D147, R19 to R119
Changed lines of the file:
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@@
 		(dnp no)
 		(fields_autoplaced yes)
-		(property "Reference" "D57"
+		(property "Reference" "D147"
 			(at 56.642 100.9563 90)
 			(effects
@@
 		(dnp no)
 		(fields_autoplaced yes)
-		(property "Reference" "#PWR041"
+		(property "Reference" "#PWR0142"
 			(at 73.66 91.44 0)
 			(effects
@@
 		(dnp no)
 		(fields_autoplaced yes)
-		(property "Reference" "#PWR035"
+		(property "Reference" "#PWR0136"
 			(at 27.94 81.28 0)
 			(effects
@@
 		(dnp no)
 		(fields_autoplaced yes)
-		(property "Reference" "#PWR039"
+		(property "Reference" "#PWR0140"
 			(at 66.04 72.39 0)
 			(effects
@@
 		(dnp no)
 		(fields_autoplaced yes)
-		(property "Reference" "C6"
+		(property "Reference" "C38"
 			(at 39.37 92.6211 90)
 			(effects
@@
 		(dnp no)
 		(fields_autoplaced yes)
-		(property "Reference" "#PWR038"
+		(property "Reference" "#PWR0139"
 			(at 54.61 111.76 0)
 			(effects
@@
 		(dnp no)
 		(fields_autoplaced yes)
-		(property "Reference" "R19"
+		(property "Reference" "R119"
 			(at 67.818 71.7463 0)
 			(effects
@@
 		(dnp no)
 		(fields_autoplaced yes)
-		(property "Reference" "C4"
+		(property "Reference" "C36"
 			(at 30.861 69.5873 0)
 			(effects
@@
 		(dnp no)
 		(fields_autoplaced yes)
-		(property "Reference" "#PWR040"
+		(property "Reference" "#PWR0141"
 			(at 66.04 111.76 0)
 			(effects
@@
 		(dnp no)
 		(fields_autoplaced yes)
-		(property "Reference" "C5"
+		(property "Reference" "C37"
 			(at 41.021 70.4763 0)
 			(effects
@@
 		(dnp no)
 		(fields_autoplaced yes)
-		(property "Reference" "#PWR037"
+		(property "Reference" "#PWR0138"
 			(at 38.1 81.28 0)
 			(effects
@@
 		(dnp no)
 		(fields_autoplaced yes)
-		(property "Reference" "#PWR036"
+		(property "Reference" "#PWR0137"
 			(at 33.02 71.12 0)
 			(effects
