File: transistor_clock/10decoder.kicad_sch (KiCad schematic)
At the start: 49 parts

Commit message: seconds_minor_wrapup
Parts:
- D10: renamed from D62; value D -> 1N4148W; Assembly (none) -> True; LCSC_PN (none) -> C81598; Price (none) -> 0.0061
- D11: renamed from D63; value D -> 1N4148W; Assembly (none) -> True; LCSC_PN (none) -> C81598; Price (none) -> 0.0061
- D12: renamed from D69; value D -> 1N4148W; Assembly (none) -> True; LCSC_PN (none) -> C81598; Price (none) -> 0.0061
- D13: renamed from D71; value D -> 1N4148W; Assembly (none) -> True; LCSC_PN (none) -> C81598; Price (none) -> 0.0061
- D14: renamed from D75; value D -> 1N4148W; Assembly (none) -> True; LCSC_PN (none) -> C81598; Price (none) -> 0.0061
- D15: renamed from D78; value D -> 1N4148W; Assembly (none) -> True; LCSC_PN (none) -> C81598; Price (none) -> 0.0061
- D16: renamed from D79; value D -> 1N4148W; Assembly (none) -> True; LCSC_PN (none) -> C81598; Price (none) -> 0.0061
- D17: renamed from D80; value D -> 1N4148W; Assembly (none) -> True; LCSC_PN (none) -> C81598; Price (none) -> 0.0061
- D18: renamed from D81; value D -> 1N4148W; Assembly (none) -> True; LCSC_PN (none) -> C81598; Price (none) -> 0.0061
- D19: renamed from D82; value D -> 1N4148W; Assembly (none) -> True; LCSC_PN (none) -> C81598; Price (none) -> 0.0061
- D20: renamed from D83; value D -> 1N4148W; Assembly (none) -> True; LCSC_PN (none) -> C81598; Price (none) -> 0.0061
- D21: renamed from D84; value D -> 1N4148W; Assembly (none) -> True; LCSC_PN (none) -> C81598; Price (none) -> 0.0061
- D22: renamed from D85; value D -> 1N4148W; Assembly (none) -> True; LCSC_PN (none) -> C81598; Price (none) -> 0.0061
- D23: renamed from D86; value D -> 1N4148W; Assembly (none) -> True; LCSC_PN (none) -> C81598; Price (none) -> 0.0061
- D24: renamed from D87; value D -> 1N4148W; Assembly (none) -> True; LCSC_PN (none) -> C81598; Price (none) -> 0.0061
- D25: renamed from D88; value D -> 1N4148W; Assembly (none) -> True; LCSC_PN (none) -> C81598; Price (none) -> 0.0061
- D26: renamed from D89; value D -> 1N4148W; Assembly (none) -> True; LCSC_PN (none) -> C81598; Price (none) -> 0.0061
- D27: renamed from D90; value D -> 1N4148W; Assembly (none) -> True; LCSC_PN (none) -> C81598; Price (none) -> 0.0061
- D28: renamed from D91; value D -> 1N4148W; Assembly (none) -> True; LCSC_PN (none) -> C81598; Price (none) -> 0.0061
- D29: renamed from D92; value D -> 1N4148W; Assembly (none) -> True; LCSC_PN (none) -> C81598; Price (none) -> 0.0061
- D30: renamed from D93; value D -> 1N4148W; Assembly (none) -> True; LCSC_PN (none) -> C81598; Price (none) -> 0.0061
- D31: renamed from D94; value D -> 1N4148W; Assembly (none) -> True; LCSC_PN (none) -> C81598; Price (none) -> 0.0061
- D32: renamed from D95; value D -> 1N4148W; Assembly (none) -> True; LCSC_PN (none) -> C81598; Price (none) -> 0.0061
- D33: renamed from D96; value D -> 1N4148W; Assembly (none) -> True; LCSC_PN (none) -> C81598; Price (none) -> 0.0061
- D34: renamed from D97; value D -> 1N4148W; Assembly (none) -> True; LCSC_PN (none) -> C81598; Price (none) -> 0.0061
- D35: renamed from D98; value D -> 1N4148W; Assembly (none) -> True; LCSC_PN (none) -> C81598; Price (none) -> 0.0061
- D36: renamed from D99; value D -> 1N4148W; Assembly (none) -> True; LCSC_PN (none) -> C81598; Price (none) -> 0.0061
- D37: renamed from D100; value D -> 1N4148W; Assembly (none) -> True; LCSC_PN (none) -> C81598; Price (none) -> 0.0061
- D38: renamed from D101; value D -> 1N4148W; Assembly (none) -> True; LCSC_PN (none) -> C81598; Price (none) -> 0.0061
- D39: renamed from D102; value D -> 1N4148W; Assembly (none) -> True; LCSC_PN (none) -> C81598; Price (none) -> 0.0061
- D40: renamed from D103; value D -> 1N4148W; Assembly (none) -> True; LCSC_PN (none) -> C81598; Price (none) -> 0.0061
- D41: renamed from D104; value D -> 1N4148W; Assembly (none) -> True; LCSC_PN (none) -> C81598; Price (none) -> 0.0061
- D42: renamed from D105; value D -> 1N4148W; Assembly (none) -> True; LCSC_PN (none) -> C81598; Price (none) -> 0.0061
- D43: renamed from D106; value D -> 1N4148W; Assembly (none) -> True; LCSC_PN (none) -> C81598; Price (none) -> 0.0061
- D44: renamed from D107; value D -> 1N4148W; Assembly (none) -> True; LCSC_PN (none) -> C81598; Price (none) -> 0.0061
- D45: renamed from D108; value D -> 1N4148W; Assembly (none) -> True; LCSC_PN (none) -> C81598; Price (none) -> 0.0061
- D46: renamed from D109; value D -> 1N4148W; Assembly (none) -> True; LCSC_PN (none) -> C81598; Price (none) -> 0.0061
- D47: renamed from D110; value D -> 1N4148W; Assembly (none) -> True; LCSC_PN (none) -> C81598; Price (none) -> 0.0061
- D48: renamed from D111; value D -> 1N4148W; Assembly (none) -> True; LCSC_PN (none) -> C81598; Price (none) -> 0.0061
- D49: renamed from D112; value D -> 1N4148W; Assembly (none) -> True; LCSC_PN (none) -> C81598; Price (none) -> 0.0061
- D50: renamed from D113; value D -> 1N4148W; Assembly (none) -> True; LCSC_PN (none) -> C81598; Price (none) -> 0.0061
- D51: renamed from D114; value D -> 1N4148W; Assembly (none) -> True; LCSC_PN (none) -> C81598; Price (none) -> 0.0061
- D52: renamed from D115; value D -> 1N4148W; Assembly (none) -> True; LCSC_PN (none) -> C81598; Price (none) -> 0.0061
- D53: renamed from D116; value D -> 1N4148W; Assembly (none) -> True; LCSC_PN (none) -> C81598; Price (none) -> 0.0061
- D54: renamed from D117; value D -> 1N4148W; Assembly (none) -> True; LCSC_PN (none) -> C81598; Price (none) -> 0.0061
- D55: renamed from D118; value D -> 1N4148W; Assembly (none) -> True; LCSC_PN (none) -> C81598; Price (none) -> 0.0061
- D56: renamed from D119; value D -> 1N4148W; Assembly (none) -> True; LCSC_PN (none) -> C81598; Price (none) -> 0.0061
- D8: renamed from D58; value D -> 1N4148W; Assembly (none) -> True; LCSC_PN (none) -> C81598; Price (none) -> 0.0061
- D9: renamed from D59; value D -> 1N4148W; Assembly (none) -> True; LCSC_PN (none) -> C81598; Price (none) -> 0.0061

Commit message: a
Parts:
- renumbered D8 to D150, D9 to D151, D10 to D152, D11 to D153, D12 to D154, D13 to D155, D14 to D156, D15 to D157, D16 to D158, D17 to D159, D18 to D160, D19 to D161, D20 to D162, D21 to D163, D22 to D164, D23 to D165, D24 to D166, D25 to D167, D26 to D168, D27 to D169, D28 to D170, D29 to D171, D30 to D172, D31 to D173, D32 to D174, D33 to D175, D34 to D176, D35 to D177, D36 to D178, D37 to D179, D38 to D180, D39 to D181, D40 to D182, D41 to D183, D42 to D184, D43 to D185, D44 to D186, D45 to D187, D46 to D188, D47 to D189, D48 to D190, D49 to D191, D50 to D192, D51 to D193, D52 to D194, D53 to D195, D54 to D196, D55 to D197, D56 to D198
Changed lines of the file:
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@@
 		(on_board yes)
 		(dnp no)
-		(property "Reference" "D42"
+		(property "Reference" "D184"
 			(at 120.65 71.12 0)
 			(effects
@@
 		(on_board yes)
 		(dnp no)
-		(property "Reference" "D23"
+		(property "Reference" "D165"
 			(at 80.01 77.47 0)
 			(effects
@@
 		(on_board yes)
 		(dnp no)
-		(property "Reference" "D10"
+		(property "Reference" "D152"
 			(at 49.53 77.47 0)
 			(effects
@@
 		(on_board yes)
 		(dnp no)
-		(property "Reference" "D35"
+		(property "Reference" "D177"
 			(at 110.49 64.77 0)
 			(effects
@@
 		(on_board yes)
 		(dnp no)
-		(property "Reference" "D46"
+		(property "Reference" "D188"
 			(at 130.81 77.47 0)
 			(effects
@@
 		(on_board yes)
 		(dnp no)
-		(property "Reference" "D29"
+		(property "Reference" "D171"
 			(at 90.17 102.87 0)
 			(effects
@@
 		(on_board yes)
 		(dnp no)
-		(property "Reference" "D27"
+		(property "Reference" "D169"
 			(at 90.17 77.47 0)
 			(effects
@@
 		(on_board yes)
 		(dnp no)
-		(property "Reference" "D48"
+		(property "Reference" "D190"
 			(at 130.81 90.17 0)
 			(effects
@@
 		(on_board yes)
 		(dnp no)
-		(property "Reference" "D8"
+		(property "Reference" "D150"
 			(at 49.53 64.77 0)
 			(effects
@@
 		(on_board yes)
 		(dnp no)
-		(property "Reference" "D40"
+		(property "Reference" "D182"
 			(at 110.49 102.87 0)
 			(effects
@@
 		(on_board yes)
 		(dnp no)
-		(property "Reference" "D17"
+		(property "Reference" "D159"
 			(at 69.85 71.12 0)
 			(effects
@@
 		(on_board yes)
 		(dnp no)
-		(property "Reference" "D9"
+		(property "Reference" "D151"
 			(at 49.53 71.12 0)
 			(effects
@@
 		(on_board yes)
 		(dnp no)
-		(property "Reference" "D28"
+		(property "Reference" "D170"
 			(at 90.17 96.52 0)
 			(effects
@@
 		(on_board yes)
 		(dnp no)
-		(property "Reference" "D47"
+		(property "Reference" "D189"
 			(at 130.81 83.82 0)
 			(effects
@@
 		(on_board yes)
 		(dnp no)
-		(property "Reference" "D22"
+		(property "Reference" "D164"
 			(at 80.01 71.12 0)
 			(effects
@@
 		(on_board yes)
 		(dnp no)
-		(property "Reference" "D50"
+		(property "Reference" "D192"
 			(at 130.81 102.87 0)
 			(effects
@@
 		(on_board yes)
 		(dnp no)
-		(property "Reference" "D41"
+		(property "Reference" "D183"
 			(at 120.65 64.77 0)
 			(effects
@@
 		(on_board yes)
 		(dnp no)
-		(property "Reference" "D38"
+		(property "Reference" "D180"
 			(at 110.49 90.17 0)
 			(effects
@@
 		(on_board yes)
 		(dnp no)
-		(property "Reference" "D43"
+		(property "Reference" "D185"
 			(at 120.65 77.47 0)
 			(effects
@@
 		(on_board yes)
 		(dnp no)
-		(property "Reference" "D30"
+		(property "Reference" "D172"
 			(at 100.33 64.77 0)
 			(effects
@@
 		(on_board yes)
 		(dnp no)
-		(property "Reference" "D44"
+		(property "Reference" "D186"
 			(at 130.81 64.77 0)
 			(effects
@@
 		(on_board yes)
 		(dnp no)
-		(property "Reference" "D15"
+		(property "Reference" "D157"
 			(at 59.69 77.47 0)
 			(effects
@@
 		(on_board yes)
 		(dnp no)
-		(property "Reference" "D21"
+		(property "Reference" "D163"
 			(at 80.01 64.77 0)
 			(effects
@@
 		(on_board yes)
 		(dnp no)
-		(property "Reference" "D14"
+		(property "Reference" "D156"
 			(at 59.69 71.12 0)
 			(effects
@@
 		(on_board yes)
 		(dnp no)
-		(property "Reference" "D11"
+		(property "Reference" "D153"
 			(at 49.53 83.82 0)
 			(effects
@@
 		(on_board yes)
 		(dnp no)
-		(property "Reference" "D32"
+		(property "Reference" "D174"
 			(at 100.33 83.82 0)
 			(effects
@@
 		(on_board yes)
 		(dnp no)
-		(property "Reference" "D13"
+		(property "Reference" "D155"
 			(at 49.53 96.52 0)
 			(effects
@@
 		(on_board yes)
 		(dnp no)
-		(property "Reference" "D56"
+		(property "Reference" "D198"
 			(at 140.97 102.87 0)
 			(effects
@@
 		(on_board yes)
 		(dnp no)
-		(property "Reference" "D12"
+		(property "Reference" "D154"
 			(at 49.53 90.17 0)
 			(effects
@@
 		(on_board yes)
 		(dnp no)
-		(property "Reference" "D31"
+		(property "Reference" "D173"
 			(at 100.33 77.47 0)
 			(effects
@@
 		(on_board yes)
 		(dnp no)
-		(property "Reference" "D24"
+		(property "Reference" "D166"
 			(at 80.01 83.82 0)
 			(effects
@@
 		(on_board yes)
 		(dnp no)
-		(property "Reference" "D54"
+		(property "Reference" "D196"
 			(at 140.97 83.82 0)
 			(effects
@@
 		(on_board yes)
 		(dnp no)
-		(property "Reference" "D52"
+		(property "Reference" "D194"
 			(at 140.97 71.12 0)
 			(effects
@@
 		(on_board yes)
 		(dnp no)
-		(property "Reference" "D19"
+		(property "Reference" "D161"
 			(at 69.85 90.17 0)
 			(effects
@@
 		(on_board yes)
 		(dnp no)
-		(property "Reference" "D37"
+		(property "Reference" "D179"
 			(at 110.49 83.82 0)
 			(effects
@@
 		(on_board yes)
 		(dnp no)
-		(property "Reference" "D20"
+		(property "Reference" "D162"
 			(at 69.85 102.87 0)
 			(effects
@@
 		(on_board yes)
 		(dnp no)
-		(property "Reference" "D51"
+		(property "Reference" "D193"
 			(at 140.97 64.77 0)
 			(effects
@@
 		(on_board yes)
 		(dnp no)
-		(property "Reference" "D16"
+		(property "Reference" "D158"
 			(at 69.85 64.77 0)
 			(effects
@@
 		(on_board yes)
 		(dnp no)
-		(property "Reference" "D33"
+		(property "Reference" "D175"
 			(at 100.33 96.52 0)
 			(effects
@@
 		(on_board yes)
 		(dnp no)
-		(property "Reference" "D34"
+		(property "Reference" "D176"
 			(at 100.33 102.87 0)
 			(effects
@@
 		(on_board yes)
 		(dnp no)
-		(property "Reference" "D45"
+		(property "Reference" "D187"
 			(at 130.81 71.12 0)
 			(effects
@@
 		(on_board yes)
 		(dnp no)
-		(property "Reference" "D49"
+		(property "Reference" "D191"
 			(at 130.81 96.52 0)
 			(effects
@@
 		(on_board yes)
 		(dnp no)
-		(property "Reference" "D26"
+		(property "Reference" "D168"
 			(at 90.17 71.12 0)
 			(effects
@@
 		(on_board yes)
 		(dnp no)
-		(property "Reference" "D53"
+		(property "Reference" "D195"
 			(at 140.97 77.47 0)
 			(effects
@@
 		(on_board yes)
 		(dnp no)
-		(property "Reference" "D36"
+		(property "Reference" "D178"
 			(at 110.49 77.47 0)
 			(effects
@@
 		(on_board yes)
 		(dnp no)
-		(property "Reference" "D18"
+		(property "Reference" "D160"
 			(at 69.85 83.82 0)
 			(effects
@@
 		(on_board yes)
 		(dnp no)
-		(property "Reference" "D55"
+		(property "Reference" "D197"
 			(at 140.97 96.52 0)
 			(effects
@@
 		(on_board yes)
 		(dnp no)
-		(property "Reference" "D25"
+		(property "Reference" "D167"
 			(at 80.01 102.87 0)
 			(effects
@@
 		(on_board yes)
 		(dnp no)
-		(property "Reference" "D39"
+		(property "Reference" "D181"
 			(at 110.49 96.52 0)
 			(effects
