File: transistor_clock/6decoder.kicad_sch (KiCad schematic)
At the start: 27 parts

Commit message: seconds_minor_wrapup
Parts:
- D10, D11, D17, D18, D19, D20, D21, D26, D27, D28, D31, D32, D33, D34, D36, D37, D44, D45, D48, D53, D55, D64, D65, D66, D67, D8, D9: value D -> 1N4148W; Assembly (none) -> True; LCSC_PN (none) -> C81598; Price (none) -> 0.0061

Commit message: a
Parts:
- renumbered D8 to D65, D17 to D66, D26 to D67, D27 to D68, D44 to D69, D45 to D70, D18 to D71, D28 to D72, D10 to D73, D19 to D74, D31 to D75, D48 to D76, D64 to D77, D11 to D78, D20 to D79, D32 to D80, D33 to D81, D65 to D82, D21 to D83, D34 to D84, D53 to D85, D66 to D86, D9 to D87, D36 to D88, D37 to D89, D55 to D90, D67 to D91

Commit message: a
Parts:
- renumbered D73 to D100, D74 to D101, D75 to D102, D76 to D103, D77 to D104, D78 to D105, D79 to D106, D80 to D107, D81 to D108, D82 to D109, D83 to D110, D84 to D111, D85 to D112, D86 to D113, D87 to D114, D88 to D115, D89 to D116, D90 to D117, D91 to D118, D65 to D92, D66 to D93, D67 to D94, D68 to D95, D69 to D96, D70 to D97, D71 to D98, D72 to D99
Changed lines of the file:
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@@
 		(on_board yes)
 		(dnp no)
-		(property "Reference" "D68"
+		(property "Reference" "D95"
 			(at 49.53 83.82 0)
 			(effects
@@
 		(on_board yes)
 		(dnp no)
-		(property "Reference" "D73"
+		(property "Reference" "D100"
 			(at 69.85 64.77 0)
 			(effects
@@
 		(on_board yes)
 		(dnp no)
-		(property "Reference" "D83"
+		(property "Reference" "D110"
 			(at 90.17 71.12 0)
 			(effects
@@
 		(on_board yes)
 		(dnp no)
-		(property "Reference" "D72"
+		(property "Reference" "D99"
 			(at 59.69 77.47 0)
 			(effects
@@
 		(on_board yes)
 		(dnp no)
-		(property "Reference" "D79"
+		(property "Reference" "D106"
 			(at 80.01 71.12 0)
 			(effects
@@
 		(on_board yes)
 		(dnp no)
-		(property "Reference" "D87"
+		(property "Reference" "D114"
 			(at 100.33 64.77 0)
 			(effects
@@
 		(on_board yes)
 		(dnp no)
-		(property "Reference" "D80"
+		(property "Reference" "D107"
 			(at 80.01 77.47 0)
 			(effects
@@
 		(on_board yes)
 		(dnp no)
-		(property "Reference" "D69"
+		(property "Reference" "D96"
 			(at 49.53 90.17 0)
 			(effects
@@
 		(on_board yes)
 		(dnp no)
-		(property "Reference" "D76"
+		(property "Reference" "D103"
 			(at 69.85 90.17 0)
 			(effects
@@
 		(on_board yes)
 		(dnp no)
-		(property "Reference" "D86"
+		(property "Reference" "D113"
 			(at 90.17 102.87 0)
 			(effects
@@
 		(on_board yes)
 		(dnp no)
-		(property "Reference" "D90"
+		(property "Reference" "D117"
 			(at 100.33 96.52 0)
 			(effects
@@
 		(on_board yes)
 		(dnp no)
-		(property "Reference" "D84"
+		(property "Reference" "D111"
 			(at 90.17 77.47 0)
 			(effects
@@
 		(on_board yes)
 		(dnp no)
-		(property "Reference" "D70"
+		(property "Reference" "D97"
 			(at 49.53 96.52 0)
 			(effects
@@
 		(on_board yes)
 		(dnp no)
-		(property "Reference" "D65"
+		(property "Reference" "D92"
 			(at 49.53 64.77 0)
 			(effects
@@
 		(on_board yes)
 		(dnp no)
-		(property "Reference" "D85"
+		(property "Reference" "D112"
 			(at 90.17 96.52 0)
 			(effects
@@
 		(on_board yes)
 		(dnp no)
-		(property "Reference" "D78"
+		(property "Reference" "D105"
 			(at 80.01 64.77 0)
 			(effects
@@
 		(on_board yes)
 		(dnp no)
-		(property "Reference" "D89"
+		(property "Reference" "D116"
 			(at 100.33 83.82 0)
 			(effects
@@
 		(on_board yes)
 		(dnp no)
-		(property "Reference" "D81"
+		(property "Reference" "D108"
 			(at 80.01 83.82 0)
 			(effects
@@
 		(on_board yes)
 		(dnp no)
-		(property "Reference" "D66"
+		(property "Reference" "D93"
 			(at 49.53 71.12 0)
 			(effects
@@
 		(on_board yes)
 		(dnp no)
-		(property "Reference" "D71"
+		(property "Reference" "D98"
 			(at 59.69 71.12 0)
 			(effects
@@
 		(on_board yes)
 		(dnp no)
-		(property "Reference" "D67"
+		(property "Reference" "D94"
 			(at 49.53 77.47 0)
 			(effects
@@
 		(on_board yes)
 		(dnp no)
-		(property "Reference" "D82"
+		(property "Reference" "D109"
 			(at 80.01 102.87 0)
 			(effects
@@
 		(on_board yes)
 		(dnp no)
-		(property "Reference" "D91"
+		(property "Reference" "D118"
 			(at 100.33 102.87 0)
 			(effects
@@
 		(on_board yes)
 		(dnp no)
-		(property "Reference" "D77"
+		(property "Reference" "D104"
 			(at 69.85 102.87 0)
 			(effects
@@
 		(on_board yes)
 		(dnp no)
-		(property "Reference" "D75"
+		(property "Reference" "D102"
 			(at 69.85 83.82 0)
 			(effects
@@
 		(on_board yes)
 		(dnp no)
-		(property "Reference" "D88"
+		(property "Reference" "D115"
 			(at 100.33 77.47 0)
 			(effects
@@
 		(on_board yes)
 		(dnp no)
-		(property "Reference" "D74"
+		(property "Reference" "D101"
 			(at 69.85 71.12 0)
 			(effects
