File: 50W_LED_boost/led_boost/led_boost_MIC3230/led_boost_MIC3230.kicad_sch (KiCad schematic)
At the start: 49 parts, among them J1 PWR, J2 FAN, Q1 Q_NMOS_GDS, Q2 VN2210N3, U1 MIC3230YTSE, U2 TC648, U4 MCP1799x-500xxTT

Commit message: found sch issue
Other:
- note added: "Output caps return should be to GND, no LED- !"
Changed lines of the file:
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@@
+    (effects (font (size 1.27 1.27)) (justify left bottom))
+  )
+  (text "Output caps return should be to GND, no LED- !" (at 278.13 41.91 0)
     (effects (font (size 1.27 1.27)) (justify left bottom))
   )
