File: Planar_XFMR/Planar_XFMR.kicad_sch (KiCad schematic)
At the start: 18 parts, among them J1 A_Pri, J10 E_Sec, J11 F_Pri, J12 F_Sec, J13 G_Pri, J14 G_Sec, J15 H_Pri, J16 H_Sec, J17 I_Pri, J18 I_Sec, J2 A_Sec, J3 B_Pri, J4 B_Sec, J5 C_Pri, J6 C_Sec, J7 D_Pri, J8 D_Sec, J9 E_Pri

Commit message: a
Parts:
- J13: value G_Pri -> G_Sec
- J14: value G_Sec -> G_Pri
- J15: value H_Pri -> H_Sec
- J16: value H_Sec -> H_Pri
- J17: value I_Pri -> I_Sec
- J18: value I_Sec -> I_Pri
Connections:
- net at J13.1 (Pin_1), J13.2 (Pin_2): no longer J13.4 (Pin_4), J13.5 (Pin_5)
- net at J15.1 (Pin_1), J15.2 (Pin_2): now also J13.4 (Pin_4), J13.5 (Pin_5); no longer J15.4 (Pin_4), J15.5 (Pin_5)
- net at J4.1 (Pin_1), J4.2 (Pin_2): now also J2.4 (Pin_4), J2.5 (Pin_5); no longer J4.4 (Pin_4), J4.5 (Pin_5)
- net at J8.1 (Pin_1), J8.2 (Pin_2): no longer J8.4 (Pin_4), J8.5 (Pin_5)
- net at J3.1 (Pin_1), J3.2 (Pin_2): now also J1.4 (Pin_4), J1.5 (Pin_5); no longer J3.4 (Pin_4), J3.5 (Pin_5)
- net at J12.1 (Pin_1), J12.2 (Pin_2): now also J10.4 (Pin_4), J10.5 (Pin_5); no longer J12.4 (Pin_4), J12.5 (Pin_5)
- net at J17.1 (Pin_1), J17.2 (Pin_2): now also J15.4 (Pin_4), J15.5 (Pin_5); no longer J17.4 (Pin_4), J17.5 (Pin_5)
- net at J1.1 (Pin_1), J1.2 (Pin_2): no longer J1.4 (Pin_4), J1.5 (Pin_5)
- net at J2.1 (Pin_1), J2.2 (Pin_2): no longer J2.4 (Pin_4), J2.5 (Pin_5)
- net at J9.1 (Pin_1), J9.2 (Pin_2): now also J7.4 (Pin_4), J7.5 (Pin_5); no longer J9.4 (Pin_4), J9.5 (Pin_5)
- net at J7.1 (Pin_1), J7.2 (Pin_2): no longer J7.4 (Pin_4), J7.5 (Pin_5)
- net at J10.1 (Pin_1), J10.2 (Pin_2): now also J8.4 (Pin_4), J8.5 (Pin_5); no longer J10.4 (Pin_4), J10.5 (Pin_5)
- net at J16.1 (Pin_1), J16.2 (Pin_2): now also J14.4 (Pin_4), J14.5 (Pin_5); no longer J16.4 (Pin_4), J16.5 (Pin_5)
- net at J5.1 (Pin_1), J5.2 (Pin_2): now also J3.4 (Pin_4), J3.5 (Pin_5); no longer J5.4 (Pin_4), J5.5 (Pin_5)
- net at J6.1 (Pin_1), J6.2 (Pin_2): now also J4.4 (Pin_4), J4.5 (Pin_5); no longer J6.4 (Pin_4), J6.5 (Pin_5)
- net at J14.1 (Pin_1), J14.2 (Pin_2): no longer J14.4 (Pin_4), J14.5 (Pin_5)
- net at J11.1 (Pin_1), J11.2 (Pin_2): now also J9.4 (Pin_4), J9.5 (Pin_5); no longer J11.4 (Pin_4), J11.5 (Pin_5)
- net at J18.1 (Pin_1), J18.2 (Pin_2): now also J16.4 (Pin_4), J16.5 (Pin_5); no longer J18.4 (Pin_4), J18.5 (Pin_5)
- new net: J12.4 (Pin_4), J12.5 (Pin_5)
- new net: J17.4 (Pin_4), J17.5 (Pin_5)
- new net: J5.4 (Pin_4), J5.5 (Pin_5)
- new net: J6.4 (Pin_4), J6.5 (Pin_5)
- new net: J11.4 (Pin_4), J11.5 (Pin_5)
- new net: J18.4 (Pin_4), J18.5 (Pin_5)
