File: Planar_XFMR/Planar_XFMR.kicad_pcb (KiCad board)
At the start: 4 copper layers, 50 x 50 mm, 24 parts, among them J1 A_Pri, J10 E_Sec, J11 F_Pri, J12 F_Sec, J13 G_Sec, J14 G_Pri, J15 H_Sec, J16 H_Pri, J17 I_Sec, J18 I_Pri, J2 A_Sec, J3 B_Pri, J4 B_Sec, J5 C_Pri, J6 C_Sec, J7 D_Pri, J8 D_Sec, J9 E_Pri

Commit message: a
Parts:
- removed the REF** at (149.0, 56.6)
- removed the REF** at (149.0, 74.0)
- removed T**: 750320521_Wurth, footprints:750320521_Wurth
- added JP1: Jumper_2_Bridged, Jumper:SolderJumper-2_P1.3mm_Bridged_RoundedPad1.0x1.5mm, B.Cu at (140.5, 56.5)
- added JP2: Jumper_2_Bridged, Jumper:SolderJumper-2_P1.3mm_Bridged_RoundedPad1.0x1.5mm, B.Cu at (123.5, 73.0)
- added JP3: Jumper_2_Bridged, Jumper:SolderJumper-2_P1.3mm_Bridged_RoundedPad1.0x1.5mm, B.Cu at (140.5, 73.0)
- added JP4: Jumper_2_Bridged, Jumper:SolderJumper-2_P1.3mm_Bridged_RoundedPad1.0x1.5mm, B.Cu at (123.5, 56.5)
- added REF**: Planar_ER9.5-5, Planar:Planar_ER9.5-5, F.Cu at (148.8, 73.5)
- added REF**: Planar_ER9.5-5, Planar:Planar_ER9.5-5, F.Cu at (132.2, 39.9)
- added REF**: Planar_ER9.5-5, Planar:Planar_ER9.5-5, F.Cu at (149.0, 39.9)
- added REF**: Planar_ER11-5, Planar:Planar_ER11-5, F.Cu at (149.0, 56.6)
- added REF**: Planar_ER9.5-5, Planar:Planar_ER9.5-5, F.Cu at (115.2, 39.9)
- added REF**: Planar_ER11-5, Planar:Planar_ER11-5, F.Cu at (114.9, 56.6)
Connections:
- J11 pad 4: Net-(J11-Pin_4) -> Net-(J11-Pin_1)
- J11 pad 5: Net-(J11-Pin_4) -> Net-(J11-Pin_1)
- J12 pad 4: Net-(J12-Pin_4) -> Net-(J10-Pin_4)
- J12 pad 5: Net-(J12-Pin_4) -> Net-(J10-Pin_4)
- J2 pad 1: Net-(J2-Pin_1) -> Net-(J1-Pin_1)
- J2 pad 2: Net-(J2-Pin_1) -> Net-(J1-Pin_1)
- J2 pad 4: Net-(J2-Pin_4) -> Net-(J1-Pin_4)
- J2 pad 5: Net-(J2-Pin_4) -> Net-(J1-Pin_4)
- J4 pad 1: Net-(J2-Pin_4) -> Net-(J1-Pin_4)
- J4 pad 2: Net-(J2-Pin_4) -> Net-(J1-Pin_4)
- J4 pad 4: Net-(J4-Pin_4) -> Net-(J3-Pin_4)
- J4 pad 5: Net-(J4-Pin_4) -> Net-(J3-Pin_4)
- J6 pad 1: Net-(J4-Pin_4) -> Net-(J3-Pin_4)
- J6 pad 2: Net-(J4-Pin_4) -> Net-(J3-Pin_4)
- J6 pad 4: Net-(J6-Pin_4) -> Net-(J5-Pin_4)
- J6 pad 5: Net-(J6-Pin_4) -> Net-(J5-Pin_4)
- J7 pad 1: Net-(J7-Pin_1) -> Net-(J11-Pin_1)
- J7 pad 2: Net-(J7-Pin_1) -> Net-(J11-Pin_1)
- J7 pad 4: Net-(J7-Pin_4) -> Net-(J11-Pin_1)
- J7 pad 5: Net-(J7-Pin_4) -> Net-(J11-Pin_1)
- J8 pad 1: Net-(J8-Pin_1) -> Net-(J10-Pin_1)
- J8 pad 2: Net-(J8-Pin_1) -> Net-(J10-Pin_1)
- J9 pad 1: Net-(J7-Pin_4) -> Net-(J11-Pin_1)
- J9 pad 2: Net-(J7-Pin_4) -> Net-(J11-Pin_1)
Routing:
- net Net-(J11-Pin_1): track 23.8 -> 856.6 mm, vias 0 -> 3
- net Net-(J1-Pin_4): track 6.84 -> 495.3 mm, vias 0 -> 2
- net Net-(J1-Pin_1): track 0.00 -> 270.8 mm, vias 0 -> 1
- net Net-(J3-Pin_4): track 6.84 -> 270.6 mm, vias 0 -> 2
- net Net-(J17-Pin_4): track 9.51 -> 134.7 mm
- net Net-(J14-Pin_1): track 8.88 -> 96.2 mm
- net Net-(J5-Pin_4): track 0.00 -> 45.5 mm, vias 0 -> 1
- net Net-(J10-Pin_1): track 15.2 -> 39.8 mm, vias 0 -> 1
- net Net-(J10-Pin_4): track 23.7 -> 40.3 mm
- net Net-(J7-Pin_4): track 15.1 -> 0.00 mm
- net Net-(J12-Pin_4): track 8.51 -> 0.00 mm
- net Net-(J11-Pin_4): track 8.39 -> 0.00 mm
- net Net-(J16-Pin_4): track 25.1 -> 33.1 mm
- net Net-(J13-Pin_4): track 25.0 -> 32.2 mm
- net Net-(J4-Pin_4): track 6.84 -> 0.00 mm
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Other:
- outline, holes or cut-outs redrawn
- board text added: "10T 0.2 L1L2"
- board text added: "16T 0.1 L1L3"
- board text added: "2T 1.3 L1L2"
- board text added: "2T 1.3 L3L4"
- board text added: "8T 0.25 INT"
- board text added: "8T 0.25 L3L4"
- board text added: "ELP 22/6/16 N87 1520nH/turns²"
- board text added: "JLCJLCJLCJLC"
- board text added: "L2L4 0.4 6T"
- board text added: "Planar XFMR coupon X.B. 05/24 rev A"
- board text removed: "SUMIDA"

Commit message: a
Routing:
- net Net-(J17-Pin_4): track 134.7 -> 9.51 mm
- net Net-(J14-Pin_1): track 96.2 -> 8.88 mm
- net Net-(J5-Pin_4): track 45.5 -> 54.5 mm
- net Net-(J3-Pin_4): track 270.6 -> 279.7 mm
- net Net-(J14-Pin_4): track 25.3 -> 33.1 mm
- net Net-(J15-Pin_4): track 24.8 -> 32.2 mm
