File: hall_sensor_matrix/hall_sensor_matrix_v2/hall_sensor_matrix_v2.kicad_sch (KiCad schematic)
At the start: 28 parts, among them J1 CTRL, J2 COL, J3 ROW, U1 74LS595, U2 74LS597, U3 74LS597

Commit message: added v2
Parts:
- added D10, D11, D12, D13, D14, D15, D16, D17, D18, D19, D20, D21, D22, D23, D24, D9: LED, LED_SMD:LED_0603_1608Metric_Pad1.05x0.95mm_HandSolder, symbol Device:LED
- added R33, R34, R35, R36, R37, R38, R39, R40, R41, R42, R43, R44, R45, R46, R47, R48: 470, Resistor_SMD:R_0805_2012Metric, symbol Device:R
Connections:
- net +5V: now also J1.2 (Pin_2), R33.1, R34.1, R35.1, R36.1, R37.1, R38.1, R39.1, R40.1, R41.1, R42.1, R43.1, R44.1, R45.1, R46.1, R47.1, R48.1; no longer J1.5 (Pin_5)
- net CLK: now also J1.5 (Pin_5); no longer J1.4 (Pin_4)
- net Din: now also J1.3 (Pin_3); no longer J1.2 (Pin_2)
- net Dout: now also J1.6 (Pin_6); no longer J1.1 (Pin_1)
- net GND: now also J1.1 (Pin_1); no longer J1.6 (Pin_6)
- net Latch: now also J1.4 (Pin_4); no longer J1.3 (Pin_3)
- net R0: now also D9.1 (K)
- net R1: now also D10.1 (K)
- net R10: now also D19.1 (K)
- net R11: now also D20.1 (K)
- net R12: now also D21.1 (K)
- net R13: now also D22.1 (K)
- net R14: now also D23.1 (K)
- net R15: now also D24.1 (K)
- net R2: now also D11.1 (K)
- net R3: now also D12.1 (K)
- net R4: now also D13.1 (K)
- net R5: now also D14.1 (K)
- net R6: now also D15.1 (K)
- net R7: now also D16.1 (K)
- net R8: now also D17.1 (K)
- net R9: now also D18.1 (K)
- new net: D24.2 (A), R48.2
- new net: D22.2 (A), R46.2
- new net: D17.2 (A), R41.2
- new net: D11.2 (A), R35.2
- new net: D10.2 (A), R34.2
- new net: D19.2 (A), R43.2
- new net: D12.2 (A), R36.2
- new net: D18.2 (A), R42.2
- new net: D16.2 (A), R40.2
- new net: D14.2 (A), R38.2
- new net: D9.2 (A), R33.2
- new net: D13.2 (A), R37.2
- new net: D23.2 (A), R47.2
- new net: D20.2 (A), R44.2
- new net: D21.2 (A), R45.2
- new net: D15.2 (A), R39.2

Commit message: added content
Parts:
- added H1, H2: MountingHole, MountingHole:MountingHole_3.2mm_M3, symbol Mechanical:MountingHole
Changed lines of the file:
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@@
+    )
+  )
+  (symbol (lib_id "Mechanical:MountingHole") (at 228.6 147.32 0) (unit 1)
+    (in_bom yes) (on_board yes) (dnp no) (fields_autoplaced)
+    (property "Reference" "H2" (at 231.14 146.6763 0)
+      (effects (font (size 1.27 1.27)) (justify left))
+    )
+    (property "Value" "MountingHole" (at 231.14 148.5973 0)
+      (effects (font (size 1.27 1.27)) (justify left))
+    )
+    (property "Footprint" "MountingHole:MountingHole_3.2mm_M3" (at 228.6 147.32 0)
+      (effects (font (size 1.27 1.27)) hide)
+    )
+    (property "Datasheet" "~" (at 228.6 147.32 0)
+      (effects (font (size 1.27 1.27)) hide)
+    )
+    (instances
+      (project "hall_sensor_matrix_v2"
+        (path "/9a30e28a-cd46-4b7f-9427-a633c652be34"
+          (reference "H2") (unit 1)
+        )
+      )
     )
   )
@@
         )
       )
+    )
+  )
+  (symbol (lib_id "Mechanical:MountingHole") (at 228.6 142.24 0) (unit 1)
+    (in_bom yes) (on_board yes) (dnp no) (fields_autoplaced)
+    (property "Reference" "H1" (at 231.14 141.5963 0)
+      (effects (font (size 1.27 1.27)) (justify left))
+    )
+    (property "Value" "MountingHole" (at 231.14 143.5173 0)
+      (effects (font (size 1.27 1.27)) (justify left))
+    )
+    (property "Footprint" "MountingHole:MountingHole_3.2mm_M3" (at 228.6 142.24 0)
+      (effects (font (size 1.27 1.27)) hide)
+    )
+    (property "Datasheet" "~" (at 228.6 142.24 0)
+      (effects (font (size 1.27 1.27)) hide)
+    )
+    (instances
+      (project "hall_sensor_matrix_v2"
+        (path "/9a30e28a-cd46-4b7f-9427-a633c652be34"
+          (reference "H1") (unit 1)
+        )
+      )
