File: elevator_altimeter/receiver/receiver.kicad_sch (KiCad schematic)
At the start: 39 parts, among them Q1 TP0606, Q2 VN2210N, SW1 UserSW, SW2 PWR_SW, U1 ATmega32U4-A, U2 5631AH-S_3digit_7segment_disp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, U3 NRF24L01_Breakout, U4 PQ070XNA1ZPH

Commit message: a
Parts:
- added C12: DNP, symbol Device:C
Connections:
- net GND: now also C12.2
- net PWR_EN: now also C12.1
Other:
- moved on the sheet: Q2, R13, R15, SW2

Commit message: a
Other:
- company: (none) -> Xavier Bourlot
- title: (none) -> Elevator altimeter receiver
Changed lines of the file:
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@@
 	(generator_version "8.0")
 	(paper "A4")
+	(title_block
+		(title "Elevator altimeter receiver")
+		(date "2024-08-06")
+		(rev "A")
+		(company "Xavier Bourlot")
+	)
 	(junction
 		(at 227.33 124.46)

Commit message: a
Parts:
- added U?: TP4056, footprints:TP4056_USB-C_module, symbol _MYLIBRARY:TP4056_USB-C_module
Connections:
- net +BATT: now also U?.1 (OUT+); no longer BT1.1 (+)
- net GND: now also U?.4 (OUT-); no longer BT1.2 (-)
- new net: BT1.1 (+), U?.2 (BAT+)
- new net: BT1.2 (-), U?.3 (BAT-)
- no-connect marks 15 -> 17
Other:
- moved on the sheet: BT1
Changed lines of the file:
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@@
 	)
 	(no_connect
+		(at 45.72 125.73)
+	)
+	(no_connect
 		(at 191.77 49.53)
 	)
@@
 	)
 	(no_connect
+		(at 45.72 132.08)
+	)
+	(no_connect
 		(at 222.25 52.07)
 	)
@@
 	(wire
 		(pts
+			(xy 54.61 140.97) (xy 53.34 140.97)
+		)
+		(stroke
+			(width 0)
+			(type default)
+		)
+	)
+	(wire
+		(pts
 			(xy 160.02 124.46) (xy 176.53 124.46)
 		)
@@
 	(wire
 		(pts
+			(xy 60.96 140.97) (xy 60.96 148.59)
+		)
+		(stroke
+			(width 0)
+			(type default)
+		)
+	)
+	(wire
+		(pts
+			(xy 53.34 140.97) (xy 53.34 148.59)
+		)
+		(stroke
+			(width 0)
+			(type default)
+		)
+	)
+	(wire
+		(pts
 			(xy 222.25 67.31) (xy 233.68 67.31)
 		)
@@
 	(wire
 		(pts
+			(xy 59.69 140.97) (xy 60.96 140.97)
+		)
+		(stroke
+			(width 0)
+			(type default)
+		)
+	)
+	(wire
+		(pts
 			(xy 140.97 58.42) (xy 148.59 58.42)
 		)
@@
 	(wire
 		(pts
+			(xy 68.58 125.73) (xy 68.58 124.46)
+		)
+		(stroke
+			(width 0)
+			(type default)
+		)
+	)
+	(wire
+		(pts
 			(xy 80.01 52.07) (xy 93.98 52.07)
 		)
@@
 	(wire
 		(pts
+			(xy 68.58 124.46) (xy 74.93 124.46)
+		)
+		(stroke
+			(width 0)
+			(type default)
+		)
+	)
+	(wire
+		(pts
+			(xy 68.58 132.08) (xy 74.93 132.08)
+		)
+		(stroke
+			(width 0)
+			(type default)
+		)
+	)
+	(wire
+		(pts
 			(xy 120.65 124.46) (xy 160.02 124.46)
 		)
@@
 	(symbol
 		(lib_id "power:PWR_FLAG")
-		(at 74.93 132.08 90)
+		(at 74.93 132.08 0)
 		(unit 1)
 		(exclude_from_sim no)
@@
 		(fields_autoplaced yes)
 		(property "Reference" "#FLG02"
-			(at 73.025 132.08 0)
+			(at 74.93 130.175 0)
 			(effects
 				(font
@@
 		)
 		(property "Value" "PWR_FLAG"
-			(at 70.7969 132.08 0)
+			(at 74.93 127.9469 0)
 			(effects
 				(font
@@
 	(symbol
 		(lib_id "power:PWR_FLAG")
-		(at 74.93 124.46 90)
+		(at 74.93 124.46 180)
 		(unit 1)
 		(exclude_from_sim no)
@@
 		(fields_autoplaced yes)
 		(property "Reference" "#FLG01"
-			(at 73.025 124.46 0)
+			(at 74.93 126.365 0)
 			(effects
 				(font
@@
 		)
 		(property "Value" "PWR_FLAG"
-			(at 70.7969 124.46 0)
+			(at 74.93 128.5931 0)
 			(effects
 				(font
@@
 	)
 	(symbol
+		(lib_id "_MYLIBRARY:TP4056_USB-C_module")
+		(at 57.15 129.54 0)
+		(unit 1)
+		(exclude_from_sim no)
+		(in_bom yes)
+		(on_board yes)
+		(dnp no)
+		(fields_autoplaced yes)
+		(property "Reference" "U?"
+			(at 57.15 120.6585 0)
+			(effects
+				(font
+					(size 1.27 1.27)
+				)
+			)
+		)
+		(property "Value" "TP4056"
+			(at 57.15 122.3399 0)
+			(effects
+				(font
+					(size 1.27 1.27)
+				)
+			)
+		)
+		(property "Footprint" "footprints:TP4056_USB-C_module"
+			(at 57.15 128.27 0)
+			(effects
+				(font
+					(size 1.27 1.27)
+				)
+				(hide yes)
+			)
+		)
+		(property "Datasheet" ""
+			(at 57.15 129.54 0)
+			(effects
+				(font
+					(size 1.27 1.27)
+				)
+				(hide yes)
+			)
+		)
+		(property "Description" ""
+			(at 57.15 129.54 0)
+			(effects
+				(font
+					(size 1.27 1.27)
+				)
+				(hide yes)
+			)
+		)
+		(pin "6"
+		)
+		(pin "3"
+		)
+		(pin "7"
+		)
+		(pin "4"
+		)
+		(pin "1"
+		)
+		(pin "2"
+		)
+		(instances
+			(project "receiver"
+				(path "/508af014-8a23-4e20-8ad2-ca910f035369"
+					(reference "U?")
+					(unit 1)
+				)
+			)
+		)
+	)
+	(symbol
 		(lib_id "power:GND")
 		(at 222.25 132.08 0)
@@
 	(symbol
 		(lib_id "Device:Battery_Cell")
-		(at 74.93 129.54 0)
+		(at 58.42 148.59 90)
 		(unit 1)
 		(exclude_from_sim no)
@@
 		(fields_autoplaced yes)
 		(property "Reference" "BT1"
-			(at 77.851 126.4863 0)
+			(at 56.5785 142.2865 90)
 			(effects
 				(font
 					(size 1.27 1.27)
 				)
-				(justify left)
 			)
 		)
 		(property "Value" "18650"
-			(at 77.851 128.9106 0)
+			(at 56.5785 144.7108 90)
 			(effects
 				(font
 					(size 1.27 1.27)
 				)
-				(justify left)
 			)
 		)
 		(property "Footprint" "TerminalBlock:TerminalBlock_bornier-2_P5.08mm"
-			(at 74.93 128.016 90)
+			(at 56.896 148.59 90)
 			(effects
 				(font
@@
 		)
 		(property "Datasheet" "~"
-			(at 74.93 128.016 90)
+			(at 56.896 148.59 90)
 			(effects
 				(font
@@
 		)
 		(property "Description" "Single-cell battery"
-			(at 74.93 129.54 0)
+			(at 58.42 148.59 0)
 			(effects
 				(font
