File: elevator_altimeter/elevator_altimeter.kicad_sch (KiCad schematic)
At the start: 39 parts, among them J1 UART, J2 AVR-ICSP-TagConnect, J3 I2C, SW1 UserSW, U1 MPL3115A2, U2 NRF24L01_Breakout, U3 ATtiny1634-S, U4 MCP1711

Commit message: a
Parts:
- added U5: TP4056, footprints:TP4056_USB-C_module, symbol _MYLIBRARY:TP4056_USB-C_module
Connections:
- net +BATT: now also U5.1 (OUT+); no longer BT1.1 (+)
- net GND: now also U5.4 (OUT-); no longer BT1.2 (-)
- new net: BT1.1 (+), U5.2 (BAT+)
- new net: BT1.2 (-), U5.3 (BAT-)
- no-connect marks 4 -> 6
Other:
- moved on the sheet: BT1, C10, C11, C12, C13, C14, C15, C4, C5, C6, C7, C8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

Commit message: a
Parts:
- added H4: ~, MountingHole:MountingHole_3.2mm_M3_Pad_Via, symbol Mechanical:MountingHole_Pad
- added JP3: NRF_pwr, Jumper:SolderJumper-2_P1.3mm_Bridged_RoundedPad1.0x1.5mm, symbol Jumper:Jumper_2_Bridged
- added JP4: MPL_pwr, Jumper:SolderJumper-2_P1.3mm_Bridged_RoundedPad1.0x1.5mm, symbol Jumper:Jumper_2_Bridged
- added JP5: MCU_pwr, Jumper:SolderJumper-2_P1.3mm_Bridged_RoundedPad1.0x1.5mm, symbol Jumper:Jumper_2_Bridged
- BT1: footprint TerminalBlock:TerminalBlock_bornier-2_P5.08mm -> Battery:BatteryHolder_Keystone_1042_1x18650
Connections:
- net GND: now also H4.1
- net VDD: now also JP3.2 (B), JP4.1 (A), JP5.1 (A); no longer C11.1, C12.1, C13.1, C6.1, C7.1, C8.1, C9.1, FB1.1, U1.4 (VDDIO), U2.2 (VCC), U3.11 (VCC)
- new net MCU_pwr: C13.1, C6.1, JP5.2 (B), U3.11 (VCC)
- new net MPL_pwr: C11.1, C9.1, FB1.1, JP4.2 (B), U1.4 (VDDIO)
- new net NRF_pwr: C12.1, C7.1, C8.1, JP3.1 (A), U2.2 (VCC)
Other:
- moved on the sheet: C10, C11, C12, C13, C14, C15, C6, C7, C8, C9, FB1

Commit message: a
Parts:
- J1, J3: now not fitted
Other:
- company: (none) -> Xavier Bourlot
- title: (none) -> Elevator altimeter
Changed lines of the file:
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@@
 	(generator_version "8.0")
 	(paper "A4")
+	(title_block
+		(title "Elevator altimeter")
+		(date "2024-09-22")
+		(rev "A")
+		(company "Xavier Bourlot")
+	)
 	(junction
 		(at 152.4 132.08)
@@
 		(in_bom yes)
 		(on_board yes)
-		(dnp no)
+		(dnp yes)
 		(property "Reference" "J3"
 			(at 111.76 134.2855 0)
@@
 		(in_bom yes)
 		(on_board yes)
-		(dnp no)
+		(dnp yes)
 		(property "Reference" "J1"
 			(at 127 135.5555 0)
