File: horse_feeder/horse_feeder.kicad_pcb (KiCad board)
At the start: 2 copper layers, 100 x 100 mm, 100 parts, among them J1 PWR, J10 Btn_RST, J11 Btn_USR2, J2 Moteur 2, J3 Moteur 1, J4 Proxi 1, J5 UART, J6 Proxi 2, J7 I2C, J8 PROG, J9 Btn_USR1, M1 SIM800L, Q1 Si7155DP, Q2 BUK766R060E, Q3 BUK766R060E, Q4 VP3203, Q5 VP3203, Q6 2N7002, U1 MCP16301x-xCH, U2 MIC4427, U3 ATmega32A-P, U4 RTC, Y1 16MHz

Commit message: a
Parts:
- U3: value ATmega32A-P -> ATmega644PA-P

Commit message: a
Parts:
- J1, J10, J11, J2, J3, J9: footprint TerminalBlock:TerminalBlock_bornier-2_P5.08mm -> footprints:TerminalBlock_bornier-2_P5.08mm
Other:
- board text added: "Horse feeder revA, Feb 2025 X.B. & C.G."
- board text added: "JLCJLCJLCJLC"
- board text added: "SIM"

Commit message: a
Parts:
- added C24: 10u, Capacitor_SMD:C_0805_2012Metric_Pad1.18x1.45mm_HandSolder, B.Cu at (174.2, 54.2)
- added C25: 10u, Capacitor_SMD:C_0805_2012Metric_Pad1.18x1.45mm_HandSolder, B.Cu at (176.2, 54.2)
- added C26: 10u, Capacitor_SMD:C_0805_2012Metric_Pad1.18x1.45mm_HandSolder, B.Cu at (178.2, 54.2)
- added C27: 10u, Capacitor_SMD:C_0805_2012Metric_Pad1.18x1.45mm_HandSolder, B.Cu at (180.2, 54.2)
- added C28: 470u, Capacitor_THT:CP_Radial_D12.5mm_P5.00mm, F.Cu at (179.2, 50.2)
- added D14: BAT54C, Package_TO_SOT_SMD:SOT-23, B.Cu at (170.6, 108.5)
- added R35: 470, Resistor_SMD:R_0805_2012Metric_Pad1.20x1.40mm_HandSolder, B.Cu at (174.6, 109.5)
- added R36: 470, Resistor_SMD:R_0805_2012Metric_Pad1.20x1.40mm_HandSolder, B.Cu at (170.8, 105.8)
Connections:
- U3 pad 38: /Mot2_I -> /Mot1_Ip
- U3 pad 39: /Mot1_I -> /Mot2_Ip
Routing:
- net /Mot1_I: track 5.13 -> 44.3 mm
- net GND: track 153.2 -> 176.1 mm
- net /Mot2_I: track 5.54 -> 25.3 mm
- net +5VP: track 22.6 -> 38.1 mm
- net +5V: track 308.2 -> 311.1 mm
- net /Mot2_Ip: track 0.00 -> 2.15 mm
- net /Mot1_Ip: track 0.00 -> 1.95 mm
