File: horse_feeder/horse_feeder.kicad_sch (KiCad schematic)
At the start: 100 parts, among them J1 PWR, J10 Btn_RST, J11 Btn_USR2, J2 Moteur 2, J3 Moteur 1, J4 Proxi 1, J5 UART, J6 Proxi 2, J7 I2C, J8 PROG, J9 Btn_USR1, M1 SIM800L, Q1 Si7155DP, Q2 BUK766R060E, Q3 BUK766R060E, Q4 VP3203, Q5 VP3203, Q6 2N7002, U1 MCP16301x-xCH, U2 MIC4427, U3 ATmega32A-P, U4 RTC, Y1 16MHz

Commit message: a
Parts:
- removed U3: ATmega32A-P, Package_DIP:DIP-40_W15.24mm, symbol MCU_Microchip_ATmega:ATmega32A-P
- added U3: ATmega644PA-P, Package_DIP:DIP-40_W15.24mm, symbol MCU_Microchip_ATmega:ATmega644PA-P
Connections:
- net +5V: now also U3.10 (VCC), U3.30 (AVCC), U3.32 (AREF)
- net Batt_mon: now also U3.40 (PA0)
- net Btn_USR1: now also U3.24 (PC2)
- net Btn_USR2: now also U3.25 (PC3)
- net GND: now also U3.11 (GND), U3.31 (GND)
- net LED_B: now also U3.37 (PA3)
- net LED_G: now also U3.36 (PA4)
- net LED_R: now also U3.34 (PA6)
- net LED_Y: now also U3.35 (PA5)
- net MISO: now also U3.7 (PB6)
- net MOSI: now also U3.6 (PB5)
- net Mot1_I: now also U3.39 (PA1)
- net Mot1_PWM: now also U3.19 (PD5)
- net Mot2_I: now also U3.38 (PA2)
- net Mot2_PWM: now also U3.18 (PD4)
- net Proxi1: now also U3.16 (PD2)
- net Proxi2: now also U3.17 (PD3)
- net Proxi_PWR: now also U3.26 (PC4)
- net RST: now also U3.9 (~{RESET})
- net RTC_SCL: now also U3.22 (PC0)
- net RTC_SDA: now also U3.23 (PC1)
- net RTC_SQW: now also U3.3 (PB2)
- net SCK: now also U3.8 (PB7)
- net SIM_PWR: now also U3.27 (PC5)
- net SIM_RST: now also U3.20 (PD6)
- net SIM_RX: now also U3.15 (PD1)
- net SIM_TX: now also U3.14 (PD0)
- net XTAL1: now also U3.13 (XTAL1)
- net XTAL2: now also U3.12 (XTAL2)

Commit message: a
Parts:
- J1, J10, J11, J2, J3, J9: footprint TerminalBlock:TerminalBlock_bornier-2_P5.08mm -> footprints:TerminalBlock_bornier-2_P5.08mm
- J5, J7: now not fitted
Changed lines of the file:
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@@
 			)
 		)
-		(property "Footprint" "TerminalBlock:TerminalBlock_bornier-2_P5.08mm"
+		(property "Footprint" "footprints:TerminalBlock_bornier-2_P5.08mm"
 			(at 271.78 25.4 0)
 			(effects
@@
 		(in_bom yes)
 		(on_board yes)
-		(dnp no)
+		(dnp yes)
 		(fields_autoplaced yes)
 		(property "Reference" "J5"
@@
 			)
 		)
-		(property "Footprint" "TerminalBlock:TerminalBlock_bornier-2_P5.08mm"
+		(property "Footprint" "footprints:TerminalBlock_bornier-2_P5.08mm"
 			(at 19.05 179.07 0)
 			(effects
@@
 		(in_bom yes)
 		(on_board yes)
-		(dnp no)
+		(dnp yes)
 		(fields_autoplaced yes)
 		(property "Reference" "J7"
@@
 			)
 		)
-		(property "Footprint" "TerminalBlock:TerminalBlock_bornier-2_P5.08mm"
+		(property "Footprint" "footprints:TerminalBlock_bornier-2_P5.08mm"
 			(at 21.59 24.13 0)
 			(effects
@@
 			)
 		)
-		(property "Footprint" "TerminalBlock:TerminalBlock_bornier-2_P5.08mm"
+		(property "Footprint" "footprints:TerminalBlock_bornier-2_P5.08mm"
 			(at 60.96 151.13 0)
 			(effects
@@
 			)
 		)
-		(property "Footprint" "TerminalBlock:TerminalBlock_bornier-2_P5.08mm"
+		(property "Footprint" "footprints:TerminalBlock_bornier-2_P5.08mm"
 			(at 271.78 62.23 0)
 			(effects
@@
 			)
 		)
-		(property "Footprint" "TerminalBlock:TerminalBlock_bornier-2_P5.08mm"
+		(property "Footprint" "footprints:TerminalBlock_bornier-2_P5.08mm"
 			(at 19.05 149.86 0)
 			(effects

Commit message: a
Parts:
- added C24, C25, C26, C27: 10u, Capacitor_SMD:C_0805_2012Metric_Pad1.18x1.45mm_HandSolder, symbol Device:C_Polarized
- added C28: 470u, Capacitor_THT:CP_Radial_D12.5mm_P5.00mm, symbol Device:C_Polarized
- added D14: BAT54C, Package_TO_SOT_SMD:SOT-23, symbol Diode:BAT54C
- added R35, R36: 470, Resistor_SMD:R_0805_2012Metric_Pad1.20x1.40mm_HandSolder, symbol Device:R
Connections:
- net +5V: now also D14.3
- net +5VP: now also C24.1, C25.1, C26.1, C27.1, C28.1
- net GND: now also C24.2, C25.2, C26.2, C27.2, C28.2
- net Mot1_I: now also R36.2; no longer U3.39 (PA1)
- net Mot2_I: now also R35.2; no longer U3.38 (PA2)
- new net Mot1_Ip: D14.1, R36.1, U3.38 (PA2)
- new net Mot2_Ip: D14.2, R35.1, U3.39 (PA1)
Other:
- moved on the sheet: C15
