File: horse_feeder/HW/v2_M590E/horse_feeder.kicad_pcb (KiCad board)
At the start: 2 copper layers, 100 x 100 mm, 109 parts, among them J1 PWR, J10 Btn_RST, J11 Btn_USR2, J2 Moteur 2, J3 Moteur 1, J4 Proxi 1, J5 UART, J6 Proxi 2, J7 I2C, J8 PROG, J9 Btn_USR1, M1 M590E, Q1 Si7155DP, Q2 BUK766R060E, Q3 BUK766R060E, Q5 VP3203, Q6 2N7002, U2 MIC4427, U3 ATmega644PA-P, U4 RTC, U5 LM2576HVT-ADJ, Y1 16MHz

Commit message: a
Parts:
- added D13: SS14, Diode_SMD:D_SMA, B.Cu at (199.0, 108.0)
- D15, D4, D6: footprint Package_TO_SOT_SMD:SOT-323_SC-70 -> Package_TO_SOT_SMD:SOT-23
- D3: value BAT54C -> SS14; footprint Package_TO_SOT_SMD:SOT-23 -> Diode_SMD:D_SMA
- moved D15 5.73 mm to (119.2, 59.2)
- moved D3 4.12 mm to (200.0, 92.0)
- moved D4 0.40 mm to (198.5, 73.0)
- moved C20 0.35 mm to (198.5, 61.8)
- moved R19 0.35 mm to (198.5, 59.8)
Connections:
- D3 pad 1: /Mot1_D -> +12V
- D3 pad 2: /Mot2_D -> /Mot1_D
Routing:
- net +12V: track 314.8 -> 325.8 mm
- net +5V: track 191.3 -> 192.7 mm
- net /Mot1_D: track 11.7 -> 10.7 mm
- net GND: track 138.3 -> 137.5 mm, vias 3 -> 16
- net +12P: track 37.1 -> 37.8 mm
- net +5VP: track 63.6 -> 64.1 mm
Other:
- board text added: "Gate Driver"
- board text added: "MCU"
- board text added: "Miam !"
- board text added: "SIM Module"
