File: horse_feeder/HW/v2_M590E/horse_feeder.kicad_sch (KiCad schematic)
At the start: 109 parts, among them J1 PWR, J10 Btn_RST, J11 Btn_USR2, J2 Moteur 2, J3 Moteur 1, J4 Proxi 1, J5 UART, J6 Proxi 2, J7 I2C, J8 PROG, J9 Btn_USR1, M1 M590E, Q1 Si7155DP, Q2 BUK766R060E, Q3 BUK766R060E, Q5 VP3203, Q6 2N7002, U2 MIC4427, U3 ATmega644PA-P, U4 RTC, U5 LM2576HVT-ADJ, Y1 16MHz

Commit message: a
Parts:
- removed D3: BAT54C, Package_TO_SOT_SMD:SOT-23, symbol Diode:BAT54C
- added D13, D3: SS14, Diode_SMD:D_SMA, symbol Diode:SS14
- D15, D4, D6: footprint Package_TO_SOT_SMD:SOT-323_SC-70 -> Package_TO_SOT_SMD:SOT-23
- J8: footprint (none) -> Connector_IDC:IDC-Header_2x05_P2.54mm_Vertical
Connections:
- net +12V: now also D13.1 (K), D3.1 (K)
- net Mot1_D: now also D3.2 (A)
- net Mot2_D: now also D13.2 (A)
Changed lines of the file:
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@@
 	)
 	(junction
+		(at 257.81 22.86)
+		(diameter 0)
+		(color 0 0 0 0)
+	)
+	(junction
 		(at 35.56 184.15)
 		(diameter 0)
@@
 	)
 	(junction
+		(at 257.81 30.48)
+		(diameter 0)
+		(color 0 0 0 0)
+	)
+	(junction
 		(at 111.76 24.13)
 		(diameter 0)
@@
 	(wire
 		(pts
+			(xy 255.27 30.48) (xy 257.81 30.48)
+		)
+		(stroke
+			(width 0)
+			(type default)
+		)
+	)
+	(wire
+		(pts
 			(xy 140.97 177.8) (xy 140.97 180.34)
 		)
@@
 	(wire
 		(pts
-			(xy 257.81 59.69) (xy 254 59.69)
+			(xy 257.81 59.69) (xy 255.27 59.69)
 		)
 		(stroke
@@
 	(wire
 		(pts
+			(xy 255.27 22.86) (xy 257.81 22.86)
+		)
+		(stroke
+			(width 0)
+			(type default)
+		)
+	)
+	(wire
+		(pts
 			(xy 78.74 24.13) (xy 90.17 24.13)
 		)
@@
 	(wire
 		(pts
-			(xy 257.81 67.31) (xy 248.92 67.31)
+			(xy 257.81 67.31) (xy 255.27 67.31)
 		)
 		(stroke
@@
 		)
 	)
-	(label "Mot2_D"
-		(at 248.92 52.07 90)
-		(effects
-			(font
-				(size 1.27 1.27)
-			)
-			(justify left bottom)
-		)
-	)
 	(label "LED_G"
 		(at 129.54 170.18 0)
@@
 	)
 	(symbol
+		(lib_id "Diode:SS14")
+		(at 255.27 63.5 270)
+		(unit 1)
+		(exclude_from_sim no)
+		(in_bom yes)
+		(on_board yes)
+		(dnp no)
+		(fields_autoplaced yes)
+		(property "Reference" "D3"
+			(at 253.238 61.9703 90)
+			(effects
+				(font
+					(size 1.27 1.27)
+				)
+				(justify right)
+			)
+		)
+		(property "Value" "SS14"
+			(at 253.238 64.3946 90)
+			(effects
+				(font
+					(size 1.27 1.27)
+				)
+				(justify right)
+			)
+		)
+		(property "Footprint" "Diode_SMD:D_SMA"
+			(at 250.825 63.5 0)
+			(effects
+				(font
+					(size 1.27 1.27)
+				)
+				(hide yes)
+			)
+		)
+		(property "Datasheet" "https://www.vishay.com/docs/88746/ss12.pdf"
+			(at 255.27 63.5 0)
+			(effects
+				(font
+					(size 1.27 1.27)
+				)
+				(hide yes)
+			)
+		)
+		(property "Description" "40V 1A Schottky Diode, SMA"
+			(at 255.27 63.5 0)
+			(effects
+				(font
+					(size 1.27 1.27)
+				)
+				(hide yes)
+			)
+		)
+		(pin "1"
+		)
+		(pin "2"
+		)
+		(instances
+			(project ""
+				(path "/bdeff217-2bc0-4651-8ab4-3cac9152fd39"
+					(reference "D3")
+					(unit 1)
+				)
+			)
+		)
+	)
+	(symbol
 		(lib_id "power:GND")
 		(at 50.8 59.69 0)
@@
 			)
 		)
-		(property "Footprint" "Package_TO_SOT_SMD:SOT-323_SC-70"
+		(property "Footprint" "Package_TO_SOT_SMD:SOT-23"
 			(at 60.96 56.515 0)
 			(effects
@@
 	)
 	(symbol
+		(lib_id "Diode:SS14")
+		(at 255.27 26.67 270)
+		(unit 1)
+		(exclude_from_sim no)
+		(in_bom yes)
+		(on_board yes)
+		(dnp no)
+		(fields_autoplaced yes)
+		(property "Reference" "D13"
+			(at 253.238 25.1403 90)
+			(effects
+				(font
+					(size 1.27 1.27)
+				)
+				(justify right)
+			)
+		)
+		(property "Value" "SS14"
+			(at 253.238 27.5646 90)
+			(effects
+				(font
+					(size 1.27 1.27)
+				)
+				(justify right)
+			)
+		)
+		(property "Footprint" "Diode_SMD:D_SMA"
+			(at 250.825 26.67 0)
+			(effects
+				(font
+					(size 1.27 1.27)
+				)
+				(hide yes)
+			)
+		)
+		(property "Datasheet" "https://www.vishay.com/docs/88746/ss12.pdf"
+			(at 255.27 26.67 0)
+			(effects
+				(font
+					(size 1.27 1.27)
+				)
+				(hide yes)
+			)
+		)
+		(property "Description" "40V 1A Schottky Diode, SMA"
+			(at 255.27 26.67 0)
+			(effects
+				(font
+					(size 1.27 1.27)
+				)
+				(hide yes)
+			)
+		)
+		(pin "1"
+		)
+		(pin "2"
+		)
+		(instances
+			(project "horse_feeder"
+				(path "/bdeff217-2bc0-4651-8ab4-3cac9152fd39"
+					(reference "D13")
+					(unit 1)
+				)
+			)
+		)
+	)
+	(symbol
 		(lib_id "power:GND")
 		(at 85.09 189.23 0)
@@
 			)
 		)
-		(property "Footprint" "Package_TO_SOT_SMD:SOT-323_SC-70"
+		(property "Footprint" "Package_TO_SOT_SMD:SOT-23"
 			(at 41.275 93.98 0)
 			(effects
@@
 			)
 		)
-		(property "Footprint" "Package_TO_SOT_SMD:SOT-323_SC-70"
+		(property "Footprint" "Package_TO_SOT_SMD:SOT-23"
 			(at 46.355 120.65 0)
 			(effects
@@
 			)
 		)
-		(property "Footprint" ""
+		(property "Footprint" "Connector_IDC:IDC-Header_2x05_P2.54mm_Vertical"
 			(at 266.7 146.05 90)
 			(effects
@@
 					(unit 1)
 				)
-			)
-		)
-	)
-	(symbol
-		(lib_id "Diode:BAT54C")
-		(at 248.92 59.69 90)
-		(unit 1)
-		(exclude_from_sim no)
-		(in_bom yes)
-		(on_board yes)
-		(dnp no)
-		(property "Reference" "D3"
-			(at 247.015 58.4778 90)
-			(effects
-				(font
-					(size 1.27 1.27)
-				)
-				(justify left)
-			)
-		)
-		(property "Value" "BAT54C"
-			(at 247.015 60.9021 90)
-			(effects
-				(font
-					(size 1.27 1.27)
-				)
-				(justify left)
-			)
-		)
-		(property "Footprint" "Package_TO_SOT_SMD:SOT-23"
-			(at 245.745 57.785 0)
-			(effects
-				(font
-					(size 1.27 1.27)
-				)
-				(justify left)
-				(hide yes)
-			)
-		)
-		(property "Datasheet" "http://www.diodes.com/_files/datasheets/ds11005.pdf"
-			(at 248.92 61.722 0)
-			(effects
-				(font
-					(size 1.27 1.27)
-				)
-				(hide yes)
-			)
-		)
-		(property "Description" "dual schottky barrier diode, common cathode"
-			(at 248.92 59.69 0)
-			(effects
-				(font
-					(size 1.27 1.27)
-				)
-				(hide yes)
-			)
-		)
-		(pin "1"
-		)
-		(pin "3"
-		)
-		(pin "2"
-		)
-		(instances
-			(project "horse_feeder"
-				(path "/bdeff217-2bc0-4651-8ab4-3cac9152fd39"
-					(reference "D3")
-					(unit 1)
-				)
