File: horse_feeder/HW/PCB_v2_M590E/horse_feeder.kicad_sch (KiCad schematic)
At the start: 110 parts, among them J1 PWR, J10 Btn_RST, J11 Btn_USR2, J2 Moteur 2, J3 Moteur 1, J4 Proxi 1, J5 UART, J6 Proxi 2, J7 I2C, J8 PROG, J9 Btn_USR1, M1 M590E, Q1 Si7155DP, Q2 BUK766R060E, Q3 BUK766R060E, Q5 VP3203, Q6 2N7002, U2 MIC4427, U3 ATmega644PA-P, U4 RTC, U5 LM2576HVT-ADJ, Y1 16MHz

Commit message: a
Parts:
- JP1, JP2: now left out of the parts list
Changed lines of the file:
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@@
 	(label "Mot1_Ip"
 		(at 157.48 76.2 180)
+		(fields_autoplaced yes)
 		(effects
 			(font
@@
 	(label "MOSI"
 		(at 241.3 144.78 0)
+		(fields_autoplaced yes)
 		(effects
 			(font
@@
 	(label "Mot2_I"
 		(at 251.46 40.64 180)
+		(fields_autoplaced yes)
 		(effects
 			(font
@@
 	(label "SIM_RXl"
 		(at 236.22 107.95 0)
+		(fields_autoplaced yes)
 		(effects
 			(font
@@
 	(label "SIM_RX"
 		(at 149.86 142.24 0)
+		(fields_autoplaced yes)
 		(effects
 			(font
@@
 	(label "Proxi2"
 		(at 41.91 116.84 0)
+		(fields_autoplaced yes)
 		(effects
 			(font
@@
 	(label "Mot2_G"
 		(at 243.84 35.56 0)
+		(fields_autoplaced yes)
 		(effects
 			(font
@@
 	(label "Btn_USR2"
 		(at 39.37 179.07 180)
+		(fields_autoplaced yes)
 		(effects
 			(font
@@
 	(label "RTC_SDA"
 		(at 149.86 119.38 0)
+		(fields_autoplaced yes)
 		(effects
 			(font
@@
 	(label "Mot2_I"
 		(at 167.64 73.66 0)
+		(fields_autoplaced yes)
 		(effects
 			(font
@@
 	(label "Proxi_PWR"
 		(at 149.86 127 0)
+		(fields_autoplaced yes)
 		(effects
 			(font
@@
 	(label "SIM_TX"
 		(at 204.47 105.41 0)
+		(fields_autoplaced yes)
 		(effects
 			(font
@@
 	(label "LED_Y_fp"
 		(at 25.4 149.86 0)
+		(fields_autoplaced yes)
 		(effects
 			(font
@@
 	(label "LED_R"
 		(at 149.86 81.28 0)
+		(fields_autoplaced yes)
 		(effects
 			(font
@@
 	(label "Vin"
 		(at 36.83 24.13 0)
+		(fields_autoplaced yes)
 		(effects
 			(font
@@
 	(label "Mot2_PWM"
 		(at 198.12 77.47 0)
+		(fields_autoplaced yes)
 		(effects
 			(font
@@
 	(label "XTAL2"
 		(at 102.87 81.28 0)
+		(fields_autoplaced yes)
 		(effects
 			(font
@@
 	(label "MISO"
 		(at 149.86 109.22 0)
+		(fields_autoplaced yes)
 		(effects
 			(font
@@
 	(label "Mot1_G"
 		(at 243.84 72.39 0)
+		(fields_autoplaced yes)
 		(effects
 			(font
@@
 	(label "LED_B"
 		(at 140.97 170.18 0)
+		(fields_autoplaced yes)
 		(effects
 			(font
@@
 	(label "LED_B_fp"
 		(at 140.97 180.34 0)
+		(fields_autoplaced yes)
 		(effects
 			(font
@@
 	(label "LED_R_fp"
 		(at 106.68 180.34 0)
+		(fields_autoplaced yes)
 		(effects
 			(font
@@
 	(label "Btn_USR1"
 		(at 40.64 142.24 180)
+		(fields_autoplaced yes)
 		(effects
 			(font
@@
 	(label "LED_Y"
 		(at 118.11 170.18 0)
+		(fields_autoplaced yes)
 		(effects
 			(font
@@
 	(label "SIM_BOOT"
 		(at 149.86 154.94 0)
+		(fields_autoplaced yes)
 		(effects
 			(font
@@
 	(label "RST"
 		(at 241.3 149.86 0)
+		(fields_autoplaced yes)
 		(effects
 			(font
@@
 	(label "LED_G_fp"
 		(at 129.54 180.34 0)
+		(fields_autoplaced yes)
 		(effects
 			(font
@@
 	(label "RTC_SCL"
 		(at 204.47 148.59 0)
+		(fields_autoplaced yes)
 		(effects
 			(font
@@
 	(label "LED_Y_fp"
 		(at 118.11 180.34 0)
+		(fields_autoplaced yes)
 		(effects
 			(font
@@
 	(label "Mot1_PWM"
 		(at 149.86 152.4 0)
+		(fields_autoplaced yes)
 		(effects
 			(font
@@
 	(label "SIM_BOOT"
 		(at 236.22 115.57 0)
+		(fields_autoplaced yes)
 		(effects
 			(font
@@
 	(label "Mot2_D"
 		(at 265.43 25.4 180)
+		(fields_autoplaced yes)
 		(effects
 			(font
@@
 	(label "Proxi2"
 		(at 149.86 144.78 0)
+		(fields_autoplaced yes)
 		(effects
 			(font
@@
 	(label "LED_Y"
 		(at 149.86 86.36 0)
+		(fields_autoplaced yes)
 		(effects
 			(font
@@
 	(label "Mot2_Ip"
 		(at 157.48 73.66 180)
+		(fields_autoplaced yes)
 		(effects
 			(font
@@
 	(label "Mot2_PWM"
 		(at 149.86 149.86 0)
+		(fields_autoplaced yes)
 		(effects
 			(font
@@
 	(label "Btn_USR2"
 		(at 149.86 124.46 0)
+		(fields_autoplaced yes)
 		(effects
 			(font
@@
 	(label "Proxi1"
 		(at 149.86 147.32 0)
+		(fields_autoplaced yes)
 		(effects
 			(font
@@
 	(label "MISO"
 		(at 241.3 142.24 0)
+		(fields_autoplaced yes)
 		(effects
 			(font
@@
 	(label "Btn_USR1"
 		(at 149.86 121.92 0)
+		(fields_autoplaced yes)
 		(effects
 			(font
@@
 	(label "Mot1_D"
 		(at 265.43 62.23 180)
+		(fields_autoplaced yes)
 		(effects
 			(font
@@
 	(label "Mot2_PWM"
 		(at 163.83 170.18 0)
+		(fields_autoplaced yes)
 		(effects
 			(font
@@
 	(label "5V_fb"
 		(at 187.96 21.59 0)
+		(fields_autoplaced yes)
 		(effects
 			(font
@@
 	(label "Batt_mon"
 		(at 147.32 71.12 0)
+		(fields_autoplaced yes)
 		(effects
 			(font
@@
 	(label "RTC_SDA"
 		(at 204.47 146.05 0)
+		(fields_autoplaced yes)
 		(effects
 			(font
@@
 	(label "Mot1_PWM"
 		(at 152.4 170.18 0)
+		(fields_autoplaced yes)
 		(effects
 			(font
@@
 	(label "Proxi_PWR"
 		(at 87.63 154.94 180)
+		(fields_autoplaced yes)
 		(effects
 			(font
@@
 	(label "XTAL1"
 		(at 102.87 76.2 0)
+		(fields_autoplaced yes)
 		(effects
 			(font
@@
 	(label "SIM_RX"
 		(at 180.34 101.6 0)
+		(fields_autoplaced yes)
 		(effects
 			(font
@@
 	(label "SIM_TXl"
 		(at 236.22 105.41 0)
+		(fields_autoplaced yes)
 		(effects
 			(font
@@
 	(label "RTC_SDA"
 		(at 180.34 119.38 0)
+		(fields_autoplaced yes)
 		(effects
 			(font
@@
 	(label "Mot1_I"
 		(at 251.46 77.47 180)
+		(fields_autoplaced yes)
 		(effects
 			(font
@@
 	(label "LED_G"
 		(at 129.54 170.18 0)
+		(fields_autoplaced yes)
 		(effects
 			(font
@@
 	(label "Mot1_PWM"
 		(at 198.12 72.39 0)
+		(fields_autoplaced yes)
 		(effects
 			(font
@@
 	(label "LED_R_fp"
 		(at 59.69 187.96 0)
+		(fields_autoplaced yes)
 		(effects
 			(font
@@
 	(label "Proxi1"
 		(at 39.37 90.17 0)
+		(fields_autoplaced yes)
 		(effects
 			(font
@@
 	(label "SIM_TX"
 		(at 180.34 104.14 0)
+		(fields_autoplaced yes)
 		(effects
 			(font
@@
 	(label "RTC_SCL"
 		(at 180.34 116.84 0)
+		(fields_autoplaced yes)
 		(effects
 			(font
@@
 	(label "Mot1_I"
 		(at 167.64 76.2 0)
+		(fields_autoplaced yes)
 		(effects
 			(font
@@
 	(label "5V_sw"
 		(at 170.18 29.21 0)
+		(fields_autoplaced yes)
 		(effects
 			(font
@@
 	(label "LED_G"
 		(at 149.86 83.82 0)
+		(fields_autoplaced yes)
 		(effects
 			(font
@@
 	(label "RTC_SCL"
 		(at 149.86 116.84 0)
+		(fields_autoplaced yes)
 		(effects
 			(font
@@
 	(label "Batt_mon"
 		(at 132.08 31.75 0)
+		(fields_autoplaced yes)
 		(effects
 			(font
@@
 	(label "LED_B"
 		(at 149.86 78.74 0)
+		(fields_autoplaced yes)
 		(effects
 			(font
@@
 	(label "SCK"
 		(at 241.3 147.32 0)
+		(fields_autoplaced yes)
 		(effects
 			(font
@@
 	(label "SCK"
 		(at 149.86 111.76 0)
+		(fields_autoplaced yes)
 		(effects
 			(font
@@
 	(label "MOSI"
 		(at 149.86 106.68 0)
+		(fields_autoplaced yes)
 		(effects
 			(font
@@
 	(label "LED_G_fp"
 		(at 24.13 186.69 0)
+		(fields_autoplaced yes)
 		(effects
 			(font
@@
 	(label "SIM_TX"
 		(at 149.86 139.7 0)
+		(fields_autoplaced yes)
 		(effects
 			(font
@@
 	(label "RST"
 		(at 67.31 180.34 0)
+		(fields_autoplaced yes)
 		(effects
 			(font
@@
 	(label "LED_R"
 		(at 106.68 170.18 0)
+		(fields_autoplaced yes)
 		(effects
 			(font
@@
 	(label "RST"
 		(at 102.87 71.12 0)
+		(fields_autoplaced yes)
 		(effects
 			(font
@@
 	(label "SIM_RX"
 		(at 204.47 107.95 0)
+		(fields_autoplaced yes)
 		(effects
 			(font
@@
 		(unit 1)
 		(exclude_from_sim yes)
-		(in_bom yes)
+		(in_bom no)
 		(on_board yes)
 		(dnp no)
@@
 		(unit 1)
 		(exclude_from_sim yes)
-		(in_bom yes)
+		(in_bom no)
 		(on_board yes)
 		(dnp no)

Commit message: a
Parts:
- R10, R6: value 22 -> 51
- R12, R9: value 0R2 -> 0R1
- R13, R17: now not fitted
Other:
- note added: "+Rpd 39k"
- note added: "15V->1V7"
- note added: "39k"
- note added: "Rpar 4k3"
- note added: "Rpd 18k"

Commit message: a
Parts:
- JP1, JP2: now not fitted
Other:
- note added: "+Rpd 18k"
- note added: "+S15L30C dual schottky"
- note added: "15A slow"
- note added: "3.8V"
- note added: "4.2V"
- note added: "Alimentation"
- note added: "Alimentation capteurs de proximité (~6mA/capteur)"
- note added: "Boutons latéraux illuminés"
- note added: "Capteurs inductifs de proximité"
- note added: "Commande moteur avec soft start/stop."
- note added: "Commande relais 12V 15A DPDT pour inversion polarité moteur."
- note added: "Entrée 12V (Pb AGM, >8A)"
- note added: "Horloge temps-réel"
- note added: "Module SIM"
- note added: "Port programmation ICSP"
- note added: "Protection inversion polarité"
- note added: "Protection surtensions foudre"
- note added: "Régulateur buck 4.2V >2A pour module SIM & MCU."
- note added: "SIM M590 ou SIM800L Alimentation 4.2V Interface UART 3.8V 115200 bauds"
- note added: "Shorted"
- note added: "Sorties moteurs"
- note added: "Surveillance tension batterie"
- note removed: "Rpd 18k"
- title: Horse Feeder Ctrl -> Horse Feeder Controller
- moved on the sheet: C10, C11, C12, C13, C14, C15, C16, C17, C18, C19, C20, C21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
