File: LabBooster/LabBooster.kicad_pcb (KiCad board)
At the start: 2 copper layers, 74.8 x 69.5 mm, 82 parts, among them J1 PWR, J2 BNC_IN, J3 BNC_OUT, Q1 TIP41, Q10 TIP42, Q2 TIP42, Q3 2N3906, Q4 2N3904, Q5 2N3904, Q6 2N3906, Q7 2N3904, Q8 2N3906, Q9 TIP41, SW1 G-Term_A, SW2 G-Term_B, SW3 Uni/Bi, U1 TL084

Commit message: a
Other:
- net class Default removed
- net class Power removed
