File: Kheprisme/HW/proto_expo_v0/proto_expo_v0.kicad_sch (KiCad schematic)
At the start: 14 parts, among them J1 GY-45 MMA8451, J2 DS3231 RTC, J3 Conn_01x15, J4 Conn_01x15, J5 Screw_Terminal_01x04, J6 PWR, U1 stepper_driver

Commit message: added proto v0
Parts:
- added C4, C5: 100n, Capacitor_SMD:C_0805_2012Metric_Pad1.18x1.45mm_HandSolder, symbol Device:C
- added D2: LED_Dual_AAKK, LED_SMD:LED_Avago_PLCC4_3.2x2.8mm_CW, symbol Device:LED_Dual_AAKK
- added J7: USR_BTN, Connector_PinHeader_2.00mm:PinHeader_2x02_P2.00mm_Vertical, symbol Connector_Generic:Conn_02x02_Counter_Clockwise
- added R1, R2, R3, R4: 1k, Resistor_SMD:R_0805_2012Metric_Pad1.20x1.40mm_HandSolder, symbol Device:R
- added SW1: USR1, Button_Switch_THT:SW_PUSH_6mm_H4.3mm, symbol Switch:SW_MEC_5E
- added SW2: USR2, Button_Switch_THT:SW_PUSH_6mm_H4.3mm, symbol Switch:SW_MEC_5E
- added U2: Mini360, footprints:Mini360_step-down, symbol _MYLIBRARY:Mini360
- C1: footprint (none) -> Capacitor_SMD:C_0805_2012Metric_Pad1.18x1.45mm_HandSolder
- C2, C3: footprint (none) -> Capacitor_THT:CP_Radial_D10.0mm_P2.50mm_P5.00mm
- D1: footprint (none) -> Diode_SMD:D_SMB
- J1: footprint (none) -> Connector_PinSocket_2.54mm:PinSocket_1x08_P2.54mm_Vertical
- J2: footprint (none) -> Connector_PinSocket_2.54mm:PinSocket_1x06_P2.54mm_Vertical
- J3, J4: footprint (none) -> Connector_PinSocket_2.54mm:PinSocket_1x15_P2.54mm_Vertical
- J5: footprint (none) -> TerminalBlock:TerminalBlock_bornier-4_P5.08mm
- J6: footprint (none) -> TerminalBlock:TerminalBlock_bornier-2_P5.08mm
- JP1, JP2: footprint (none) -> Jumper:SolderJumper-2_P1.3mm_Bridged_RoundedPad1.0x1.5mm
- NT1: footprint (none) -> NetTie:NetTie-2_SMD_Pad0.5mm
- U1: footprint (none) -> easy_stepper_driver:easy_stepper_driver
Connections:
- net +12V: now also U2.2 (IN+)
- net +5V: now also U2.4 (OUT+)
- net DIR: now also J4.11 (Pin_11)
- net EN: now also J4.15 (Pin_15)
- net GNDD: now also C4.2, C5.2, D2.3 (K1), D2.4 (K2), J7.3 (Pin_3), J7.4 (Pin_4), SW1.3 (K), SW1.4 (A), SW2.3 (K), SW2.4 (A), U2.3 (OUT-)
- net GNDPWR: now also U2.1 (IN-)
- net SLEEP: now also J4.6 (Pin_6)
- net STEP: now also J4.12 (Pin_12)
- net LED_2: now reaches J3.11 (Pin_11)
- net LED_2: now also R4.2
- net LED_1: now reaches J3.12 (Pin_12)
- net LED_1: now also R3.2
- net USR_2: now reaches J4.7 (Pin_7)
- net USR_2: now also C4.1, R1.1
- net USR_1: now reaches J4.8 (Pin_8)
- net USR_1: now also C5.1, R2.1
- new net: J7.1 (Pin_1), R2.2, SW1.1, SW1.2
- new net: J7.2 (Pin_2), R1.2, SW2.1, SW2.2
- new net: D2.2 (A2), R3.1
- new net: D2.1 (A1), R4.1
- no-connect marks 7 -> 19
Other:
- company: (none) -> X.B.
- title: (none) -> Kheprisme_proto_cntl

Commit message: added TODO list
Parts:
- added C6: 100n, Capacitor_SMD:C_0805_2012Metric_Pad1.18x1.45mm_HandSolder, symbol Device:C
- J1: value GY-45 MMA8451 -> Accelero MMA8451
Connections:
- net +5V: now also C6.1
- net GNDD: now also C6.2
Other:
- note added: "12V -> 5V buck regulator"
- moved on the sheet: C1, C2, C3, J5, J6, JP1, JP2, NT1, U1, U2
