File: Kheprism/HW/proto_expo_v0/proto_expo_v0.kicad_sch (KiCad schematic)
At the start: 26 parts, among them J1 Accelero MMA8451, J2 DS3231 RTC, J3 Conn_01x15, J4 Conn_01x15, J5 Screw_Terminal_01x04, J6 PWR, J7 USR_BTN, SW1 USR1, SW2 USR2, U1 stepper_driver, U2 Mini360

Commit message: fix typo
Other:
- title: Kheprisme_proto_cntl -> Kheprism_proto_cntl
Changed lines of the file:
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@@
 	(paper "A4")
 	(title_block
-		(title "Kheprisme_proto_cntl")
+		(title "Kheprism_proto_cntl")
 		(date "2025-11-06")
 		(rev "A")
