File: Kheprism/HW/PCB_Ventil/Kicad/PCB_Ventil.kicad_pcb (KiCad board)
At the start: 2 copper layers, 87.5 x 100 mm, 53 parts, among them J1 Vin+, J10 Peltier3-, J11 Fan1A, J12 Fan1B, J13 Fan2A, J14 Fan2B, J15 Vin+, J16 Vin-, J17 Peltier1+, J18 Peltier1+, J2 Vin-, J3 Raspberry_Pi_4, J4 NTC, J5 Peltier1+, J6 Peltier1-, J7 Peltier2+, J8 Peltier2-, J9 Peltier3+, Q1 DMT6009LCT, Q2 DMT6009LCT, Q3 DMT6009LCT

Commit message: new rev with Mano
Parts:
- added J19: NTC2, TerminalBlock:TerminalBlock_MaiXu_MX126-5.0-03P_1x03_P5.00mm, F.Cu at (53.5, 115.8)
- added J20: Peltier1+, MountingHole:MountingHole_3.2mm_M3, F.Cu at (35.5, 25.8)
- added J21: Peltier1+, MountingHole:MountingHole_3.2mm_M3, F.Cu at (113.0, 115.8)
- added R22: 10k, Resistor_THT:R_Axial_DIN0309_L9.0mm_D3.2mm_P2.54mm_Vertical, F.Cu at (54.9, 108.8)
- added U1: CD74HCT241E, Package_DIP:DIP-20_W7.62mm_LongPads, F.Cu at (76.9, 64.6)
- J4: value NTC -> NTC1
- R1, R16, R2, R9: footprint Resistor_THT:R_Axial_DIN0309_L9.0mm_D3.2mm_P12.70mm_Horizontal -> Resistor_THT:R_Axial_DIN0309_L9.0mm_D3.2mm_P2.54mm_Vertical
- moved C2 46.8 mm to (81.9, 55.5), turned to 180 degrees
- moved PS1 45.7 mm to (82.7, 41.0), turned to 180 degrees
- moved R21 32.0 mm to (73.6, 51.8), turned to 180 degrees
- moved C1 29.0 mm to (46.0, 29.4)
- moved D8 27.0 mm to (64.0, 52.5), turned to 0 degrees
- moved J14 23.9 mm to (38.0, 118.6), turned to 90 degrees
- moved R1 16.6 mm to (88.0, 73.8)
- moved J13 16.6 mm to (38.3, 99.8), turned to 90 degrees
- moved R16 13.3 mm to (50.4, 91.5), turned to 180 degrees
- moved R2 12.4 mm to (88.0, 79.2)
- moved R9 8.23 mm to (43.8, 105.8), turned to 180 degrees
- moved R3 8.19 mm to (83.8, 90.4), turned to -90 degrees
- moved D7 7.61 mm to (107.5, 112.2)
- moved R17 7.34 mm to (49.0, 95.2)
- moved R14 4.58 mm to (44.5, 101.6)
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Connections:
- net /T_sensor renamed /T_sensor_1
- J3 pad 3: unconnected-(J3-SDA_I2C1/GPIO02-Pad3) -> /T_sensor_2
- R1 pad 1: /GPIO_Peltier1 -> /Gate_Peltier1
- R2 pad 1: /GPIO_Peltier2 -> /Gate_Peltier2
- R3 pad 1: /GPIO_Peltier3 -> /Gate_Peltier3
Routing:
- net GND: track 110.5 -> 61.2 mm
- net /GPIO_Peltier3: track 5.92 -> 40.1 mm
- net +3.3V: track 50.3 -> 76.9 mm, vias 0 -> 1
- net /T_sensor_2: track 0.00 -> 25.5 mm
- net /Gate_Peltier3: track 0.00 -> 22.9 mm
- net +24V: track 414.5 -> 433.2 mm
- net /Gate_Peltier1: track 0.00 -> 16.7 mm
- net /GPIO_Peltier1: track 4.66 -> 20.5 mm
- net /GPIO_Tacho_Fan2A: track 34.7 -> 19.9 mm
- net +5V: track 148.3 -> 161.7 mm, vias 4 -> 8
- net /Gate_Peltier2: track 0.00 -> 11.8 mm
- net Net-(Q3-G): track 23.2 -> 12.8 mm
- net /Tacho_Fan2A: track 6.68 -> 16.1 mm
- net /Tacho_Fan2B: track 6.64 -> 15.8 mm
- net /GPIO_Fan2: track 20.4 -> 28.8 mm
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Other:
- board text added: "PCB Ventil HUYGHE M.B. & J.M."
- board text added: "rev A"
