File: Kheprism/HW/PCB_Ventil/Kicad/PCB_Ventil.kicad_sch (KiCad schematic)
At the start: 53 parts, among them J1 Vin+, J10 Peltier3-, J11 Fan1A, J12 Fan1B, J13 Fan2A, J14 Fan2B, J15 Vin+, J16 Vin-, J17 Peltier1+, J18 Peltier1+, J2 Vin-, J3 Raspberry_Pi_4, J4 DS18B20, J5 Peltier1+, J6 Peltier1-, J7 Peltier2+, J8 Peltier2-, J9 Peltier3+, Q1 DMT6009LCT, Q2 DMT6009LCT, Q3 DMT6009LCT

Commit message: new rev with Mano
Parts:
- added J19: NTC2, TerminalBlock:TerminalBlock_MaiXu_MX126-5.0-03P_1x03_P5.00mm, symbol Connector:Screw_Terminal_01x03
- added J20, J21: Peltier1+, MountingHole:MountingHole_3.2mm_M3, symbol Mechanical:MountingHole
- added R22: 10k, Resistor_THT:R_Axial_DIN0309_L9.0mm_D3.2mm_P2.54mm_Vertical, symbol Device:R
- added U1: CD74HCT241E, Package_DIP:DIP-20_W7.62mm_LongPads, symbol 74xx:74LS241
- D5, D6, D7, D8: Farnell Part Number (none) -> BL-B5134-1-TBS20A; Farnell Price/Stock (none) -> 0.075
- J1, J10, J15, J16, J17, J18, J2, J5, J6, J7, J8, J9: Farnell Part Number 1287 -> 4966; Farnell Price/Stock 0.08 -> .18
- J11, J12, J13, J14: Farnell Part Number SWR25X-NRTC-S04-ST-BA -> 0470531000; Farnell Price/Stock 0.11 -> 0.44
- J4: value DS18B20 -> NTC1
- R1, R16, R2, R9: footprint Resistor_THT:R_Axial_DIN0309_L9.0mm_D3.2mm_P12.70mm_Horizontal -> Resistor_THT:R_Axial_DIN0309_L9.0mm_D3.2mm_P2.54mm_Vertical
Connections:
- net +3.3V: now also J19.1 (Pin_1), R22.1
- net +5V: now also U1.19 (OEb), U1.20 (VCC)
- net GND: now also J19.3 (Pin_3), U1.1 (OEa), U1.10 (GND)
- net GPIO_Peltier1: now also U1.17 (I3b), U1.2 (I0a), U1.4 (I1a); no longer R1.1
- net GPIO_Peltier2: now also U1.6 (I2a), U1.8 (I3a); no longer R2.1
- net GPIO_Peltier3: now also U1.11 (I0b), U1.13 (I1b), U1.15 (I2b); no longer R3.1
- net T_sensor_2: now reaches J3.3 (SDA_I2C1/GPIO02)
- net T_sensor_2: now also J19.2 (Pin_2), R22.2
- net T_sensor renamed T_sensor_1
- new net Gate_Peltier1: R1.1, U1.16 (O1a), U1.18 (O0a), U1.3 (O3b)
- new net Gate_Peltier2: R2.1, U1.12 (O3a), U1.14 (O2a)
- new net Gate_Peltier3: R3.1, U1.5 (O2b), U1.7 (O1b), U1.9 (O0b)
- no-connect marks 20 -> 19
Other:
- moved on the sheet: D8, J17, J18, J3, J4, R21, R7
