File: bike_lights2/bike_lights2.kicad_pcb (KiCad board)
At the start: 2 copper layers, 36 x 18 mm, 35 parts, among them J2 LED, J3 B+, P1 USB_C_Plug_USB2.0, U1 TL431DBZ, U3 MIC2289, U4 MCP6002-xMS, U5 MCP73831-2-ADI/OT

Commit message: a
Parts:
- removed H1: MountingHole_Pad, Connector_Wire:SolderWirePad_1x01_SMD_5x10mm
- added C10: 10u, Capacitor_SMD:C_0603_1608Metric, F.Cu at (90.1, 71.1)
- added SW1: TL49, footprints:TL49PO, F.Cu at (90.2, 64.8)
- C7: footprint Capacitor_SMD:C_0805_2012Metric_Pad1.18x1.45mm_HandSolder -> Capacitor_SMD:C_0603_1608Metric
- L1: value 10µ -> 6.8µ; footprint footprints:DO1813H -> footprints:EPL2014_2x2mm_inductor_Coilcraft
- moved J2 41.0 mm to (105.1, 57.6)
- moved L1 39.5 mm to (103.3, 64.8)
- moved R11 38.6 mm to (110.0, 65.7), turned to 90 degrees
- moved R12 38.4 mm to (109.5, 63.4)
- moved C6 38.2 mm to (102.8, 59.4)
- moved C8 38.2 mm to (101.8, 59.4)
- moved C9 38.2 mm to (100.8, 59.4)
- moved C3 38.0 mm to (102.4, 61.9)
- moved C4 38.0 mm to (100.8, 61.9)
- moved U3 37.6 mm to (104.9, 61.5)
- moved R15 37.3 mm to (108.9, 61.1)
- moved R19 37.3 mm to (107.4, 61.1)
- moved J3 14.4 mm to (98.1, 58.0)
- moved D1 8.90 mm to (99.1, 64.9)
- moved R21 8.03 mm to (96.2, 64.9), turned to 0 degrees
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Connections:
- D1 pad 2: +BATT -> /Vusb
- J3 pad 1: +BATT -> /Battery
- U5 pad 3: +BATT -> /Battery
Routing:
- net +BATT: track 1.60 -> 31.2 mm
- net GND: track 18.6 -> 39.1 mm, vias 0 -> 12
- net /Battery: track 0.00 -> 17.6 mm
- net +2V5: track 5.95 -> 15.2 mm
- net /LowBat: track 2.07 -> 6.63 mm
- net /CHG: track 0.00 -> 4.49 mm
- net /SW: track 0.00 -> 2.16 mm
- net /Blink: track 3.46 -> 5.04 mm
- net /Batt_mon: track 4.90 -> 6.40 mm
- net /FB: track 5.26 -> 6.68 mm
- net Net-(D1-K): track 0.00 -> 1.38 mm
- net /LED-: track 5.39 -> 4.23 mm
- net /LED+: track 6.05 -> 6.63 mm

Commit message: a
Parts:
- added R1: 5k1, Resistor_SMD:R_0603_1608Metric, F.Cu at (105.0, 59.5)
- added R14: 5k1, Resistor_SMD:R_0603_1608Metric, F.Cu at (106.5, 59.5)
- J2: footprint Connector_PinHeader_2.54mm:PinHeader_1x02_P2.54mm_Vertical -> footprints:JST_PH_1x02_P2.0-2.5mm_Vertical
- moved C10 31.9 mm to (116.2, 52.9), turned to -90 degrees
- moved C5 31.0 mm to (88.9, 56.0), turned to 180 degrees
- moved U1 30.4 mm to (88.5, 58.2), turned to 180 degrees
- moved R7 29.6 mm to (91.5, 52.9), turned to 0 degrees
- moved R3 28.6 mm to (90.6, 55.2), turned to -90 degrees
- moved U5 27.5 mm to (113.4, 52.8), turned to 180 degrees
- moved SW1 26.6 mm to (116.2, 59.2), turned to 180 degrees
- moved C1 26.3 mm to (91.9, 55.3), turned to 90 degrees
- moved R6 25.6 mm to (94.5, 52.6), turned to 0 degrees
- moved R2 25.0 mm to (91.3, 58.2), turned to -90 degrees
- moved C7 24.5 mm to (110.5, 52.0), turned to -90 degrees
- moved R4 23.9 mm to (91.3, 61.2), turned to 90 degrees
- moved R8 23.5 mm to (94.5, 54.1), turned to 180 degrees
- moved R5 21.2 mm to (92.9, 64.4), turned to 90 degrees
- moved U4 20.2 mm to (93.9, 58.1), turned to -90 degrees
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Connections:
- P1 pad A5: unconnected-(P1-CC-PadA5) -> /CC1
- P1 pad B5: unconnected-(P1-VCONN-PadB5) -> /CC2
Routing:
- net /Vusb: track 0.00 -> 20.7 mm
- net GND: track 39.1 -> 52.4 mm, vias 12 -> 18
- net +BATT: track 31.2 -> 44.0 mm, vias 0 -> 2
- net /Battery: track 17.6 -> 23.3 mm
- net /LowBat: track 6.63 -> 3.56 mm
- net /CC1: track 0.00 -> 2.98 mm
- net Net-(U5-PROG): track 0.00 -> 2.81 mm
- net /CC2: track 0.00 -> 2.53 mm
- net /LED-: track 4.23 -> 6.66 mm
- net Net-(D1-K): track 1.38 -> 2.66 mm
- net +2V5: track 15.2 -> 13.9 mm
- net /LED+: track 6.63 -> 7.83 mm
- net /FB: track 6.68 -> 7.82 mm
- net /CHG: track 4.49 -> 5.46 mm
- added copper zone on F.Cu, net +2V5
- added copper zone on F.Cu, net /Battery
- added copper zone on F.Cu, net /LED+
- added copper zone on F.Cu, net /Vref
- added copper zone on F.Cu, net /Vusb
Other:
- board text added: "+"
- board text added: "-"
- board text added: "Bike Lights"
- board text added: "ON"
- board text added: "revA 8/26 X.B."

Commit message: a
Parts:
- moved R5 4.58 mm to (89.0, 62.0), turned to 0 degrees
- moved C2 3.57 mm to (90.9, 63.7), turned to 180 degrees
- moved R10 2.13 mm to (93.9, 63.7), turned to 180 degrees
- moved R19 1.13 mm to (97.1, 62.0), turned to 0 degrees
- moved C3 1.12 mm to (103.4, 61.5)
- moved C4 1.12 mm to (105.0, 61.5)
- moved C6 1.12 mm to (103.0, 64.0)
- moved C8 1.12 mm to (104.0, 64.0)
- moved C9 1.12 mm to (105.0, 64.0)
- moved D1 1.10 mm to (108.8, 58.4)
- moved P1 1.10 mm to (104.2, 52.5)
- moved R1 1.10 mm to (105.0, 58.4)
- moved R14 1.10 mm to (106.5, 58.4)
- moved L1 1.00 mm to (103.1, 58.8)
- moved U3 1.00 mm to (100.4, 61.4)
Routing:
- net GND: track 52.4 -> 48.6 mm, vias 18 -> 19
- net /Vusb: track 20.7 -> 18.1 mm
- net +BATT: track 44.0 -> 45.3 mm
- net /Blink: track 5.18 -> 6.33 mm
- net /LED-: track 6.66 -> 7.53 mm
- net Net-(D1-K): track 2.66 -> 1.81 mm
- removed copper zone on F.Cu, net /Vusb

Commit message: update TL431 to T092
Parts:
- removed U1: TL431DBZ, Package_TO_SOT_SMD:SOT-23
- added U2: TL431LP, Package_TO_SOT_THT:TO-92_Inline, F.Cu at (89.0, 60.3)
- moved R5 2.12 mm to (90.5, 63.5)
- moved C2 1.30 mm to (90.9, 65.0)
- moved C5 0.85 mm to (89.2, 55.2), turned to 90 degrees
Routing:
- net +2V5: track 13.9 -> 16.4 mm
- net GND: track 48.6 -> 49.7 mm, vias 19 -> 15
- net /BlinkRC: track 5.11 -> 5.65 mm
