File: split-flap_display/split-flap_display.kicad_sch (KiCad schematic)
At the start: 27 parts, among them J1 A, J10 Hall4, J11 Hall5, J12 Conn_01x10, J13 Conn_01x10, J2 B, J3 C, J4 D, J5 E, J6 F, J7 Hall1, J8 Hall2, J9 Hall3, U1 MIC59P60, U2 ESP-12, U3 MIC59P60, U4 MIC59P60, U5 74LS597

Commit message: added split flap source files & assembly
Parts:
- removed J12, J13: Conn_01x10, symbol Connector_Generic:Conn_01x10
- removed JP1, JP2: Jumper_2_Bridged, symbol Jumper:Jumper_2_Bridged
- removed R6, R7: R, symbol Device:R
- added C1, C3, C4: 100n, Capacitor_THT:C_Disc_D6.0mm_W2.5mm_P5.00mm, symbol Device:C
- added C2, C5, C6, C7: 100u, Capacitor_THT:CP_Radial_D8.0mm_P5.00mm, symbol Device:C_Polarized
- added J12: Chain_OUT, Connector_PinHeader_2.54mm:PinHeader_1x07_P2.54mm_Vertical, symbol Connector_Generic:Conn_01x07
- added J13: Chain_IN, Connector_PinHeader_2.54mm:PinHeader_1x07_P2.54mm_Vertical, symbol Connector_Generic:Conn_01x07
- added R8: 10k, Resistor_THT:R_Axial_DIN0207_L6.3mm_D2.5mm_P2.54mm_Vertical, symbol Device:R
- added U6: LevelShifter_4ch, footprints:DIP-12_LevelShifter, symbol _MYLIBRARY:LevelShifter_4ch
- J1, J2, J3, J4, J5, J6: footprint (none) -> Connector_PinHeader_2.54mm:PinHeader_1x05_P2.54mm_Vertical
- J10, J11, J7, J8, J9: footprint (none) -> Connector_PinHeader_2.54mm:PinHeader_1x03_P2.54mm_Vertical
- R1, R2, R3, R4, R5: footprint (none) -> Resistor_THT:R_Axial_DIN0207_L6.3mm_D2.5mm_P5.08mm_Vertical
Connections:
- net Hall5 is gone; now on net Hall0: U5.5 (F)
- net Hall6 is gone; now on net GND: U5.6 (G)
- net Hall7 is gone; now on net GND: U5.7 (H)
- net +3.3V: now also U2.1 (REST), U2.3 (CH_PD), C1.1, C2.1, U6.3 (VCCL)
- net +5V: now also C3.1, C4.1, C5.1, C6.1, C7.1, J12.2 (Pin_2), J13.2 (Pin_2), U6.10 (VCCH)
- net CLK: now also U5.11 (SCK), J12.5 (Pin_5), J13.5 (Pin_5), U6.11 (B2)
- net D1: no longer U1.4 (DIN)
- net D2: no longer U1.7 (DOUT), U3.4 (DIN)
- net D3: no longer U3.7 (DOUT), U4.4 (DIN)
- net D4: no longer U4.7 (DOUT), U5.14 (SER)
- net GND: now also U5.15 (A), C1.2, C2.2, C3.2, C4.2, C5.2, C6.2, C7.2, J12.1 (Pin_1), J12.7 (Pin_7), J13.1 (Pin_1), J13.7 (Pin_7), R8.2, U6.4 (GND), U6.9 (GND)
- net Hall0: no longer U5.15 (A)
- net Hall1: now also U5.4 (E); no longer U5.1 (B)
- net Hall2: now also U5.3 (D); no longer U5.2 (C)
- net Hall3: now also U5.2 (C); no longer U5.3 (D)
- net Hall4: now also U5.1 (B); no longer U5.4 (E)
- net ~{CS}: now also J12.6 (Pin_6), J13.6 (Pin_6), U6.12 (B1)
- net ~{CS}_3v3: now reaches U2.4 (GPIO16)
- net ~{CS}_3v3: now also U6.1 (A1)
- net CLK_3v3: now reaches U2.5 (GPIO14)
- net CLK_3v3: now also U6.2 (A2)
- net Dm_3v3: now reaches U2.6 (GPIO12)
- net Dm_3v3: now also U6.5 (A3)
- net D5 renamed Dhout
- net Dhout: now also J13.3 (Pin_3), U6.7 (B4)
- net DOUT renamed Dhout_3v3
- net Dhout_3v3: now also U6.6 (A4)
- new net DHin: J12.3 (Pin_3), R8.1, U5.14 (SER)
- new net Dm1: J13.4 (Pin_4), U1.4 (DIN), U6.8 (B3)
- new net Dm2: U1.7 (DOUT), U3.4 (DIN)
- new net Dm3: U3.7 (DOUT), U4.4 (DIN)
- new net Dm4: J12.4 (Pin_4), U4.7 (DOUT)
- no-connect marks 6 -> 3
Other:
- note removed: "Open when chaining Close when MCU is placed"
