File: RCP_PWM_breakout/RCP_PWM_breakout.kicad_pcb (KiCad board)
At the start: 4 copper layers, 99.5 x 75.2 mm, 135 parts, among them IC2 TLS208D1EJVXUMA1, J1 VSUP 12V, J11 Conn_02x23_Odd_Even, J13 GND, J14 FlexGUI, J19 SSW-102-02-T-T-RA, J2 PWM, SW1 SW_DIP_x03, U1 FR50MHNR, U11 74LVC2G04, U12 74LVC2G04, U13 74LVC2G04, U14 74LVC2G04, U2 FR50MHNR, U3 FR50MHNR, U4 FR50MHNR, U5 FR50MHNR, U6 FR50MHNR, U7 FR50MHNR, U8 FR50MHNR

Commit message: added revB
Parts:
- JP2, JP3, JP4: moved to B.Cu
- JP5: value SolderJumper_3_Bridged123 -> PS_EN
- U1, U2, U3, U4, U5, U6, U7, U8: value FR50MHNR -> HBFR-2521Z
- moved JP2 3.60 mm to (69.6, 108.0)
- moved JP4 2.15 mm to (67.1, 108.0)
- moved D12 1.06 mm to (54.4, 70.9)
- moved D13 1.06 mm to (72.2, 70.9)
- moved D8 1.06 mm to (89.9, 70.9)
- moved R24 1.06 mm to (58.4, 70.9)
- moved R21 1.06 mm to (94.0, 70.8)
- moved R25 1.06 mm to (76.1, 70.9)
- moved R23 1.05 mm to (42.1, 70.9)
- moved D9 1.05 mm to (38.0, 70.9)
- moved TP8 0.76 mm to (97.0, 96.3)
- moved TP21 0.32 mm to (85.1, 70.9)
- moved TP35 0.32 mm to (33.2, 70.9)
- moved TP36 0.32 mm to (49.5, 70.9)
- moved TP37 0.32 mm to (67.3, 70.9)
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Connections:
- J11 pad 10: /INTA_GD_VH -> /INTA_GD_VL
- J11 pad 11: /INTA_GD_WL -> /INTA_GD_WH
- J11 pad 12: /INTA_GD_WH -> /INTA_GD_WL
- J11 pad 13: GND -> /SCLK_GD_HS
- J11 pad 14: /SCLK_GD_HS -> GND
- J11 pad 15: /SCLK_GD_LS -> /MISO_GD_HS
- J11 pad 16: /MISO_GD_HS -> /SCLK_GD_LS
- J11 pad 17: /MISO_GD_LS -> /MOSI_GD_HS
- J11 pad 18: /MOSI_GD_HS -> /MISO_GD_LS
- J11 pad 19: /MOSI_GD_LS -> /CS_GD_HSn
- J11 pad 20: /CS_GD_HSn -> /MOSI_GD_LS
- J11 pad 21: /CS_GD_LSn -> /FSS_HS_u
- J11 pad 22: /FSS_HS_u -> /CS_GD_LSn
- J11 pad 23: /MCU_EN_FLYBK_LS -> /MCU_EN_FLYBK_HS
- J11 pad 24: /MCU_EN_FLYBK_HS -> /MCU_EN_FLYBK_LS
- J11 pad 25: /FSENB_n_u -> VCC
- J11 pad 26: VCC -> /FSENB_n_u
- J11 pad 27: /FSS_LS_u -> /VBUSDIVX
- J11 pad 28: /VBUSDIVbyX -> /FSS_LS_u
- J11 pad 29: /VGD_LDO -> AGND_u
- J11 pad 30: AGND_u -> /VGD_LDO
- J11 pad 31: /INTB_GD_LSn -> /INTB_GD_HSn
- J11 pad 32: /INTB_GD_HSn -> /INTB_GD_LSn
- J11 pad 33: /VDDIO -> GND
- J11 pad 34: GND -> /VDDIO
- J11 pad 35: /AOUT_GD_UL -> /AOUT_GD_UH
- J11 pad 36: /AOUT_GD_UH -> /AOUT_GD_UL
- J11 pad 37: /AOUT_GD_VL -> /AOUT_GD_VH
- J11 pad 38: /AOUT_GD_VH -> /AOUT_GD_VL
- J11 pad 39: /AOUT_GD_WL -> /AOUT_GD_WH
- J11 pad 40: /AOUT_GD_WH -> /AOUT_GD_WL
- J11 pad 41: /PWMLU -> /PWMHU
- J11 pad 42: /PWMHU -> /PWMLU
- J11 pad 43: /PWMLV -> /PWMHV
- J11 pad 44: /PWMHV -> /PWMLV
- J11 pad 45: /PWMLW -> /PWMHW
- J11 pad 46: /PWMHW -> /PWMLW
- J11 pad 5: /GSENLW -> /GSENHW
- J11 pad 6: /GSENHW -> /GSENLW
- J11 pad 7: /INTA_GD_UL -> /INTA_GD_UH
- J11 pad 8: /INTA_GD_UH -> /INTA_GD_UL
- J11 pad 9: /INTA_GD_VL -> /INTA_GD_VH
- J19 pad 1: GND -> /Vin_12V
- J19 pad 3: /Vin_12V -> GND
- J19 pad 4: GND -> /Vin_12V
- J19 pad 6: /Vin_12V -> GND
- TP62 pad 1: /VBUSDIVbyX -> /VBUSDIVX
- U1 pad 4: unconnected-(U1-NC-Pad4) -> /PWMHU_i
- U2 pad 4: unconnected-(U2-NC-Pad4) -> /PWMLU_i
- U3 pad 4: unconnected-(U3-NC-Pad4) -> /PWMHV_i
- U4 pad 4: unconnected-(U4-NC-Pad4) -> /PWMLV_i
- U5 pad 4: unconnected-(U5-NC-Pad4) -> /PWMHW_i
- U6 pad 4: unconnected-(U6-NC-Pad4) -> /PWMLW_i
- U7 pad 4: unconnected-(U7-NC-Pad4) -> /PWMHM_i
- U8 pad 4: unconnected-(U8-NC-Pad4) -> /PWMLM_i
Routing:
- net GND: track 127.9 -> 44.3 mm, vias 18 -> 26
- net /VBUSDIVbyX: track 33.6 -> 0.00 mm, vias 2 -> 0
- net /VBUSDIVX: track 0.00 -> 29.5 mm, vias 0 -> 2
- net VCC: track 140.5 -> 123.2 mm, vias 25 -> 27
- net /INTA_GD_WH: track 103.8 -> 89.9 mm, vias 4 -> 2
- net /PWMLM_i: track 12.8 -> 24.2 mm
- net /PWMLU_i: track 6.52 -> 17.9 mm
- net /PWMLW_i: track 12.8 -> 24.2 mm
- net /PWMLV_i: track 7.71 -> 19.1 mm
- net /PWMHW_i: track 10.3 -> 21.6 mm
- net /PWMHV_i: track 10.8 -> 22.1 mm
- net /PWMHM_i: track 6.26 -> 17.6 mm
- net /Vin_12V: track 54.0 -> 43.6 mm, vias 1 -> 3
- net /AOUT_GD_WL: track 111.3 -> 119.0 mm
- net /PWMHU_i: track 12.9 -> 20.3 mm
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Other:
- board text added: "+"
- board text added: "-"
- board text removed: "+ -"
