File: RCP_PWM_breakout/RCP_PWM_breakout.kicad_sch (KiCad schematic)
At the start: 134 parts, among them IC2 TLS208D1EJVXUMA1, J1 VSUP 12V, J11 Conn_02x23_Odd_Even, J13 GND, J14 FlexGUI, J19 SSW-102-02-T-T-RA, J2 PWM, SW1 SW_DIP_x03, U1 FR50MHNR, U11 74LVC2G04, U12 74LVC2G04, U13 74LVC2G04, U14 74LVC2G04, U2 FR50MHNR, U3 FR50MHNR, U4 FR50MHNR, U5 FR50MHNR, U6 FR50MHNR, U7 FR50MHNR, U8 FR50MHNR

Commit message: added revB
Parts:
- JP5: value SolderJumper_3_Bridged123 -> PS_EN
- U1, U2, U3, U4, U5, U6, U7, U8: value FR50MHNR -> HBFR-2521Z; symbol _MYLIBRARY:FR50MHNR -> GD_lib:HBFR-2521Z; Site https://www.deumol.com/goods.php?id=1722 -> https://www.broadcom.com/products/fiber-optic-modules-compo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
Connections:
- net AGND_u: now also J11.29 (Pin_29); no longer J11.30 (Pin_30)
- net AOUT_GD_UH: now also J11.35 (Pin_35); no longer J11.36 (Pin_36)
- net AOUT_GD_UL: now also J11.36 (Pin_36); no longer J11.35 (Pin_35)
- net AOUT_GD_VH: now also J11.37 (Pin_37); no longer J11.38 (Pin_38)
- net AOUT_GD_VL: now also J11.38 (Pin_38); no longer J11.37 (Pin_37)
- net AOUT_GD_WH: now also J11.39 (Pin_39); no longer J11.40 (Pin_40)
- net AOUT_GD_WL: now also J11.40 (Pin_40); no longer J11.39 (Pin_39)
- net CS_GD_HSn: now also J11.19 (Pin_19); no longer J11.20 (Pin_20)
- net CS_GD_LSn: now also J11.22 (Pin_22); no longer J11.21 (Pin_21)
- net FSENB_n_u: now also J11.26 (Pin_26); no longer J11.25 (Pin_25)
- net FSS_HS_u: now also J11.21 (Pin_21); no longer J11.22 (Pin_22)
- net FSS_LS_u: now also J11.28 (Pin_28); no longer J11.27 (Pin_27)
- net GND: now also J11.14 (Pin_14), J11.33 (Pin_33), J19.3 (Pin_3), J19.6 (Pin_6); no longer J11.13 (Pin_13), J11.34 (Pin_34), J19.1 (Pin_1), J19.4 (Pin_4)
- net GSENHW: now also J11.5 (Pin_5); no longer J11.6 (Pin_6)
- net GSENLW: now also J11.6 (Pin_6); no longer J11.5 (Pin_5)
- net INTA_GD_UH: now also J11.7 (Pin_7); no longer J11.8 (Pin_8)
- net INTA_GD_UL: now also J11.8 (Pin_8); no longer J11.7 (Pin_7)
- net INTA_GD_VH: now also J11.9 (Pin_9); no longer J11.10 (Pin_10)
- net INTA_GD_VL: now also J11.10 (Pin_10); no longer J11.9 (Pin_9)
- net INTA_GD_WH: now also J11.11 (Pin_11); no longer J11.12 (Pin_12)
- net INTA_GD_WL: now also J11.12 (Pin_12); no longer J11.11 (Pin_11)
- net INTB_GD_HSn: now also J11.31 (Pin_31); no longer J11.32 (Pin_32)
- net INTB_GD_LSn: now also J11.32 (Pin_32); no longer J11.31 (Pin_31)
- net MCU_EN_FLYBK_HS: now also J11.23 (Pin_23); no longer J11.24 (Pin_24)
- net MCU_EN_FLYBK_LS: now also J11.24 (Pin_24); no longer J11.23 (Pin_23)
- net MISO_GD_HS: now also J11.15 (Pin_15); no longer J11.16 (Pin_16)
- net MISO_GD_LS: now also J11.18 (Pin_18); no longer J11.17 (Pin_17)
- net MOSI_GD_HS: now also J11.17 (Pin_17); no longer J11.18 (Pin_18)
- net MOSI_GD_LS: now also J11.20 (Pin_20); no longer J11.19 (Pin_19)
- net PWMHM_i: now also U7.4 (RL)
- net PWMHU: now also J11.41 (Pin_41); no longer J11.42 (Pin_42)
- net PWMHU_i: now also U1.4 (RL)
- net PWMHV: now also J11.43 (Pin_43); no longer J11.44 (Pin_44)
- net PWMHV_i: now also U3.4 (RL)
- net PWMHW: now also J11.45 (Pin_45); no longer J11.46 (Pin_46)
- net PWMHW_i: now also U5.4 (RL)
- net PWMLM_i: now also U8.4 (RL)
- net PWMLU: now also J11.42 (Pin_42); no longer J11.41 (Pin_41)
- net PWMLU_i: now also U2.4 (RL)
- net PWMLV: now also J11.44 (Pin_44); no longer J11.43 (Pin_43)
- net PWMLV_i: now also U4.4 (RL)
- net PWMLW: now also J11.46 (Pin_46); no longer J11.45 (Pin_45)
- net PWMLW_i: now also U6.4 (RL)
- net SCLK_GD_HS: now also J11.13 (Pin_13); no longer J11.14 (Pin_14)
- net SCLK_GD_LS: now also J11.16 (Pin_16); no longer J11.15 (Pin_15)
- net VBUSDIVX: now also J11.27 (Pin_27); no longer J11.28 (Pin_28)
- net VCC: now also J11.25 (Pin_25); no longer J11.26 (Pin_26)
- net VDDIO: now also J11.34 (Pin_34); no longer J11.33 (Pin_33)
- net VGD_LDO: now also J11.30 (Pin_30); no longer J11.29 (Pin_29)
- net Vin_12V: now also J19.1 (Pin_1), J19.4 (Pin_4); no longer J19.3 (Pin_3), J19.6 (Pin_6)
Other:
- moved on the sheet: J19
